File: design/CAN.sch (KiCad schematic (older format))
At the start: 4 parts, among them U4 TJA1051TK3

Commit message: initial commit
Parts:
- C33, C34: footprint CRF1:SMD-0603_c -> Capacitors_SMD:C_0603
- R23: footprint CRF1:SMD-0603_r -> Resistors_SMD:R_0603
Changed lines of the file:
@@
 U 1 1 53F59FA3
 P 5050 4450
-F 0 "C33" H 5075 4550 40  0000 L CNN
-F 1 "2.2u" H 5075 4375 40  0000 L CNN
-F 2 "CRF1:SMD-0603_c" H 5088 4300 30  0001 C CNN
-F 3 "" H 5050 4450 60  0000 C CNN
+F 0 "C33" H 5075 4550 40 0000 L CNN
+F 1 "2.2u" H 5075 4375 40 0000 L CNN
+F 2 "Capacitors_SMD:C_0603" H 5088 4300 30 0001 C CNN
+F 3 "" H 5050 4450 60 0000 C CNN
 	1    5050 4450
+	1    0    0    -1
+$EndComp
+$Comp
+L TJA1051TK3 U4
+U 1 1 5A8B2B4D
+P 6000 4000
+F 0 "U4" H 6000 4300 60 0000 C CNN
+F 1 "TJA1051TK3" H 6000 4400 60 0000 C CNN
+F 2 "Housings_DFN_QFN:DFN-8-1EP_3x3mm_Pitch0.65mm" H 6000 4000 60 0001 C CNN
+F 3 "" H 6000 4000 60 0000 C CNN
+	1    6000 4000
+	1    0    0    -1
+$EndComp
+$Comp
+L C C34
+U 1 1 5A8B2DCC
+P 6625 4450
+F 0 "C34" H 6650 4550 40 0000 L CNN
+F 1 "2.2u" H 6650 4375 40 0000 L CNN
+F 2 "Capacitors_SMD:C_0603" H 6663 4300 30 0001 C CNN
+F 3 "" H 6625 4450 60 0000 C CNN
+	1    6625 4450
+	1    0    0    -1
+$EndComp
+$Comp
+L +5V #PWR063
+U 1 1 5A8B3017
+P 5050 3750
+F 0 "#PWR063" H 5050 3600 50 0001 C CNN
+F 1 "+5V" H 5050 3890 50 0000 C CNN
+F 2 "" H 5050 3750 50 0001 C CNN
+F 3 "" H 5050 3750 50 0001 C CNN
+	1    5050 3750
+	1    0    0    -1
+$EndComp
+$Comp
+L R R23
+U 1 1 5A8B3269
+P 6875 4000
+F 0 "R23" V 6955 4000 50 0000 C CNN
+F 1 "220R" V 6875 4000 50 0000 C CNN
+F 2 "Resistors_SMD:R_0603" V 6805 4000 50 0001 C CNN
+F 3 "" H 6875 4000 50 0001 C CNN
+	1    6875 4000
+	1    0    0    -1
+$EndComp
+$Comp
+L VCC #PWR064
+U 1 1 5A8B3886
+P 6625 3675
+F 0 "#PWR064" H 6625 3525 50 0001 C CNN
+F 1 "VCC" H 6625 3825 50 0000 C CNN
+F 2 "" H 6625 3675 50 0001 C CNN
+F 3 "" H 6625 3675 50 0001 C CNN
+	1    6625 3675
+	1    0    0    -1
+$EndComp
+$Comp
+L GND #PWR065
+U 1 1 5A8B3BF5
+P 6625 4825
+F 0 "#PWR065" H 6625 4575 50 0001 C CNN
+F 1 "GND" H 6625 4675 50 0000 C CNN
+F 2 "" H 6625 4825 50 0001 C CNN
+F 3 "" H 6625 4825 50 0001 C CNN
+	1    6625 4825
 	1    0    0    -1
 $EndComp
@@
 Text HLabel 7225 4050 2    60   Input ~ 0
 CANL
-$Comp
-L TJA1051TK3 U4
-U 1 1 5A8B2B4D
-P 6000 4000
-F 0 "U4" H 6000 4300 60  0000 C CNN
-F 1 "TJA1051TK3" H 6000 4400 60  0000 C CNN
-F 2 "Housings_DFN_QFN:DFN-8-1EP_3x3mm_Pitch0.65mm" H 6000 4000 60  0001 C CNN
-F 3 "" H 6000 4000 60  0000 C CNN
-	1    6000 4000
-	1    0    0    -1
-$EndComp
-$Comp
-L C C34
-U 1 1 5A8B2DCC
-P 6625 4450
-F 0 "C34" H 6650 4550 40  0000 L CNN
-F 1 "2.2u" H 6650 4375 40  0000 L CNN
-F 2 "CRF1:SMD-0603_c" H 6663 4300 30  0001 C CNN
-F 3 "" H 6625 4450 60  0000 C CNN
-	1    6625 4450
-	1    0    0    -1
-$EndComp
-$Comp
-L +5V #PWR063
-U 1 1 5A8B3017
-P 5050 3750
-F 0 "#PWR063" H 5050 3600 50  0001 C CNN
-F 1 "+5V" H 5050 3890 50  0000 C CNN
-F 2 "" H 5050 3750 50  0001 C CNN
-F 3 "" H 5050 3750 50  0001 C CNN
-	1    5050 3750
-	1    0    0    -1
-$EndComp
-$Comp
-L R R23
-U 1 1 5A8B3269
-P 6875 4000
-F 0 "R23" V 6955 4000 50  0000 C CNN
-F 1 "220R" V 6875 4000 50  0000 C CNN
-F 2 "CRF1:SMD-0603_r" V 6805 4000 50  0001 C CNN
-F 3 "" H 6875 4000 50  0001 C CNN
-	1    6875 4000
-	1    0    0    -1
-$EndComp
-$Comp
-L VCC #PWR064
-U 1 1 5A8B3886
-P 6625 3675
-F 0 "#PWR064" H 6625 3525 50  0001 C CNN
-F 1 "VCC" H 6625 3825 50  0000 C CNN
-F 2 "" H 6625 3675 50  0001 C CNN
-F 3 "" H 6625 3675 50  0001 C CNN
-	1    6625 3675
-	1    0    0    -1
-$EndComp
-$Comp
-L GND #PWR065
-U 1 1 5A8B3BF5
-P 6625 4825
-F 0 "#PWR065" H 6625 4575 50  0001 C CNN
-F 1 "GND" H 6625 4675 50  0000 C CNN
-F 2 "" H 6625 4825 50  0001 C CNN
-F 3 "" H 6625 4825 50  0001 C CNN
-	1    6625 4825
-	1    0    0    -1
-$EndComp
 Wire Wire Line
 	6750 4200 6750 4050
@@
 Wire Wire Line
 	6000 4775 6000 4450
-Connection ~ 6000 4775
 Wire Wire Line
 	5275 3950 5550 3950
 Wire Wire Line
 	5050 4600 5050 4775
-Connection ~ 5275 4775
 Wire Wire Line
 	5050 4050 5550 4050
-Connection ~ 5050 4050
 Wire Wire Line
 	6450 3850 6500 3850
 Wire Wire Line
 	6500 3850 6500 4775
-Connection ~ 6500 4775
 Wire Wire Line
 	6875 3850 6875 3800
-Connection ~ 6875 3800
 Wire Wire Line
 	6875 4150 6875 4200
-Connection ~ 6875 4200
 Wire Wire Line
 	7025 4200 7025 4050
@@
 Wire Wire Line
 	6750 4200 7025 4200
-Connection ~ 6625 4150
-Connection ~ 6625 4775
 Wire Wire Line
 	5050 4775 6625 4775
@@
 Wire Wire Line
 	5275 3950 5275 4775
+Connection ~ 6000 4775
+Connection ~ 5275 4775
+Connection ~ 5050 4050
+Connection ~ 6500 4775
+Connection ~ 6875 3800
+Connection ~ 6875 4200
+Connection ~ 6625 4150
+Connection ~ 6625 4775
 $EndSCHEMATC

Commit message: TESC 1.4
Parts:
- U4: manf# (none) -> TJA1051TK/3
Changed lines of the file:
@@
 F 2 "Housings_DFN_QFN:DFN-8-1EP_3x3mm_Pitch0.65mm" H 6000 4000 60  0001 C CNN
 F 3 "" H 6000 4000 60  0000 C CNN
+F 4 "TJA1051TK/3" H 6000 4000 60  0001 C CNN "manf#"
 	1    6000 4000
 	1    0    0    -1

Commit message: Add manf# field
Parts:
- C33, C34: manf# (none) -> C1608X5R1C225K080AB
- R23: manf# (none) -> CR0603-FX-2200ELF
- U4: manf# TJA1051TK/3 -> TJA1051TK/3,118
Changed lines of the file:
@@
 U 1 1 53F59FA3
 P 5050 4450
-F 0 "C33" H 5075 4550 40  0000 L CNN
-F 1 "2.2u" H 5075 4375 40  0000 L CNN
-F 2 "Capacitors_SMD:C_0603" H 5088 4300 30  0001 C CNN
-F 3 "" H 5050 4450 60  0000 C CNN
+F 0 "C33" H 5075 4550 40 0000 L CNN
+F 1 "2.2u" H 5075 4375 40 0000 L CNN
+F 2 "Capacitors_SMD:C_0603" H 5088 4300 30 0001 C CNN
+F 3 "" H 5050 4450 60 0000 C CNN
+F 4 "C1608X5R1C225K080AB" H 5075 4650 50 0001 C CNN "manf#"
 	1    5050 4450
 	1    0    0    -1
@@
 U 1 1 5A8B2B4D
 P 6000 4000
-F 0 "U4" H 6000 4300 60  0000 C CNN
-F 1 "TJA1051TK3" H 6000 4400 60  0000 C CNN
-F 2 "Housings_DFN_QFN:DFN-8-1EP_3x3mm_Pitch0.65mm" H 6000 4000 60  0001 C CNN
-F 3 "" H 6000 4000 60  0000 C CNN
-F 4 "TJA1051TK/3" H 6000 4000 60  0001 C CNN "manf#"
+F 0 "U4" H 6000 4300 60 0000 C CNN
+F 1 "TJA1051TK3" H 6000 4400 60 0000 C CNN
+F 2 "Housings_DFN_QFN:DFN-8-1EP_3x3mm_Pitch0.65mm" H 6000 4000 60 0001 C CNN
+F 3 "" H 6000 4000 60 0000 C CNN
+F 4 "TJA1051TK/3,118" H 6000 4000 60 0001 C CNN "manf#"
 	1    6000 4000
 	1    0    0    -1
@@
 U 1 1 5A8B2DCC
 P 6625 4450
-F 0 "C34" H 6650 4550 40  0000 L CNN
-F 1 "2.2u" H 6650 4375 40  0000 L CNN
-F 2 "Capacitors_SMD:C_0603" H 6663 4300 30  0001 C CNN
-F 3 "" H 6625 4450 60  0000 C CNN
+F 0 "C34" H 6650 4550 40 0000 L CNN
+F 1 "2.2u" H 6650 4375 40 0000 L CNN
+F 2 "Capacitors_SMD:C_0603" H 6663 4300 30 0001 C CNN
+F 3 "" H 6625 4450 60 0000 C CNN
+F 4 "C1608X5R1C225K080AB" H 6650 4650 50 0001 C CNN "manf#"
 	1    6625 4450
 	1    0    0    -1
@@
 U 1 1 5A8B3017
 P 5050 3750
-F 0 "#PWR063" H 5050 3600 50  0001 C CNN
-F 1 "+5V" H 5050 3890 50  0000 C CNN
-F 2 "" H 5050 3750 50  0001 C CNN
-F 3 "" H 5050 3750 50  0001 C CNN
+F 0 "#PWR063" H 5050 3600 50 0001 C CNN
+F 1 "+5V" H 5050 3890 50 0000 C CNN
+F 2 "" H 5050 3750 50 0001 C CNN
+F 3 "" H 5050 3750 50 0001 C CNN
 	1    5050 3750
 	1    0    0    -1
@@
 U 1 1 5A8B3269
 P 6875 4000
-F 0 "R23" V 6955 4000 50  0000 C CNN
-F 1 "220R" V 6875 4000 50  0000 C CNN
-F 2 "Resistors_SMD:R_0603" V 6805 4000 50  0001 C CNN
-F 3 "" H 6875 4000 50  0001 C CNN
+F 0 "R23" V 6955 4000 50 0000 C CNN
+F 1 "220R" V 6875 4000 50 0000 C CNN
+F 2 "Resistors_SMD:R_0603" V 6805 4000 50 0001 C CNN
+F 3 "" H 6875 4000 50 0001 C CNN
+F 4 "CR0603-FX-2200ELF" H 6955 4100 50 0001 C CNN "manf#"
 	1    6875 4000
 	1    0    0    -1
@@
 U 1 1 5A8B3886
 P 6625 3675
-F 0 "#PWR064" H 6625 3525 50  0001 C CNN
-F 1 "VCC" H 6625 3825 50  0000 C CNN
-F 2 "" H 6625 3675 50  0001 C CNN
-F 3 "" H 6625 3675 50  0001 C CNN
+F 0 "#PWR064" H 6625 3525 50 0001 C CNN
+F 1 "VCC" H 6625 3825 50 0000 C CNN
+F 2 "" H 6625 3675 50 0001 C CNN
+F 3 "" H 6625 3675 50 0001 C CNN
 	1    6625 3675
 	1    0    0    -1
@@
 U 1 1 5A8B3BF5
 P 6625 4825
-F 0 "#PWR065" H 6625 4575 50  0001 C CNN
-F 1 "GND" H 6625 4675 50  0000 C CNN
-F 2 "" H 6625 4825 50  0001 C CNN
-F 3 "" H 6625 4825 50  0001 C CNN
+F 0 "#PWR065" H 6625 4575 50 0001 C CNN
+F 1 "GND" H 6625 4675 50 0000 C CNN
+F 2 "" H 6625 4825 50 0001 C CNN
+F 3 "" H 6625 4825 50 0001 C CNN
 	1    6625 4825
 	1    0    0    -1

Commit message: Support KiCad 5.1.4
Parts:
- C33, C34: footprint Capacitors_SMD:C_0603 -> Capacitor_SMD:C_0603_1608Metric; symbol C -> Device:C
- R23: footprint Resistors_SMD:R_0603 -> Resistor_SMD:R_0603_1608Metric; symbol R -> Device:R
- U4: footprint Housings_DFN_QFN:DFN-8-1EP_3x3mm_Pitch0.65mm -> Package_DFN_QFN:DFN-8-1EP_3x3mm_P0.65mm_EP1.55x2.4mm; symbol TJA1051TK3 -> crf_1:TJA1051TK3
Connections:
- wire segments 24 -> 32
Changed lines of the file:
@@
-EESchema Schematic File Version 2
-LIBS:power
-LIBS:device
-LIBS:transistors
-LIBS:conn
-LIBS:linear
-LIBS:regul
-LIBS:74xx
-LIBS:cmos4000
-LIBS:adc-dac
-LIBS:memory
-LIBS:xilinx
-LIBS:microcontrollers
-LIBS:dsp
-LIBS:microchip
-LIBS:analog_switches
-LIBS:motorola
-LIBS:texas
-LIBS:switches
-LIBS:intel
-LIBS:audio
-LIBS:interface
-LIBS:digital-audio
-LIBS:philips
-LIBS:display
-LIBS:cypress
-LIBS:siliconi
-LIBS:opto
-LIBS:atmel
-LIBS:contrib
-LIBS:valves
-LIBS:crf_1
+EESchema Schematic File Version 4
 LIBS:VESC_6-cache
-EELAYER 25 0
+EELAYER 30 0
 EELAYER END
 $Descr A4 11693 8268
@@
 $EndDescr
 $Comp
-L C C33
+L Device:C C33
 U 1 1 53F59FA3
 P 5050 4450
 F 0 "C33" H 5075 4550 40  0000 L CNN
 F 1 "2.2u" H 5075 4375 40  0000 L CNN
-F 2 "Capacitors_SMD:C_0603" H 5088 4300 30  0001 C CNN
+F 2 "Capacitor_SMD:C_0603_1608Metric" H 5088 4300 30  0001 C CNN
 F 3 "" H 5050 4450 60  0000 C CNN
 F 4 "C1608X5R1C225K080AB" H 5075 4650 50  0001 C CNN "manf#"
@@
 $EndComp
 $Comp
-L TJA1051TK3 U4
+L crf_1:TJA1051TK3 U4
 U 1 1 5A8B2B4D
 P 6000 4000
 F 0 "U4" H 6000 4300 60  0000 C CNN
 F 1 "TJA1051TK3" H 6000 4400 60  0000 C CNN
-F 2 "Housings_DFN_QFN:DFN-8-1EP_3x3mm_Pitch0.65mm" H 6000 4000 60  0001 C CNN
+F 2 "Package_DFN_QFN:DFN-8-1EP_3x3mm_P0.65mm_EP1.55x2.4mm" H 6000 4000 60  0001 C CNN
 F 3 "" H 6000 4000 60  0000 C CNN
 F 4 "TJA1051TK/3,118" H 6000 4000 60  0001 C CNN "manf#"
@@
 $EndComp
 $Comp
-L C C34
+L Device:C C34
 U 1 1 5A8B2DCC
 P 6625 4450
 F 0 "C34" H 6650 4550 40  0000 L CNN
 F 1 "2.2u" H 6650 4375 40  0000 L CNN
-F 2 "Capacitors_SMD:C_0603" H 6663 4300 30  0001 C CNN
+F 2 "Capacitor_SMD:C_0603_1608Metric" H 6663 4300 30  0001 C CNN
 F 3 "" H 6625 4450 60  0000 C CNN
 F 4 "C1608X5R1C225K080AB" H 6650 4650 50  0001 C CNN "manf#"
@@
 $EndComp
 $Comp
-L +5V #PWR063
+L power:+5V #PWR063
 U 1 1 5A8B3017
 P 5050 3750
@@
 $EndComp
 $Comp
-L R R23
+L Device:R R23
 U 1 1 5A8B3269
 P 6875 4000
 F 0 "R23" V 6955 4000 50  0000 C CNN
 F 1 "220R" V 6875 4000 50  0000 C CNN
-F 2 "Resistors_SMD:R_0603" V 6805 4000 50  0001 C CNN
+F 2 "Resistor_SMD:R_0603_1608Metric" V 6805 4000 50  0001 C CNN
 F 3 "" H 6875 4000 50  0001 C CNN
 F 4 "CR0603-FX-2200ELF" H 6955 4100 50  0001 C CNN "manf#"
@@
 $EndComp
 $Comp
-L VCC #PWR064
+L power:VCC #PWR064
 U 1 1 5A8B3886
 P 6625 3675
@@
 $EndComp
 $Comp
-L GND #PWR065
+L power:GND #PWR065
 U 1 1 5A8B3BF5
 P 6625 4825
@@
 	6750 3950 6750 3800
 Wire Wire Line
-	6750 3800 7025 3800
+	6750 3800 6875 3800
 Wire Wire Line
 	6450 4150 6625 4150
 Wire Wire Line
-	6625 3675 6625 4300
+	6625 3675 6625 4150
 Wire Wire Line
-	6625 4600 6625 4825
+	6625 4600 6625 4775
 Wire Wire Line
 	6000 4775 6000 4450
@@
 	7025 3950 7225 3950
 Wire Wire Line
-	6750 4200 7025 4200
+	6750 4200 6875 4200
 Wire Wire Line
-	5050 4775 6625 4775
+	5050 4775 5275 4775
 Wire Wire Line
-	5050 3750 5050 4300
+	5050 3750 5050 4050
 Wire Wire Line
 	5275 3950 5275 4775
+Wire Wire Line
+	6000 4775 6500 4775
+Wire Wire Line
+	5275 4775 6000 4775
+Wire Wire Line
+	5050 4050 5050 4300
+Wire Wire Line
+	6500 4775 6625 4775
+Wire Wire Line
+	6875 3800 7025 3800
+Wire Wire Line
+	6875 4200 7025 4200
+Wire Wire Line
+	6625 4150 6625 4300
+Wire Wire Line
+	6625 4775 6625 4825
 Connection ~ 6000 4775
 Connection ~ 5275 4775

Commit message: Load KiCad 4.0.7 schematic symbols, footprints & 3D models
Parts:
- C33, C34: footprint Capacitor_SMD:C_0603_1608Metric -> Capacitors_SMD:C_0603
- R23: footprint Resistor_SMD:R_0603_1608Metric -> Resistors_SMD:R_0603
- U4: footprint Package_DFN_QFN:DFN-8-1EP_3x3mm_P0.65mm_EP1.55x2.4mm -> Housings_DFN_QFN:DFN-8-1EP_3x3mm_Pitch0.65mm
Changed lines of the file:
@@
 F 0 "C33" H 5075 4550 40  0000 L CNN
 F 1 "2.2u" H 5075 4375 40  0000 L CNN
-F 2 "Capacitor_SMD:C_0603_1608Metric" H 5088 4300 30  0001 C CNN
+F 2 "Capacitors_SMD:C_0603" H 5088 4300 30  0001 C CNN
 F 3 "" H 5050 4450 60  0000 C CNN
 F 4 "C1608X5R1C225K080AB" H 5075 4650 50  0001 C CNN "manf#"
@@
 F 0 "U4" H 6000 4300 60  0000 C CNN
 F 1 "TJA1051TK3" H 6000 4400 60  0000 C CNN
-F 2 "Package_DFN_QFN:DFN-8-1EP_3x3mm_P0.65mm_EP1.55x2.4mm" H 6000 4000 60  0001 C CNN
+F 2 "Housings_DFN_QFN:DFN-8-1EP_3x3mm_Pitch0.65mm" H 6000 4000 60  0001 C CNN
 F 3 "" H 6000 4000 60  0000 C CNN
 F 4 "TJA1051TK/3,118" H 6000 4000 60  0001 C CNN "manf#"
@@
 F 0 "C34" H 6650 4550 40  0000 L CNN
 F 1 "2.2u" H 6650 4375 40  0000 L CNN
-F 2 "Capacitor_SMD:C_0603_1608Metric" H 6663 4300 30  0001 C CNN
+F 2 "Capacitors_SMD:C_0603" H 6663 4300 30  0001 C CNN
 F 3 "" H 6625 4450 60  0000 C CNN
 F 4 "C1608X5R1C225K080AB" H 6650 4650 50  0001 C CNN "manf#"
@@
 F 0 "R23" V 6955 4000 50  0000 C CNN
 F 1 "220R" V 6875 4000 50  0000 C CNN
-F 2 "Resistor_SMD:R_0603_1608Metric" V 6805 4000 50  0001 C CNN
+F 2 "Resistors_SMD:R_0603" V 6805 4000 50  0001 C CNN
 F 3 "" H 6875 4000 50  0001 C CNN
 F 4 "CR0603-FX-2200ELF" H 6955 4100 50  0001 C CNN "manf#"
