File: design/nrf.sch (KiCad schematic (older format))
At the start: 17 parts, among them U8 NRF24L01P, U9 CONN_U_FL, X2 16M

Commit message: initial commit
Parts:
- C48, C49, C50, C51, C52, C53, C54, C55, C56, C57: footprint CRF1:SMD-0603_c -> Capacitors_SMD:C_0603
- R38: footprint CRF1:SMD-0603_r -> Resistors_SMD:R_0603

Commit message: initial commit
Parts:
- X2: footprint mojaKniznica:5x3.2KRISTALL -> Crystals:Crystal_SMD_5032_4Pads

Commit message: initial commit
Parts:
- C54, C55, C56, C57: footprint Capacitors_SMD:C_0603 -> Capacitors_SMD:C_0402
Changed lines of the file:
@@
 F 0 "C56" V 7225 3275 50  0000 L CNN
 F 1 "1.5p" V 7125 3275 50  0000 L CNN
-F 2 "Capacitors_SMD:C_0603" H 7013 3200 50  0001 C CNN
+F 2 "Capacitors_SMD:C_0402" H 7013 3200 50  0001 C CNN
 F 3 "" H 6975 3350 50  0001 C CNN
 	1    6975 3350
@@
 F 0 "C57" H 7375 3650 50  0000 L CNN
 F 1 "1p" H 7375 3550 50  0000 L CNN
-F 2 "Capacitors_SMD:C_0603" H 7288 3450 50  0001 C CNN
+F 2 "Capacitors_SMD:C_0402" H 7288 3450 50  0001 C CNN
 F 3 "" H 7250 3600 50  0001 C CNN
 	1    7250 3600
@@
 F 0 "C55" H 6750 4650 50  0000 L CNN
 F 1 "4.7p" H 6750 4575 50  0000 L CNN
-F 2 "Capacitors_SMD:C_0603" H 6663 4450 50  0001 C CNN
+F 2 "Capacitors_SMD:C_0402" H 6663 4450 50  0001 C CNN
 F 3 "" H 6625 4600 50  0001 C CNN
 	1    6625 4600
@@
 F 0 "C54" H 6325 4650 50  0000 L CNN
 F 1 "2.2n" H 6325 4575 50  0000 L CNN
-F 2 "Capacitors_SMD:C_0603" H 6238 4450 50  0001 C CNN
+F 2 "Capacitors_SMD:C_0402" H 6238 4450 50  0001 C CNN
 F 3 "" H 6200 4600 50  0001 C CNN
 	1    6200 4600
