File: design/nrf.sch (KiCad schematic (older format))
At the start: 17 parts, among them U8 NRF24L01P, U9 CONN_U_FL, X2 16M

Commit message: TESC 1.4
Parts:
- U8: manf# (none) -> nRF24L01P-T
Changed lines of the file:
@@
 F 2 "Housings_DFN_QFN:QFN-20-1EP_4x4mm_Pitch0.5mm" H 4175 3675 60  0001 C CNN
 F 3 "" H 4175 3675 60  0001 C CNN
+F 4 "nRF24L01P-T" H 4175 3675 60  0001 C CNN "manf#"
 	1    4175 3675
 	1    0    0    -1

Commit message: Add manf# field
Parts:
- C48, C49, C50, C53: manf# (none) -> C0603X104J5RACTU
- C51, C52: manf# (none) -> 06031A150JAT2A
- C54: manf# (none) -> GRM155R71H222JA01J
- C55: manf# (none) -> GRM1555C2A4R7WA01D
- C56: manf# (none) -> GRM1555C2A1R5CA01D
- C57: manf# (none) -> GRM1555C2A1R0CA01D
- L3: manf# (none) -> LQG18HN8N2J00D
- L4: manf# (none) -> LQG18HN3N9S00D
- L5: manf# (none) -> LQG18HN2N7S00D
- R38: manf# (none) -> CR0603-FX-2202ELF
- U9: manf# (none) -> U.FL-R-SMT-1(40)
- X2: manf# (none) -> ABM3B-16.000MHZ-10-1-U-T

Commit message: Support KiCad 5.1.4
Parts:
- C48, C49, C50, C51, C52, C53: footprint Capacitors_SMD:C_0603 -> Capacitor_SMD:C_0603_1608Metric; symbol C -> Device:C
- C54, C55, C56, C57: footprint Capacitors_SMD:C_0402 -> Capacitor_SMD:C_0402_1005Metric; symbol C -> Device:C
- L3, L4, L5: footprint Inductors_SMD:L_0603 -> Inductor_SMD:L_0402_1005Metric; symbol L -> Device:L
- R38: footprint Resistors_SMD:R_0603 -> Resistor_SMD:R_0603_1608Metric; symbol R -> Device:R
- U8: footprint Housings_DFN_QFN:QFN-20-1EP_4x4mm_Pitch0.5mm -> Package_DFN_QFN:QFN-20-1EP_4x4mm_P0.5mm_EP2.5x2.5mm; symbol NRF24L01 -> crf_1:NRF24L01
- U9: symbol CONN_U_FL -> crf_1:CONN_U_FL
- X2: footprint Crystals:Crystal_SMD_5032_4Pads -> Crystal:Crystal_SMD_5032-4Pin_5.0x3.2mm; symbol CRYSTAL_SMD -> crf_1:CRYSTAL_SMD

Commit message: Load KiCad 4.0.7 schematic symbols, footprints & 3D models
Parts:
- C48, C49, C50, C51, C52, C53: footprint Capacitor_SMD:C_0603_1608Metric -> Capacitors_SMD:C_0603
- C54, C55, C56, C57: footprint Capacitor_SMD:C_0402_1005Metric -> Capacitors_SMD:C_0402
- L3, L4, L5: footprint Inductor_SMD:L_0402_1005Metric -> Inductors_SMD:L_0402
- R38: footprint Resistor_SMD:R_0603_1608Metric -> Resistors_SMD:R_0603
- U8: footprint Package_DFN_QFN:QFN-20-1EP_4x4mm_P0.5mm_EP2.5x2.5mm -> Housings_DFN_QFN:QFN-20-1EP_4x4mm_Pitch0.5mm
- X2: footprint Crystal:Crystal_SMD_5032-4Pin_5.0x3.2mm -> Crystals:Crystal_SMD_5032_4Pads
Changed lines of the file:
@@
 F 0 "U8" H 4500 4250 60  0000 C CNN
 F 1 "NRF24L01P" H 4800 3050 60  0000 C CNN
-F 2 "Package_DFN_QFN:QFN-20-1EP_4x4mm_P0.5mm_EP2.5x2.5mm" H 4175 3675 60  0001 C CNN
+F 2 "Housings_DFN_QFN:QFN-20-1EP_4x4mm_Pitch0.5mm" H 4175 3675 60  0001 C CNN
 F 3 "" H 4175 3675 60  0001 C CNN
 F 4 "nRF24L01P-T" H 4175 3675 60  0001 C CNN "manf#"
@@
 F 0 "C50" H 3925 5050 50  0000 L CNN
 F 1 "100n" H 3900 4900 50  0000 L CNN
-F 2 "Capacitor_SMD:C_0603_1608Metric" H 4138 4825 50  0001 C CNN
+F 2 "Capacitors_SMD:C_0603" H 4138 4825 50  0001 C CNN
 F 3 "" H 4100 4975 50  0001 C CNN
 F 4 "C0603X104J5RACTU" H 3925 5150 50  0001 C CNN "manf#"
@@
 F 0 "C51" V 5025 4725 50  0000 L CNN
 F 1 "15p" V 5025 4425 50  0000 L CNN
-F 2 "Capacitor_SMD:C_0603_1608Metric" H 5013 4475 50  0001 C CNN
+F 2 "Capacitors_SMD:C_0603" H 5013 4475 50  0001 C CNN
 F 3 "" H 4975 4625 50  0001 C CNN
 F 4 "06031A150JAT2A" H 5025 4825 50  0001 C CNN "manf#"
@@
 F 0 "C52" V 5025 5225 50  0000 L CNN
 F 1 "15p" V 5025 4925 50  0000 L CNN
-F 2 "Capacitor_SMD:C_0603_1608Metric" H 5013 4975 50  0001 C CNN
+F 2 "Capacitors_SMD:C_0603" H 5013 4975 50  0001 C CNN
 F 3 "" H 4975 5125 50  0001 C CNN
 F 4 "06031A150JAT2A" H 5025 5325 50  0001 C CNN "manf#"
@@
 F 0 "L5" V 6225 4050 50  0000 C CNN
 F 1 "2.7n" V 6300 4050 50  0000 C CNN
-F 2 "Inductor_SMD:L_0402_1005Metric" H 6350 4050 50  0001 C CNN
+F 2 "Inductors_SMD:L_0402" H 6350 4050 50  0001 C CNN
 F 3 "" H 6350 4050 50  0001 C CNN
 F 4 "LQG18HN2N7S00D" H 6225 4150 50  0001 C CNN "manf#"
@@
 F 0 "L3" H 5975 3725 50  0000 L CNN
 F 1 "8.2n" H 5975 3650 50  0000 L CNN
-F 2 "Inductor_SMD:L_0402_1005Metric" H 5925 3700 50  0001 C CNN
+F 2 "Inductors_SMD:L_0402" H 5925 3700 50  0001 C CNN
 F 3 "" H 5925 3700 50  0001 C CNN
 F 4 "LQG18HN8N2J00D" H 5975 3825 50  0001 C CNN "manf#"
@@
 F 0 "C56" V 7225 3275 50  0000 L CNN
 F 1 "1.5p" V 7125 3275 50  0000 L CNN
-F 2 "Capacitor_SMD:C_0402_1005Metric" H 7013 3200 50  0001 C CNN
+F 2 "Capacitors_SMD:C_0402" H 7013 3200 50  0001 C CNN
 F 3 "" H 6975 3350 50  0001 C CNN
 F 4 "GRM1555C2A1R5CA01D" H 7225 3375 50  0001 C CNN "manf#"
@@
 F 0 "C57" H 7375 3650 50  0000 L CNN
 F 1 "1p" H 7375 3550 50  0000 L CNN
-F 2 "Capacitor_SMD:C_0402_1005Metric" H 7288 3450 50  0001 C CNN
+F 2 "Capacitors_SMD:C_0402" H 7288 3450 50  0001 C CNN
 F 3 "" H 7250 3600 50  0001 C CNN
 F 4 "GRM1555C2A1R0CA01D" H 7375 3750 50  0001 C CNN "manf#"
@@
 F 0 "C55" H 6750 4650 50  0000 L CNN
 F 1 "4.7p" H 6750 4575 50  0000 L CNN
-F 2 "Capacitor_SMD:C_0402_1005Metric" H 6663 4450 50  0001 C CNN
+F 2 "Capacitors_SMD:C_0402" H 6663 4450 50  0001 C CNN
 F 3 "" H 6625 4600 50  0001 C CNN
 F 4 "GRM1555C2A4R7WA01D" H 6750 4750 50  0001 C CNN "manf#"
@@
 F 0 "C54" H 6325 4650 50  0000 L CNN
 F 1 "2.2n" H 6325 4575 50  0000 L CNN
-F 2 "Capacitor_SMD:C_0402_1005Metric" H 6238 4450 50  0001 C CNN
+F 2 "Capacitors_SMD:C_0402" H 6238 4450 50  0001 C CNN
 F 3 "" H 6200 4600 50  0001 C CNN
 F 4 "GRM155R71H222JA01J" H 6325 4750 50  0001 C CNN "manf#"
@@
 F 0 "L4" V 6225 3350 50  0000 C CNN
 F 1 "3.9n" V 6300 3350 50  0000 C CNN
-F 2 "Inductor_SMD:L_0402_1005Metric" H 6350 3350 50  0001 C CNN
+F 2 "Inductors_SMD:L_0402" H 6350 3350 50  0001 C CNN
 F 3 "" H 6350 3350 50  0001 C CNN
 F 4 "LQG18HN3N9S00D" H 6225 3450 50  0001 C CNN "manf#"
@@
 F 0 "C53" H 5275 3000 50  0000 L CNN
 F 1 "100n" H 5275 2925 50  0000 L CNN
-F 2 "Capacitor_SMD:C_0603_1608Metric" H 5188 2800 50  0001 C CNN
+F 2 "Capacitors_SMD:C_0603" H 5188 2800 50  0001 C CNN
 F 3 "" H 5150 2950 50  0001 C CNN
 F 4 "C0603X104J5RACTU" H 5275 3100 50  0001 C CNN "manf#"
@@
 F 0 "C48" H 3500 2775 50  0000 L CNN
 F 1 "100n" H 3500 2700 50  0000 L CNN
-F 2 "Capacitor_SMD:C_0603_1608Metric" H 3413 2575 50  0001 C CNN
+F 2 "Capacitors_SMD:C_0603" H 3413 2575 50  0001 C CNN
 F 3 "" H 3375 2725 50  0001 C CNN
 F 4 "C0603X104J5RACTU" H 3500 2875 50  0001 C CNN "manf#"
@@
 F 0 "R38" H 4575 2700 50  0000 C CNN
 F 1 "22k" H 4575 2600 50  0000 C CNN
-F 2 "Resistor_SMD:R_0603_1608Metric" V 4355 2650 50  0001 C CNN
+F 2 "Resistors_SMD:R_0603" V 4355 2650 50  0001 C CNN
 F 3 "" H 4425 2650 50  0001 C CNN
 F 4 "CR0603-FX-2202ELF" H 4575 2800 50  0001 C CNN "manf#"
@@
 F 0 "C49" V 4175 2825 50  0000 L CNN
 F 1 "100n" V 4175 2425 50  0000 L CNN
-F 2 "Capacitor_SMD:C_0603_1608Metric" H 4163 2525 50  0001 C CNN
+F 2 "Capacitors_SMD:C_0603" H 4163 2525 50  0001 C CNN
 F 3 "" H 4125 2675 50  0001 C CNN
 F 4 "C0603X104J5RACTU" H 4175 2925 50  0001 C CNN "manf#"
@@
 F 0 "X2" V 4575 5000 50  0000 C CNN
 F 1 "16M" V 4675 4950 50  0000 L CNN
-F 2 "Crystal:Crystal_SMD_5032-4Pin_5.0x3.2mm" H 4625 4875 60  0001 C CNN
+F 2 "Crystals:Crystal_SMD_5032_4Pads" H 4625 4875 60  0001 C CNN
 F 3 "" H 4625 4875 60  0000 C CNN
 F 4 "ABM3B-16.000MHZ-10-1-U-T" H 4575 5100 50  0001 C CNN "manf#"
@@
 Wire Wire Line
 	3725 2350 3925 2350
+Wire Wire Line
+	4625 4625 4825 4625
+Wire Wire Line
+	4625 5125 4825 5125
+Wire Wire Line
+	5250 5125 5250 5200
+Wire Wire Line
+	3375 2225 3375 2575
+Wire Wire Line
+	4025 2350 4125 2350
+Wire Wire Line
+	4100 4725 4100 4825
+Wire Wire Line
+	3925 2350 4025 2350
+Wire Wire Line
+	4100 5175 4100 5200
+Wire Wire Line
+	5150 3150 5150 3575
+Wire Wire Line
+	5150 2775 5150 2800
+Wire Wire Line
+	3375 3075 3375 3125
+Wire Wire Line
+	5925 4050 6200 4050
+Wire Wire Line
+	5925 3350 6200 3350
+Wire Wire Line
+	6200 4350 6625 4350
+Wire Wire Line
+	6625 4350 6825 4350
+Wire Wire Line
+	7250 3350 8250 3350
+Wire Wire Line
+	4125 2350 4325 2350
+Wire Wire Line
+	4325 2350 4425 2350
 Connection ~ 4625 4625
 Connection ~ 4625 5125
@@
 Connection ~ 4125 2350
 Connection ~ 4325 2350
-Wire Wire Line
-	4625 4625 4825 4625
-Wire Wire Line
-	4625 5125 4825 5125
-Wire Wire Line
-	5250 5125 5250 5200
-Wire Wire Line
-	3375 2225 3375 2575
-Wire Wire Line
-	4025 2350 4125 2350
-Wire Wire Line
-	4100 4725 4100 4825
-Wire Wire Line
-	3925 2350 4025 2350
-Wire Wire Line
-	4100 5175 4100 5200
-Wire Wire Line
-	5150 3150 5150 3575
-Wire Wire Line
-	5150 2775 5150 2800
-Wire Wire Line
-	3375 3075 3375 3125
-Wire Wire Line
-	5925 4050 6200 4050
-Wire Wire Line
-	5925 3350 6200 3350
-Wire Wire Line
-	6200 4350 6625 4350
-Wire Wire Line
-	6625 4350 6825 4350
-Wire Wire Line
-	7250 3350 8250 3350
-Wire Wire Line
-	4125 2350 4325 2350
-Wire Wire Line
-	4325 2350 4425 2350
 $EndSCHEMATC

Commit message: Update part number
Parts:
- C51, C52: manf# 06031A150JAT2A -> 06035A150GAT2A
- C56: manf# GRM1555C2A1R5CA01D -> GRM1555C1H1R5BA01D
- C57: manf# GRM1555C2A1R0CA01D -> GRM1555C1H1R0BA01D
Changed lines of the file:
@@
 F 2 "Capacitors_SMD:C_0603" H 5013 4475 50  0001 C CNN
 F 3 "" H 4975 4625 50  0001 C CNN
-F 4 "06031A150JAT2A" H 5025 4825 50  0001 C CNN "manf#"
+F 4 "06035A150GAT2A" H 5025 4825 50  0001 C CNN "manf#"
 	1    4975 4625
 	0    1    -1   0
@@
 F 2 "Capacitors_SMD:C_0603" H 5013 4975 50  0001 C CNN
 F 3 "" H 4975 5125 50  0001 C CNN
-F 4 "06031A150JAT2A" H 5025 5325 50  0001 C CNN "manf#"
+F 4 "06035A150GAT2A" H 5025 5325 50  0001 C CNN "manf#"
 	1    4975 5125
 	0    1    -1   0
@@
 F 2 "Capacitors_SMD:C_0402" H 7013 3200 50  0001 C CNN
 F 3 "" H 6975 3350 50  0001 C CNN
-F 4 "GRM1555C2A1R5CA01D" H 7225 3375 50  0001 C CNN "manf#"
+F 4 "GRM1555C1H1R5BA01D" H 7225 3375 50  0001 C CNN "manf#"
 	1    6975 3350
 	0    1    -1   0
@@
 F 2 "Capacitors_SMD:C_0402" H 7288 3450 50  0001 C CNN
 F 3 "" H 7250 3600 50  0001 C CNN
-F 4 "GRM1555C2A1R0CA01D" H 7375 3750 50  0001 C CNN "manf#"
+F 4 "GRM1555C1H1R0BA01D" H 7375 3750 50  0001 C CNN "manf#"
 	1    7250 3600
 	1    0    0    -1
