File: design/VESC_6.sch (KiCad schematic (older format))
At the start: 23 parts, among them P1 USB_OTG, P2 CAN, P4 HALL_ENC, P5 COM, P6 SERVO, P7 SWD, U11 SENSOR_VOLTAGE

Commit message: initial commit
Parts:
- C1, C58: footprint CRF1:SMD-0603_c -> Capacitors_SMD:C_0603
- R1, R2, R3, R39, R42, R43, R44, R6, R7, R8, R9: footprint CRF1:SMD-0603_r -> Resistors_SMD:R_0603
