File: design/VESC_6.sch (KiCad schematic (older format))
At the start: 23 parts, among them P1 USB_OTG, P2 CAN, P4 HALL_ENC, P5 COM, P6 SERVO, P7 SWD, U11 SENSOR_VOLTAGE

Commit message: Load KiCad 4.0.7 schematic symbols, footprints & 3D models
Parts:
- C1, C58: footprint Capacitor_SMD:C_0603_1608Metric -> Capacitors_SMD:C_0603
- D1, D2, D3: footprint LED_SMD:LED_0603_1608Metric -> LEDs:LED_0603
- P1: footprint Connector_USB:USB_Micro-B_Molex-105133-0001 -> Connectors_USB:USB_Micro-B_Vertical_Molex-105133-0001
- R1, R2, R3, R39, R42, R43, R44, R6, R7, R8, R9: footprint Resistor_SMD:R_0603_1608Metric -> Resistors_SMD:R_0603
- U11: footprint Button_Switch_SMD:SW_SPDT_PCM12 -> Buttons_Switches_SMD:SW_SPDT_PCM12
Changed lines of the file:
@@
 F 0 "R2" V 3500 1350 40  0000 C CNN
 F 1 "22R" V 3557 1151 40  0000 C CNN
-F 2 "Resistor_SMD:R_0603_1608Metric" V 3480 1150 30  0001 C CNN
+F 2 "Resistors_SMD:R_0603" V 3480 1150 30  0001 C CNN
 F 3 "" H 3550 1150 30  0000 C CNN
 F 4 "CR0603-FX-22R0ELF" H 3500 1450 50  0001 C CNN "manf#"
@@
 F 0 "R3" V 3500 1450 40  0000 C CNN
 F 1 "22R" V 3557 1251 40  0000 C CNN
-F 2 "Resistor_SMD:R_0603_1608Metric" V 3480 1250 30  0001 C CNN
+F 2 "Resistors_SMD:R_0603" V 3480 1250 30  0001 C CNN
 F 3 "" H 3550 1250 30  0000 C CNN
 F 4 "CR0603-FX-22R0ELF" H 3500 1550 50  0001 C CNN "manf#"
@@
 F 0 "D2" H 8225 5425 50  0000 C CNN
 F 1 "RED" H 7750 5425 50  0000 C CNN
-F 2 "LED_SMD:LED_0603_1608Metric" H 8025 5475 60  0001 C CNN
+F 2 "LEDs:LED_0603" H 8025 5475 60  0001 C CNN
 F 3 "" H 8025 5475 60  0001 C CNN
 F 4 "VLMS1300-GS08" H 8225 5525 50  0001 C CNN "manf#"
@@
 F 0 "R8" V 8575 5675 50  0000 C CNN
 F 1 "220R" V 8625 5475 50  0000 C CNN
-F 2 "Resistor_SMD:R_0603_1608Metric" H 8625 5475 60  0001 C CNN
+F 2 "Resistors_SMD:R_0603" H 8625 5475 60  0001 C CNN
 F 3 "" H 8625 5475 60  0001 C CNN
 F 4 "CR0603-FX-2200ELF" H 8575 5775 50  0001 C CNN "manf#"
@@
 F 0 "D3" H 8225 5575 50  0000 C CNN
 F 1 "GREEN" H 7700 5575 50  0000 C CNN
-F 2 "LED_SMD:LED_0603_1608Metric" H 8025 5625 60  0001 C CNN
+F 2 "LEDs:LED_0603" H 8025 5625 60  0001 C CNN
 F 3 "" H 8025 5625 60  0001 C CNN
 F 4 "VLMTG1300-GS08" H 8225 5675 50  0001 C CNN "manf#"
@@
 F 0 "R9" V 8575 5825 50  0000 C CNN
 F 1 "220R" V 8625 5625 50  0000 C CNN
-F 2 "Resistor_SMD:R_0603_1608Metric" H 8625 5625 60  0001 C CNN
+F 2 "Resistors_SMD:R_0603" H 8625 5625 60  0001 C CNN
 F 3 "" H 8625 5625 60  0001 C CNN
 F 4 "CR0603-FX-2200ELF" H 8575 5925 50  0001 C CNN "manf#"
@@
 F 0 "D1" H 8225 5250 50  0000 C CNN
 F 1 "BLUE" H 7725 5250 50  0000 C CNN
-F 2 "LED_SMD:LED_0603_1608Metric" H 8025 5300 60  0001 C CNN
+F 2 "LEDs:LED_0603" H 8025 5300 60  0001 C CNN
 F 3 "" H 8025 5300 60  0001 C CNN
 F 4 "VLMB1300-GS08" H 8225 5350 50  0001 C CNN "manf#"
@@
 F 0 "R7" V 8575 5500 50  0000 C CNN
 F 1 "1k" V 8625 5300 50  0000 C CNN
-F 2 "Resistor_SMD:R_0603_1608Metric" H 8725 5400 60  0001 C CNN
+F 2 "Resistors_SMD:R_0603" H 8725 5400 60  0001 C CNN
 F 3 "" H 8625 5300 60  0001 C CNN
 F 4 "CR0603-FX-1001ELF" H 8575 5600 50  0001 C CNN "manf#"
@@
 F 0 "R44" V 2350 3225 40  0000 C CNN
 F 1 "2k2" V 2407 3026 40  0000 C CNN
-F 2 "Resistor_SMD:R_0603_1608Metric" V 2330 3025 30  0001 C CNN
+F 2 "Resistors_SMD:R_0603" V 2330 3025 30  0001 C CNN
 F 3 "" H 2400 3025 30  0000 C CNN
 F 4 "CR0603-FX-3902ELF" H 2350 3325 50  0001 C CNN "manf#"
@@
 F 0 "R43" V 2350 3125 40  0000 C CNN
 F 1 "2k2" V 2407 2926 40  0000 C CNN
-F 2 "Resistor_SMD:R_0603_1608Metric" V 2330 2925 30  0001 C CNN
+F 2 "Resistors_SMD:R_0603" V 2330 2925 30  0001 C CNN
 F 3 "" H 2400 2925 30  0000 C CNN
 F 4 "CR0603-FX-3902ELF" H 2350 3225 50  0001 C CNN "manf#"
@@
 F 0 "R42" V 2350 3025 40  0000 C CNN
 F 1 "2k2" V 2407 2826 40  0000 C CNN
-F 2 "Resistor_SMD:R_0603_1608Metric" V 2330 2825 30  0001 C CNN
+F 2 "Resistors_SMD:R_0603" V 2330 2825 30  0001 C CNN
 F 3 "" H 2400 2825 30  0000 C CNN
 F 4 "CR0603-FX-3902ELF" H 2350 3125 50  0001 C CNN "manf#"
@@
 F 0 "C58" V 4100 3475 50  0000 L CNN
 F 1 "100n" V 4200 3450 50  0000 L CNN
-F 2 "Capacitor_SMD:C_0603_1608Metric" H 4188 3550 50  0001 C CNN
+F 2 "Capacitors_SMD:C_0603" H 4188 3550 50  0001 C CNN
 F 3 "" H 4150 3700 50  0001 C CNN
 F 4 "C0603X104J5RACTU" H 4100 3575 50  0001 C CNN "manf#"
@@
 F 0 "R39" V 4280 3100 50  0000 C CNN
 F 1 "10k" V 4100 3100 50  0000 C CNN
-F 2 "Resistor_SMD:R_0603_1608Metric" V 4130 3100 50  0001 C CNN
+F 2 "Resistors_SMD:R_0603" V 4130 3100 50  0001 C CNN
 F 3 "" H 4200 3100 50  0001 C CNN
 F 4 "CR0603-FX-1002ELF" H 4280 3200 50  0001 C CNN "manf#"
@@
 F 0 "R6" V 3955 4850 50  0000 C CNN
 F 1 "100R" V 3875 4850 50  0000 C CNN
-F 2 "Resistor_SMD:R_0603_1608Metric" V 3805 4850 50  0001 C CNN
+F 2 "Resistors_SMD:R_0603" V 3805 4850 50  0001 C CNN
 F 3 "" H 3875 4850 50  0001 C CNN
 F 4 "CR0603-FX-1000ELF" H 3955 4950 50  0001 C CNN "manf#"
@@
 F 0 "C1" H 4160 5145 50  0000 L CNN
 F 1 "100n" H 4160 4995 50  0000 L CNN
-F 2 "Capacitor_SMD:C_0603_1608Metric" H 4150 5075 50  0001 C CNN
+F 2 "Capacitors_SMD:C_0603" H 4150 5075 50  0001 C CNN
 F 3 "" H 4150 5075 50  0001 C CNN
 F 4 "C0603X104J5RACTU" H 4160 5245 50  0001 C CNN "manf#"
@@
 F 0 "R1" V 3500 850 50  0000 C CNN
 F 1 "0R" V 3550 1050 50  0000 C CNN
-F 2 "Resistor_SMD:R_0603_1608Metric" H 3550 1050 60  0001 C CNN
+F 2 "Resistors_SMD:R_0603" H 3550 1050 60  0001 C CNN
 F 3 "" H 3550 1050 60  0001 C CNN
 F 4 "CR0603-J/-000EAS" H 3500 950 50  0001 C CNN "manf#"
@@
 F 0 "P1" V 2950 850 50  0000 L CNN
 F 1 "USB_OTG" V 2500 1100 50  0000 L CNN
-F 2 "Connector_USB:USB_Micro-B_Molex-105133-0001" H 2900 1200 50  0001 C CNN
+F 2 "Connectors_USB:USB_Micro-B_Vertical_Molex-105133-0001" H 2900 1200 50  0001 C CNN
 F 3 "" H 2900 1200 50  0001 C CNN
 F 4 "1051330001" H 2950 950 50  0001 C CNN "manf#"
@@
 F 0 "U11" V 1825 2500 50  0000 C CNN
 F 1 "SENSOR_VOLTAGE" H 1750 1925 50  0000 C CNN
-F 2 "Button_Switch_SMD:SW_SPDT_PCM12" H 1745 2200 50  0001 C CNN
+F 2 "Buttons_Switches_SMD:SW_SPDT_PCM12" H 1745 2200 50  0001 C CNN
 F 3 "" H 1745 2200 50  0001 C CNN
 F 4 "PCM12SMTR" H 1825 2600 50  0001 C CNN "manf#"

Commit message: Design VESC6 plus sch done
Parts:
- added C48: 2.2u, Capacitors_SMD:C_0603, symbol Device:C
- added D6: RED, LEDs:LED_0603, symbol Device:LED
- added J1: IO, Pin_Headers:Pin_Header_Straight_1x01, symbol Connector_Generic:Conn_01x01
- added J2: CLK, Pin_Headers:Pin_Header_Straight_1x01, symbol Connector_Generic:Conn_01x01
- added J3: GND, Pin_Headers:Pin_Header_Straight_1x01, symbol Connector_Generic:Conn_01x01
- added J4, J5: HOLE, Pin_Headers:Pin_Header_Straight_1x01, symbol Connector_Generic:Conn_01x01
- added R38, R5: 10k, Resistors_SMD:R_0603, symbol Device:R
- added R4: 1k, Resistors_SMD:R_0603, symbol Device:R
- added U2: NRF51822-TY_EYSGJNZWY, CRF1:Taiyo-Yuden_EYSGJNZWY, symbol crf_1:NRF51822-TY_EYSGJNZWY
Connections:
- wire segments 133 -> 179
- no-connect marks 2 -> 16
Other:
- moved on the sheet: C1, C58, D1, D2, D3, P1, P2, P4, P5, P6, P7, R1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

Commit message: Update footprints
Parts:
- C48: manf# C0603X104J5RACTU -> C1608X5R1C225K080AB
- R38, R5: value 10k -> 1k; manf# CR0603-FX-1002ELF -> CR0603-FX-1001ELF
- R4: manf# CR0603-FX-1000ELF -> CR0603-FX-1001ELF
Changed lines of the file:
@@
 P 8375 4275
 F 0 "R5" V 8410 4080 50  0000 C CNN
-F 1 "10k" V 8375 4275 50  0000 C CNN
+F 1 "1k" V 8375 4275 50  0000 C CNN
 F 2 "Resistors_SMD:R_0603" V 8305 4275 50  0001 C CNN
 F 3 "" H 8375 4275 50  0001 C CNN
-F 4 "CR0603-FX-1002ELF" H 8455 4375 50  0001 C CNN "manf#"
+F 4 "CR0603-FX-1001ELF" H 8455 4375 50  0001 C CNN "manf#"
 	1    8375 4275
 	0    -1   -1   0
@@
 P 8375 4375
 F 0 "R38" V 8410 4180 50  0000 C CNN
-F 1 "10k" V 8375 4375 50  0000 C CNN
+F 1 "1k" V 8375 4375 50  0000 C CNN
 F 2 "Resistors_SMD:R_0603" V 8305 4375 50  0001 C CNN
 F 3 "" H 8375 4375 50  0001 C CNN
-F 4 "CR0603-FX-1002ELF" H 8455 4475 50  0001 C CNN "manf#"
+F 4 "CR0603-FX-1001ELF" H 8455 4475 50  0001 C CNN "manf#"
 	1    8375 4375
 	0    -1   -1   0
@@
 F 2 "Resistors_SMD:R_0603" V 2705 4975 50  0001 C CNN
 F 3 "" H 2775 4975 50  0001 C CNN
-F 4 "CR0603-FX-1000ELF" H 2855 5075 50  0001 C CNN "manf#"
+F 4 "CR0603-FX-1001ELF" H 2855 5075 50  0001 C CNN "manf#"
 	1    2775 4975
 	-1   0    0    1
@@
 F 2 "Capacitors_SMD:C_0603" H 700 5225 50  0001 C CNN
 F 3 "" H 700 5225 50  0001 C CNN
-F 4 "C0603X104J5RACTU" H 710 5395 50  0001 C CNN "manf#"
+F 4 "C1608X5R1C225K080AB" H 710 5395 50  0001 C CNN "manf#"
 	1    700  5225
 	1    0    0    -1

Commit message: Update layout
Parts:
- J1, J2, J3, J4, J5: footprint Pin_Headers:Pin_Header_Straight_1x01 -> CRF1:1PAD
Changed lines of the file:
@@
 F 0 "J5" H 4725 6475 50  0000 C CNN
 F 1 "HOLE" H 4775 6375 50  0000 C CNN
-F 2 "Pin_Headers:Pin_Header_Straight_1x01" H 4625 6425 50  0001 C CNN
+F 2 "CRF1:1PAD" H 4625 6425 50  0001 C CNN
 F 3 "" H 4625 6425 50  0001 C CNN
 F 4 "B1B-PH-K-S (LF)(SN)" H 4625 6725 50  0001 C CNN "manf#"
@@
 F 0 "J4" H 4725 6300 50  0000 C CNN
 F 1 "HOLE" H 4775 6200 50  0000 C CNN
-F 2 "Pin_Headers:Pin_Header_Straight_1x01" H 4625 6250 50  0001 C CNN
+F 2 "CRF1:1PAD" H 4625 6250 50  0001 C CNN
 F 3 "" H 4625 6250 50  0001 C CNN
 F 4 "B1B-PH-K-S (LF)(SN)" H 4625 6550 50  0001 C CNN "manf#"
@@
 F 0 "J1" H 2575 4125 50  0000 C CNN
 F 1 "IO" H 2925 4075 50  0000 C CNN
-F 2 "Pin_Headers:Pin_Header_Straight_1x01" H 2775 4075 50  0001 C CNN
+F 2 "CRF1:1PAD" H 2775 4075 50  0001 C CNN
 F 3 "" H 2775 4075 50  0001 C CNN
 F 4 "B1B-PH-K-S (LF)(SN)" H 2775 4375 50  0001 C CNN "manf#"
@@
 F 0 "J2" H 2575 4025 50  0000 C CNN
 F 1 "CLK" H 2925 3975 50  0000 C CNN
-F 2 "Pin_Headers:Pin_Header_Straight_1x01" H 2775 3975 50  0001 C CNN
+F 2 "CRF1:1PAD" H 2775 3975 50  0001 C CNN
 F 3 "" H 2775 3975 50  0001 C CNN
 F 4 "B1B-PH-K-S (LF)(SN)" H 2775 4275 50  0001 C CNN "manf#"
@@
 F 0 "J3" H 2575 3925 50  0000 C CNN
 F 1 "GND" H 2775 3975 50  0000 C CNN
-F 2 "Pin_Headers:Pin_Header_Straight_1x01" H 2775 3875 50  0001 C CNN
+F 2 "CRF1:1PAD" H 2775 3875 50  0001 C CNN
 F 3 "" H 2775 3875 50  0001 C CNN
 F 4 "B1B-PH-K-S (LF)(SN)" H 2775 4175 50  0001 C CNN "manf#"
