File: design/DRV8301.sch (KiCad schematic (older format))
At the start: 38 parts, among them U2 LM3671, U3 DRV8301

Commit message: initial commit
Parts:
- C13, C14, C15, C16, C17, C18, C19, C20, C22, C23, C24, C25, C28, C31, C64: footprint CRF1:SMD-0603_c -> Capacitors_SMD:C_0603
- R10, R11, R12, R13, R14, R15, R16, R17, R18, R19, R20, R21, R22: footprint CRF1:SMD-0603_r -> Resistors_SMD:R_0603

Commit message: initial commit
Parts:
- C26, C27: footprint w_smd_cap:c_1210 -> Capacitors_SMD:C_1210
Changed lines of the file:
@@
 F 0 "C26" H 6300 5100 50 0000 L CNN
 F 1 "4.7u_100V" H 6300 4900 50 0000 L CNN
-F 2 "w_smd_cap:c_1210" H 6250 5000 60 0001 C CNN
+F 2 "Capacitors_SMD:C_1210" H 6250 5000 60 0001 C CNN
 F 3 "" H 6250 5000 60 0001 C CNN
 	1    6250 5000
@@
 F 0 "C27" H 6625 1850 50 0000 L CNN
 F 1 "4.7u_100V" H 6625 1650 50 0000 L CNN
-F 2 "w_smd_cap:c_1210" H 6575 1750 60 0001 C CNN
+F 2 "Capacitors_SMD:C_1210" H 6575 1750 60 0001 C CNN
 F 3 "" H 6575 1750 60 0001 C CNN
 	1    6575 1750

Commit message: initial commit -m
Parts:
- C21, C32: footprint Capacitors_Tantalum_SMD:CP_Tantalum_Case-B_EIA-3528-21_Wave -> Capacitors_Tantalum_SMD:CP_Tantalum_Case-A_EIA-3216-18_Wave
Changed lines of the file:
@@
 LIBS:valves
 LIBS:crf_1
-LIBS:VESC_6-cache
 EELAYER 25 0
 EELAYER END
@@
 F 0 "C32" H 7650 2825 50  0000 L CNN
 F 1 "100u" H 7650 2625 50  0000 L CNN
-F 2 "Capacitors_Tantalum_SMD:CP_Tantalum_Case-B_EIA-3528-21_Wave" H 7663 2575 50  0001 C CNN
+F 2 "Capacitors_Tantalum_SMD:CP_Tantalum_Case-A_EIA-3216-18_Wave" H 7663 2575 50  0001 C CNN
 F 3 "" H 7625 2725 50  0001 C CNN
 	1    7625 2725
@@
 F 0 "C21" H 4775 6675 50  0000 L CNN
 F 1 "100u" H 4775 6475 50  0000 L CNN
-F 2 "Capacitors_Tantalum_SMD:CP_Tantalum_Case-B_EIA-3528-21_Wave" H 4788 6425 50  0001 C CNN
+F 2 "Capacitors_Tantalum_SMD:CP_Tantalum_Case-A_EIA-3216-18_Wave" H 4788 6425 50  0001 C CNN
 F 3 "" H 4750 6575 50  0001 C CNN
 	1    4750 6575

Commit message: initial commit
Parts:
- L2: footprint w_smd_inductors:inductor_smd_4.8x2.8mm -> CRF1:L_Coilcraft_XAL5050
Changed lines of the file:
@@
 LIBS:valves
 LIBS:crf_1
+LIBS:VESC_6-cache
 EELAYER 25 0
 EELAYER END
@@
 F 0 "L2" V 7050 2525 50  0000 C CNN
 F 1 "22u" V 7175 2525 50  0000 C CNN
-F 2 "w_smd_inductors:inductor_smd_4.8x2.8mm" H 7100 2525 50  0001 C CNN
+F 2 "CRF1:L_Coilcraft_XAL5050" H 7100 2525 50  0001 C CNN
 F 3 "" H 7100 2525 50  0001 C CNN
 	1    7100 2525

Commit message: initial commit
Parts:
- C21, C32: footprint Capacitors_Tantalum_SMD:CP_Tantalum_Case-A_EIA-3216-18_Wave -> Capacitors_Tantalum_SMD:CP_Tantalum_Case-A_EIA-3216-18_Reflow
- D5: footprint w_smd_diode:do214ac -> Diodes_SMD:D_SMA
Changed lines of the file:
@@
 F 0 "C32" H 7650 2825 50  0000 L CNN
 F 1 "100u" H 7650 2625 50  0000 L CNN
-F 2 "Capacitors_Tantalum_SMD:CP_Tantalum_Case-A_EIA-3216-18_Wave" H 7663 2575 50  0001 C CNN
+F 2 "Capacitors_Tantalum_SMD:CP_Tantalum_Case-A_EIA-3216-18_Reflow" H 7663 2575 50  0001 C CNN
 F 3 "" H 7625 2725 50  0001 C CNN
 	1    7625 2725
@@
 F 0 "D5" V 9175 2850 50  0000 L CNN
 F 1 "TVS 5V" V 9275 2850 50  0000 L CNN
-F 2 "w_smd_diode:do214ac" H 9225 2750 50  0001 C CNN
+F 2 "Diodes_SMD:D_SMA" H 9225 2750 50  0001 C CNN
 F 3 "" H 9225 2750 50  0001 C CNN
 	1    9225 2750
@@
 F 0 "C21" H 4775 6675 50  0000 L CNN
 F 1 "100u" H 4775 6475 50  0000 L CNN
-F 2 "Capacitors_Tantalum_SMD:CP_Tantalum_Case-A_EIA-3216-18_Wave" H 4788 6425 50  0001 C CNN
+F 2 "Capacitors_Tantalum_SMD:CP_Tantalum_Case-A_EIA-3216-18_Reflow" H 4788 6425 50  0001 C CNN
 F 3 "" H 4750 6575 50  0001 C CNN
 	1    4750 6575
