File: design/VESC_6.kicad_pcb (KiCad board)
At the start: 4 copper layers, 60 x 60 mm, 303 parts, among them P1 USB_OTG, P10 PH_C, P11 SUPPLY, P12 GND, P2 BATT_-, P2 CAN, P4 HALL_ENC, P5 COM, P6 SERVO, P7 SWD, P8 PH_A, P9 PH_B, Q1 IRF7749, Q2 IRF7749, Q3 IRF7749, Q4 IRF7749, Q5 IRF7749, Q6 IRF7749, U1 STM32F40X_LQFP64, U10 MPU9150, U11 SENSOR_VOLTAGE, U2 LM3671, U3 DRV8301, U4 TJA1051TK3, U5 AD8418, U6 AD8418, U7 AD8418, U8 NRF24L01P, U9 CONN_U_FL, X1 8m, X2 16M

Commit message: initial commit
Parts:
- moved R44 3.28 mm to (125.0, 59.9)
- turned C42 to 270 degrees
- turned U7 to 90 degrees
Routing:
- net Net-(R32-Pad4): track 12.5 -> 53.0 mm, vias 1 -> 2
- net /Power/C_A: track 14.6 -> 53.9 mm
- net /Power/C_B: track 8.80 -> 47.4 mm, vias 1 -> 2
- net Net-(R32-Pad3): track 13.2 -> 50.8 mm, vias 1 -> 2
- net /Power/C_C: track 0.00 -> 35.9 mm, vias 0 -> 2
- net Net-(R29-Pad3): track 10.1 -> 33.1 mm, vias 1 -> 2
- net Net-(R29-Pad4): track 11.2 -> 33.8 mm, vias 1 -> 2
- net VCC: track 129.3 -> 144.9 mm
- net /MCU/H3: track 26.1 -> 27.1 mm

Commit message: initial commit
Routing:
- net /MCU/ADC_TEMP: track 26.8 -> 28.8 mm

Commit message: initial commit
Parts:
- moved C58 2.42 mm to (136.1, 56.1)
- moved R39 2.09 mm to (133.3, 56.1)
- moved D5 0.90 mm to (118.4, 58.3)
- moved R44 0.40 mm to (124.8, 59.6), turned to 180 degrees
- moved R43 0.39 mm to (124.8, 57.9)
- moved R42 0.25 mm to (124.8, 56.3)
Routing:
- net /DRV8301/FAULT: track 45.3 -> 28.9 mm
- net /MCU/TEMP_MOTOR: track 1.96 -> 5.25 mm
- net /MCU/ADC_TEMP: track 28.8 -> 27.0 mm

Commit message: initial commit
Parts:
- moved C42 3.94 mm to (125.5, 65.2)
- moved U7 3.94 mm to (128.1, 65.2)
- moved C38 3.43 mm to (130.9, 63.7)
- moved U6 3.43 mm to (133.5, 63.7)
- moved C35 1.85 mm to (136.0, 67.7)
- moved P6 1.65 mm to (118.0, 104.0)
- moved R23 1.65 mm to (120.3, 108.2)
- moved P2 1.65 mm to (120.3, 110.4)
Routing:
- net GND: track 111.7 -> 151.5 mm, vias 128 -> 134
- net +5V: track 46.6 -> 58.0 mm
- net /Power/C_C: track 35.9 -> 42.6 mm
- net (no net): track 4.67 -> 0.00 mm, vias 1 -> 0
- net Net-(R29-Pad3): track 33.1 -> 29.4 mm
- net Net-(R32-Pad4): track 53.0 -> 49.4 mm
- net Net-(R32-Pad3): track 50.8 -> 47.3 mm
- net VCC: track 144.9 -> 148.1 mm, vias 8 -> 9
- net Net-(R29-Pad4): track 33.8 -> 30.7 mm
- net /Power/C_B: track 47.5 -> 49.7 mm
- net /MCU/TEMP_MOTOR: track 5.25 -> 3.29 mm, vias 1 -> 0
- net Net-(P6-Pad3): track 7.98 -> 6.02 mm
- net /MCU/HALL_3: track 1.75 -> 0.00 mm, vias 1 -> 0
- net /MCU/HALL_2: track 1.53 -> 0.00 mm, vias 1 -> 0
- net /MCU/HALL_1: track 1.37 -> 0.00 mm, vias 1 -> 0
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
Commit message: initial commit
Routing:
- net /MCU/HALL_3: track 0.00 -> 61.7 mm, vias 0 -> 1
- net /MCU/HALL_2: track 0.00 -> 60.1 mm, vias 0 -> 1
- net /MCU/HALL_1: track 0.00 -> 58.8 mm, vias 0 -> 1
- net /MCU/CAN_RX: track 29.4 -> 28.6 mm
- net /DRV8301/INL_B: track 29.6 -> 29.0 mm
- added copper zone on GND.Cu, net GND
- added copper zone on PWR.Cu, net VCC

Commit message: initial commit
Parts:
- moved C52 0.40 mm to (137.9, 108.1)
Routing:
- net +5V: track 58.4 -> 84.1 mm
- net GND: track 151.5 -> 174.3 mm, vias 134 -> 144
- net Net-(C52-Pad2): track 7.45 -> 10.4 mm
- net /MCU/TEMP_MOTOR: track 3.29 -> 5.01 mm, vias 0 -> 1
- net VCC: track 148.2 -> 149.4 mm, vias 9 -> 10

Commit message: initial commit
Routing:
- net GND: track 174.3 -> 180.1 mm, vias 144 -> 149
Changed lines of the file:
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@@
   (general
     (links 607)
-    (no_connects 62)
+    (no_connects 61)
     (area 114.924999 54.924999 175.075001 115.075001)
     (thickness 1.6)
     (drawings 47)
-    (tracks 1714)
+    (tracks 1731)
     (zones 0)
     (modules 303)
@@
   )
   (setup
-    (last_trace_width 0.35052)
+    (last_trace_width 0.2032)
     (user_trace_width 0.2032)
     (user_trace_width 0.254)
@@
   (segment (start 137.194999 92.213999) (end 138.237409 92.213999) (width 0.2032) (layer F.Cu) (net 1) (status 10))
   (via (at 138.581702 92.558292) (size 0.6) (drill 0.3) (layers F.Cu B.Cu) (net 1))
+  (segment (start 132.328883 106.68) (end 131.445 105.796117) (width 0.2032) (layer F.Cu) (net 2))
+  (segment (start 131.445 107.563883) (end 132.328883 106.68) (width 0.2032) (layer F.Cu) (net 2))
+  (via (at 132.328883 106.68) (size 0.6) (drill 0.3) (layers F.Cu B.Cu) (net 2))
+  (segment (start 130.561117 106.68) (end 131.445 107.563883) (width 0.2032) (layer F.Cu) (net 2))
+  (via (at 131.445 107.563883) (size 0.6) (drill 0.3) (layers F.Cu B.Cu) (net 2))
+  (segment (start 131.445 105.796117) (end 130.561117 106.68) (width 0.2032) (layer F.Cu) (net 2))
+  (via (at 130.561117 106.68) (size 0.6) (drill 0.3) (layers F.Cu B.Cu) (net 2))
+  (segment (start 132.127358 104.583428) (end 131.445 105.265786) (width 0.2032) (layer F.Cu) (net 2))
+  (segment (start 131.445 105.265786) (end 131.445 105.796117) (width 0.2032) (layer F.Cu) (net 2))
+  (via (at 131.445 105.796117) (size 0.6) (drill 0.3) (layers F.Cu B.Cu) (net 2))
+  (segment (start 132.127358 104.583428) (end 132.127358 103.776187) (width 0.2032) (layer F.Cu) (net 2))
+  (segment (start 132.127358 103.776187) (end 132.127284 103.776113) (width 0.2032) (layer F.Cu) (net 2))
+  (via (at 132.127284 103.776113) (size 0.6) (drill 0.3) (layers F.Cu B.Cu) (net 2))
   (segment (start 134.220485 107.795458) (end 134.750814 108.325787) (width 0.35052) (layer B.Cu) (net 2))
   (segment (start 134.750814 108.325787) (end 135.387213 108.325787) (width 0.35052) (layer B.Cu) (net 2))
@@
   (segment (start 124.321 82.042) (end 124.321 82.973) (width 0.508) (layer B.Cu) (net 2) (status 30))
   (segment (start 124.321 82.973) (end 124.875 83.527) (width 0.508) (layer B.Cu) (net 2) (status 30))
-  (segment (start 131.445 105.796117) (end 131.445 105.265786) (width 0.2032) (layer F.Cu) (net 2) (status 30))
-  (segment (start 131.445 105.265786) (end 132.127358 104.583428) (width 0.2032) (layer F.Cu) (net 2) (status 30))
   (segment (start 132.328883 106.68) (end 132.328883 106.503224) (width 0.2032) (layer F.Cu) (net 2) (status 30))
   (segment (start 132.328883 106.503224) (end 133.188018 105.644089) (width 0.2032) (layer F.Cu) (net 2) (status 30))
@@
   (segment (start 134.62 100.2665) (end 134.695001 100.191499) (width 0.2032) (layer F.Cu) (net 5) (status 30))
   (segment (start 134.695001 100.191499) (end 134.695001 98.713999) (width 0.2032) (layer F.Cu) (net 5) (status 30))
-  (segment (start 128.016 106.807) (end 129.921 104.902) (width 0.2032) (layer B.Cu) (net 6))
-  (segment (start 129.921 104.902) (end 129.921 104.267) (width 0.2032) (layer B.Cu) (net 6))
+  (segment (start 132.2 102.524264) (end 132.2 102.1) (width 0.2032) (layer B.Cu) (net 6))
+  (segment (start 132.2 102.877) (end 132.2 102.524264) (width 0.2032) (layer B.Cu) (net 6))
   (segment (start 130.429 103.759) (end 131.318 103.759) (width 0.2032) (layer B.Cu) (net 6))
   (segment (start 129.921 104.267) (end 130.429 103.759) (width 0.2032) (layer B.Cu) (net 6))
-  (segment (start 131.318 103.759) (end 132.1 102.977) (width 0.2032) (layer B.Cu) (net 6))
-  (segment (start 132.1 102.2) (end 132.2 102.1) (width 0.2032) (layer B.Cu) (net 6))
-  (segment (start 132.1 102.977) (end 132.1 102.2) (width 0.2032) (layer B.Cu) (net 6))
+  (segment (start 129.921 104.902) (end 129.921 104.267) (width 0.2032) (layer B.Cu) (net 6))
+  (segment (start 128.016 106.807) (end 129.921 104.902) (width 0.2032) (layer B.Cu) (net 6))
+  (segment (start 131.318 103.759) (end 132.2 102.877) (width 0.2032) (layer B.Cu) (net 6))
   (segment (start 125.695001 90.214) (end 126.829 90.214) (width 0.2032) (layer F.Cu) (net 6))
   (segment (start 126.829 90.214) (end 126.873 90.17) (width 0.2032) (layer F.Cu) (net 6))
@@
   (segment (start 138.291353 94.713999) (end 138.556532 94.44882) (width 0.2032) (layer F.Cu) (net 97))
   (via (at 138.556532 94.44882) (size 0.6) (drill 0.3) (layers F.Cu B.Cu) (net 97))
-  (segment (start 124.159997 104.313003) (end 124.159997 105.110001) (width 0.2032) (layer PWR.Cu) (net 98))
-  (segment (start 134.091183 102.869989) (end 125.603011 102.869989) (width 0.2032) (layer PWR.Cu) (net 98))
-  (segment (start 136.779 100.182172) (end 134.091183 102.869989) (width 0.2032) (layer PWR.Cu) (net 98))
   (segment (start 125.603011 102.869989) (end 124.159997 104.313003) (width 0.2032) (layer PWR.Cu) (net 98))
-  (segment (start 124.159997 105.110001) (end 124.459996 105.41) (width 0.2032) (layer PWR.Cu) (net 98))
+  (segment (start 134.162584 102.798588) (end 131.644068 102.798588) (width 0.2032) (layer PWR.Cu) (net 98))
+  (segment (start 131.572667 102.869989) (end 125.603011 102.869989) (width 0.2032) (layer PWR.Cu) (net 98))
+  (segment (start 124.159997 104.313003) (end 124.159997 105.110001) (width 0.2032) (layer PWR.Cu) (net 98))
   (segment (start 136.779 94.487988) (end 136.779 100.182172) (width 0.2032) (layer PWR.Cu) (net 98))
+  (segment (start 131.644068 102.798588) (end 131.572667 102.869989) (width 0.2032) (layer PWR.Cu) (net 98))
+  (segment (start 136.779 100.182172) (end 134.162584 102.798588) (width 0.2032) (layer PWR.Cu) (net 98))
   (segment (start 135.128 92.836988) (end 136.779 94.487988) (width 0.2032) (layer PWR.Cu) (net 98))
+  (segment (start 124.159997 105.110001) (end 124.459996 105.41) (width 0.2032) (layer PWR.Cu) (net 98))
   (segment (start 125.047638 105.997642) (end 124.459996 105.41) (width 0.2032) (layer F.Cu) (net 98))
   (segment (start 129.348428 105.997642) (end 125.047638 105.997642) (width 0.2032) (layer F.Cu) (net 98) (status 10))
@@
   (segment (start 137.194999 94.214) (end 136.080748 94.214) (width 0.2032) (layer F.Cu) (net 98) (status 10))
   (via (at 135.128 92.836988) (size 0.6) (drill 0.3) (layers F.Cu B.Cu) (net 98))
-  (segment (start 134.249002 103.251) (end 125.940736 103.251) (width 0.2032) (layer PWR.Cu) (net 99))
+  (segment (start 131.730486 103.251) (end 125.940736 103.251) (width 0.2032) (layer PWR.Cu) (net 99))
+  (segment (start 134.320403 103.179599) (end 131.801887 103.179599) (width 0.2032) (layer PWR.Cu) (net 99))
+  (segment (start 125.009996 104.43574) (end 125.009996 104.860004) (width 0.2032) (layer PWR.Cu) (net 99))
+  (segment (start 125.940736 103.251) (end 125.009996 104.18174) (width 0.2032) (layer PWR.Cu) (net 99))
+  (segment (start 131.801887 103.179599) (end 131.730486 103.251) (width 0.2032) (layer PWR.Cu) (net 99))
+  (segment (start 137.160011 100.339991) (end 134.320403 103.179599) (width 0.2032) (layer PWR.Cu) (net 99))
   (segment (start 135.130017 91.805191) (end 137.160011 93.835185) (width 0.2032) (layer PWR.Cu) (net 99))
   (segment (start 137.160011 93.835185) (end 137.160011 100.339991) (width 0.2032) (layer PWR.Cu) (net 99))
-  (segment (start 125.940736 103.251) (end 125.009996 104.18174) (width 0.2032) (layer PWR.Cu) (net 99))
-  (segment (start 137.160011 100.339991) (end 134.249002 103.251) (width 0.2032) (layer PWR.Cu) (net 99))
-  (segment (start 125.009996 104.18174) (end 125.009996 104.860004) (width 0.2032) (layer PWR.Cu) (net 99))
+  (segment (start 125.009996 104.18174) (end 125.009996 104.43574) (width 0.2032) (layer PWR.Cu) (net 99))
   (segment (start 125.250393 105.100401) (end 125.009996 104.860004) (width 0.2032) (layer F.Cu) (net 99))
   (segment (start 129.158294 105.100401) (end 125.250393 105.100401) (width 0.2032) (layer F.Cu) (net 99))
@@
   (segment (start 135.207707 91.805191) (end 135.130017 91.805191) (width 0.2032) (layer F.Cu) (net 99))
   (via (at 135.130017 91.805191) (size 0.6) (drill 0.3) (layers F.Cu B.Cu) (net 99))
-  (segment (start 133.644832 104.394) (end 125.73 104.394) (width 0.2032) (layer PWR.Cu) (net 100))
-  (segment (start 137.541022 100.49781) (end 133.644832 104.394) (width 0.2032) (layer PWR.Cu) (net 100))
   (segment (start 136 91.7) (end 137.541022 93.241022) (width 0.2032) (layer PWR.Cu) (net 100))
+  (segment (start 133.344833 104.693999) (end 126.029999 104.693999) (width 0.2032) (layer PWR.Cu) (net 100))
   (segment (start 137.541022 93.241022) (end 137.541022 100.49781) (width 0.2032) (layer PWR.Cu) (net 100))
+  (segment (start 126.029999 104.693999) (end 125.73 104.394) (width 0.2032) (layer PWR.Cu) (net 100))
+  (segment (start 137.541022 100.49781) (end 133.344833 104.693999) (width 0.2032) (layer PWR.Cu) (net 100))
   (segment (start 129.159 104.394) (end 125.73 104.394) (width 0.2032) (layer F.Cu) (net 100))
   (segment (start 130.055535 105.290535) (end 129.159 104.394) (width 0.2032) (layer F.Cu) (net 100) (status 10))

Commit message: initial commit
Routing:
- net GND: track 180.1 -> 195.1 mm, vias 149 -> 153
- net VCC: track 149.4 -> 152.4 mm, vias 10 -> 11
- net +5V: track 84.1 -> 84.7 mm
