File: design/VESC_6.kicad_pcb (KiCad board)
At the start: 4 copper layers, 60 x 60 mm, 303 parts, among them P1 USB_OTG, P10 PH_C, P11 SUPPLY, P12 GND, P2 BATT_-, P2 CAN, P4 HALL_ENC, P5 COM, P6 SERVO, P7 SWD, P8 PH_A, P9 PH_B, Q1 IRF7749, Q2 IRF7749, Q3 IRF7749, Q4 IRF7749, Q5 IRF7749, Q6 IRF7749, U1 STM32F40X_LQFP64, U10 MPU9150, U11 SENSOR_VOLTAGE, U2 LM3671, U3 DRV8301, U4 TJA1051TK3, U5 AD8418, U6 AD8418, U7 AD8418, U8 NRF24L01P, U9 CONN_U_FL, X1 8m, X2 16M

Commit message: initial commit
Routing:
- net +5V: track 84.7 -> 101.7 mm, vias 0 -> 2
- net VCC: track 152.4 -> 164.8 mm, vias 11 -> 12
- net Net-(R10-Pad2): track 1.09 -> 12.8 mm, vias 0 -> 2
- net GND: track 195.1 -> 204.8 mm, vias 153 -> 157
- net /MCU/HALL_1: track 58.8 -> 60.4 mm
- net /Power/C_A: track 54.1 -> 55.2 mm
- net /Power/C_C: track 42.6 -> 43.7 mm

Commit message: initial commit
Routing:
- net /MCU/RX_SDA_NSS: track 12.0 -> 15.2 mm
- net GND: track 204.8 -> 207.5 mm, vias 157 -> 158

Commit message: initial commit
Parts:
- moved R42 1.02 mm to (123.8, 56.3)
- moved R43 1.02 mm to (123.8, 57.9)
- moved R44 1.02 mm to (123.8, 59.6)
- moved U11 0.82 mm to (120.4, 59.8)
- moved D5 0.63 mm to (118.4, 58.9)
Routing:
- net GND: track 207.5 -> 236.8 mm, vias 158 -> 169
- net +5V: track 101.7 -> 128.1 mm, vias 2 -> 4
- net VCC: track 164.7 -> 159.1 mm, vias 12 -> 11
- net /Power/C_A: track 55.1 -> 50.9 mm
- net Net-(P4-Pad6): track 0.00 -> 3.26 mm
- net /Power/C_C: track 43.7 -> 45.9 mm
- net /MCU/HALL_3: track 62.0 -> 62.9 mm
- net Net-(Q2-PadG): track 11.2 -> 12.0 mm

Commit message: initial commit
Routing:
- net GND: track 236.8 -> 257.2 mm, vias 169 -> 170
- net +5V: track 128.1 -> 144.0 mm
- net /MCU/RX_SDA_NSS: track 15.2 -> 22.3 mm
- net /MPU9150/SCL: track 20.4 -> 25.0 mm
- net VCC: track 159.1 -> 162.4 mm

Commit message: initial commit
Routing:
- net /MCU/TEMP_MOTOR: track 5.01 -> 56.7 mm, vias 1 -> 2
- net VCC: track 162.4 -> 193.4 mm, vias 11 -> 12
- net GND: track 257.2 -> 281.9 mm, vias 170 -> 171
- net /MCU/HALL_1: track 59.8 -> 70.9 mm
- net /MCU/HALL_2: track 60.6 -> 69.9 mm
- net /MCU/HALL_3: track 62.9 -> 69.2 mm
- net /Power/C_C: track 45.9 -> 44.8 mm
- net /Power/C_B: track 50.1 -> 49.4 mm

Commit message: initial commit
Routing:
- net Net-(P4-Pad6): track 3.26 -> 25.1 mm, vias 0 -> 1
- net /DRV8301/SH_A: track 13.2 -> 29.6 mm
- net /DRV8301/SH_B: track 24.8 -> 40.9 mm
- net VCC: track 193.4 -> 202.0 mm
- net GND: track 281.9 -> 289.8 mm, vias 171 -> 173
- net /DRV8301/SH_C: track 64.3 -> 68.7 mm
- net SUPPLY: track 43.3 -> 45.5 mm
- net Net-(C56-Pad1): track 0.00 -> 2.07 mm
- net +5V: track 144.0 -> 145.7 mm
- net Net-(C20-Pad1): track 2.73 -> 4.22 mm
- net Net-(C28-Pad2): track 19.2 -> 20.4 mm
- net /MPU9150/SCL: track 25.0 -> 26.0 mm

Commit message: initial commit
Routing:
- net VCC: track 202.0 -> 225.2 mm
- net /MCU/H3: track 27.1 -> 26.2 mm
- net /MCU/H2: track 26.1 -> 25.4 mm
- net /DRV8301/INL_A: track 25.6 -> 26.3 mm

Commit message: initial commit
Routing:
- net /Power/C_B: track 49.4 -> 47.4 mm
- net /MCU/TEMP_MOTOR: track 56.7 -> 54.9 mm
- net GND: track 290.0 -> 291.3 mm
- net /Power/C_C: track 44.8 -> 43.7 mm
