File: design/Power.sch (KiCad schematic (older format))
At the start: 43 parts, among them P10 PH_C, P11 SUPPLY, P12 GND, P8 PH_A, P9 PH_B, Q1 IRF7749, Q2 IRF7749, Q3 IRF7749, Q4 IRF7749, Q5 IRF7749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

Commit message: initial commit
Parts:
- C29, C30, C35, C36, C38, C42, C45: footprint CRF1:SMD-0603_c -> Capacitors_SMD:C_0603
- R25, R26, R27, R28, R30, R31, R33, R34, R35, R36, R37: footprint CRF1:SMD-0603_r -> Capacitors_SMD:C_0603

Commit message: initial commit
Parts:
- C37, C39, C40, C41, C43, C44: footprint w_smd_cap:c_1210 -> Capacitors_SMD:C_1210
Changed lines of the file:
@@
 F 0 "C37" V 3800 2475 50 0000 C TNN
 F 1 "4.7u_100V" V 3800 2850 50 0000 C TNN
-F 2 "w_smd_cap:c_1210" H 3913 2450 50 0001 C CNN
+F 2 "Capacitors_SMD:C_1210" H 3913 2450 50 0001 C CNN
 F 3 "" H 3875 2600 50 0001 C CNN
 	1    3875 2600
@@
 F 0 "C39" V 4000 2475 50 0000 C TNN
 F 1 "4.7u_100V" V 4000 2850 50 0000 C TNN
-F 2 "w_smd_cap:c_1210" H 4113 2450 50 0001 C CNN
+F 2 "Capacitors_SMD:C_1210" H 4113 2450 50 0001 C CNN
 F 3 "" H 4075 2600 50 0001 C CNN
 	1    4075 2600
@@
 F 0 "C41" V 7150 2475 50 0000 C TNN
 F 1 "4.7u_100V" V 7150 2850 50 0000 C TNN
-F 2 "w_smd_cap:c_1210" H 7263 2450 50 0001 C CNN
+F 2 "Capacitors_SMD:C_1210" H 7263 2450 50 0001 C CNN
 F 3 "" H 7225 2600 50 0001 C CNN
 	1    7225 2600
@@
 F 0 "C40" V 7350 2475 50 0000 C TNN
 F 1 "4.7u_100V" V 7350 2850 50 0000 C TNN
-F 2 "w_smd_cap:c_1210" H 7463 2450 50 0001 C CNN
+F 2 "Capacitors_SMD:C_1210" H 7463 2450 50 0001 C CNN
 F 3 "" H 7425 2600 50 0001 C CNN
 	1    7425 2600
@@
 F 0 "C43" V 10475 2475 50 0000 C TNN
 F 1 "4.7u_100V" V 10475 2850 50 0000 C TNN
-F 2 "w_smd_cap:c_1210" H 10588 2450 50 0001 C CNN
+F 2 "Capacitors_SMD:C_1210" H 10588 2450 50 0001 C CNN
 F 3 "" H 10550 2600 50 0001 C CNN
 	1    10550 2600
@@
 F 0 "C44" V 10675 2475 50 0000 C TNN
 F 1 "4.7u_100V" V 10675 2850 50 0000 C TNN
-F 2 "w_smd_cap:c_1210" H 10788 2450 50 0001 C CNN
+F 2 "Capacitors_SMD:C_1210" H 10788 2450 50 0001 C CNN
 F 3 "" H 10750 2600 50 0001 C CNN
 	1    10750 2600

Commit message: initial commit
Parts:
- R25, R26, R27, R28, R30, R31, R33, R34, R35, R36, R37: footprint Capacitors_SMD:C_0603 -> Resistors_SMD:R_0603
Changed lines of the file:
@@
 F 0 "R26" V 3000 3200 50  0000 C CNN
 F 1 "4.7R" V 2900 3200 50  0000 C CNN
-F 2 "Capacitors_SMD:C_0603" H 2900 3200 60  0001 C CNN
+F 2 "Resistors_SMD:R_0603" H 2900 3200 60  0001 C CNN
 F 3 "" H 2900 3200 60  0001 C CNN
 	1    2900 3200
@@
 F 0 "R25" V 3000 2100 50  0000 C CNN
 F 1 "4.7R" V 2900 2100 50  0000 C CNN
-F 2 "Capacitors_SMD:C_0603" H 2900 2100 60  0001 C CNN
+F 2 "Resistors_SMD:R_0603" H 2900 2100 60  0001 C CNN
 F 3 "" H 2900 2100 60  0001 C CNN
 	1    2900 2100
@@
 F 0 "R35" V 1975 5175 50  0000 C CNN
 F 1 "100R" V 1775 5175 50  0000 C CNN
-F 2 "Capacitors_SMD:C_0603" H 1875 5175 60  0001 C CNN
+F 2 "Resistors_SMD:R_0603" H 1875 5175 60  0001 C CNN
 F 3 "" H 1875 5175 60  0001 C CNN
 	1    1875 5175
@@
 F 0 "R31" V 6350 3200 50  0000 C CNN
 F 1 "4.7R" V 6250 3200 50  0000 C CNN
-F 2 "Capacitors_SMD:C_0603" H 6250 3200 60  0001 C CNN
+F 2 "Resistors_SMD:R_0603" H 6250 3200 60  0001 C CNN
 F 3 "" H 6250 3200 60  0001 C CNN
 	1    6250 3200
@@
 F 0 "R30" V 6350 2100 50  0000 C CNN
 F 1 "4.7R" V 6250 2100 50  0000 C CNN
-F 2 "Capacitors_SMD:C_0603" H 6250 2100 60  0001 C CNN
+F 2 "Resistors_SMD:R_0603" H 6250 2100 60  0001 C CNN
 F 3 "" H 6250 2100 60  0001 C CNN
 	1    6250 2100
@@
 F 0 "R34" V 9675 3200 50  0000 C CNN
 F 1 "4.7R" V 9575 3200 50  0000 C CNN
-F 2 "Capacitors_SMD:C_0603" H 9575 3200 60  0001 C CNN
+F 2 "Resistors_SMD:R_0603" H 9575 3200 60  0001 C CNN
 F 3 "" H 9575 3200 60  0001 C CNN
 	1    9575 3200
@@
 F 0 "R33" V 9675 2100 50  0000 C CNN
 F 1 "4.7R" V 9575 2100 50  0000 C CNN
-F 2 "Capacitors_SMD:C_0603" H 9575 2100 60  0001 C CNN
+F 2 "Resistors_SMD:R_0603" H 9575 2100 60  0001 C CNN
 F 3 "" H 9575 2100 60  0001 C CNN
 	1    9575 2100
@@
 F 0 "R36" V 1975 5950 50  0000 C CNN
 F 1 "100R" V 1775 5950 50  0000 C CNN
-F 2 "Capacitors_SMD:C_0603" H 1875 5950 60  0001 C CNN
+F 2 "Resistors_SMD:R_0603" H 1875 5950 60  0001 C CNN
 F 3 "" H 1875 5950 60  0001 C CNN
 	1    1875 5950
@@
 F 0 "R37" V 1975 6725 50  0000 C CNN
 F 1 "100R" V 1775 6725 50  0000 C CNN
-F 2 "Capacitors_SMD:C_0603" H 1875 6725 60  0001 C CNN
+F 2 "Resistors_SMD:R_0603" H 1875 6725 60  0001 C CNN
 F 3 "" H 1875 6725 60  0001 C CNN
 	1    1875 6725
@@
 F 0 "R27" V 4030 5825 40  0000 C CNN
 F 1 "NTC 10k" V 3850 5826 40  0000 C CNN
-F 2 "Capacitors_SMD:C_0603" V 3880 5825 30  0001 C CNN
+F 2 "Resistors_SMD:R_0603" V 3880 5825 30  0001 C CNN
 F 3 "" H 3950 5825 30  0000 C CNN
 	1    3950 5825
@@
 F 0 "R28" V 4030 6525 40  0000 C CNN
 F 1 "10k" V 3850 6526 40  0000 C CNN
-F 2 "Capacitors_SMD:C_0603" V 3880 6525 30  0001 C CNN
+F 2 "Resistors_SMD:R_0603" V 3880 6525 30  0001 C CNN
 F 3 "" H 3950 6525 30  0000 C CNN
 	1    3950 6525

Commit message: initial commit
Parts:
- P11, P12: footprint CRF1:1PAD_6x5mm -> CRF1:1PAD_7x6mm
Changed lines of the file:
@@
 F 0 "P12" H 10600 4300 50  0000 C CNN
 F 1 "GND" H 10600 4100 50  0000 C CNN
-F 2 "CRF1:1PAD_6x5mm" H 10600 4200 50  0001 C CNN
+F 2 "CRF1:1PAD_7x6mm" H 10600 4200 50  0001 C CNN
 F 3 "" H 10600 4200 50  0001 C CNN
 	1    10600 4200
@@
 F 0 "P11" H 10600 1550 50  0000 C CNN
 F 1 "SUPPLY" H 10600 1350 50  0000 C CNN
-F 2 "CRF1:1PAD_6x5mm" H 10600 1450 50  0001 C CNN
+F 2 "CRF1:1PAD_7x6mm" H 10600 1450 50  0001 C CNN
 F 3 "" H 10600 1450 50  0001 C CNN
 	1    10600 1450

Commit message: initial commit
Parts:
- C46, C47: footprint Capacitors_THT:CP_Radial_D12.5mm_P5.00mm -> CRF1:CP_Radial_D12.5mm_P5.00mm
Changed lines of the file:
@@
 F 0 "C46" H 8850 5375 50  0000 L CNN
 F 1 "680u_63V" H 8850 5300 50  0000 L CNN
-F 2 "Capacitors_THT:CP_Radial_D12.5mm_P5.00mm" H 8750 5325 50  0001 C CNN
+F 2 "CRF1:CP_Radial_D12.5mm_P5.00mm" H 8750 5325 50  0001 C CNN
 F 3 "" H 8750 5325 50  0001 C CNN
 	1    8750 5325
@@
 F 0 "C47" H 9450 5375 50  0000 L CNN
 F 1 "680u_63V" H 9450 5300 50  0000 L CNN
-F 2 "Capacitors_THT:CP_Radial_D12.5mm_P5.00mm" H 9350 5325 50  0001 C CNN
+F 2 "CRF1:CP_Radial_D12.5mm_P5.00mm" H 9350 5325 50  0001 C CNN
 F 3 "" H 9350 5325 50  0001 C CNN
 	1    9350 5325

Commit message: Prepare version 1.0
Parts:
- P11, P12: footprint CRF1:1PAD_7x6mm -> CRF1:1PAD_6x5mm
Changed lines of the file:
@@
 F 0 "P12" H 10600 4300 50  0000 C CNN
 F 1 "GND" H 10600 4100 50  0000 C CNN
-F 2 "CRF1:1PAD_7x6mm" H 10600 4200 50  0001 C CNN
+F 2 "CRF1:1PAD_6x5mm" H 10600 4200 50  0001 C CNN
 F 3 "" H 10600 4200 50  0001 C CNN
 	1    10600 4200
@@
 F 0 "P11" H 10600 1550 50  0000 C CNN
 F 1 "SUPPLY" H 10600 1350 50  0000 C CNN
-F 2 "CRF1:1PAD_7x6mm" H 10600 1450 50  0001 C CNN
+F 2 "CRF1:1PAD_6x5mm" H 10600 1450 50  0001 C CNN
 F 3 "" H 10600 1450 50  0001 C CNN
 	1    10600 1450
