File: design/Power.sch (KiCad schematic (older format))
At the start: 49 parts, among them P10 PH_C, P11 SUPPLY, P12 GND, P8 PH_A, P9 PH_B, Q1 IRF7749, Q2 IRF7749, Q3 IRF7749, Q4 IRF7749, Q5 IRF7749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

Commit message: assign component footprint
Parts:
- U10, U12, U13: footprint TO_SOT_Packages_SMD:SOT-353 -> TO_SOT_Packages_SMD:SOT-23-5
Changed lines of the file:
@@
 F 0 "U10" H 1850 5200 50  0000 C CNN
 F 1 "MC74VHC1GT66" H 2325 5484 50  0000 C CNN
-F 2 "TO_SOT_Packages_SMD:SOT-353" H 2375 4850 50  0001 C CNN
+F 2 "TO_SOT_Packages_SMD:SOT-23-5" H 2375 4850 50  0001 C CNN
 F 3 "" H 2975 4500 50  0001 C CNN
 	1    2325 5200
@@
 F 0 "U12" H 4525 5200 50  0000 C CNN
 F 1 "MC74VHC1GT66" H 5000 5484 50  0000 C CNN
-F 2 "TO_SOT_Packages_SMD:SOT-353" H 5050 4850 50  0001 C CNN
+F 2 "TO_SOT_Packages_SMD:SOT-23-5" H 5050 4850 50  0001 C CNN
 F 3 "" H 5650 4500 50  0001 C CNN
 	1    5000 5200
@@
 F 0 "U13" H 7525 5225 50  0000 C CNN
 F 1 "MC74VHC1GT66" H 8000 5509 50  0000 C CNN
-F 2 "TO_SOT_Packages_SMD:SOT-353" H 8050 4875 50  0001 C CNN
+F 2 "TO_SOT_Packages_SMD:SOT-23-5" H 8050 4875 50  0001 C CNN
 F 3 "" H 8650 4525 50  0001 C CNN
 	1    8000 5225

Commit message: Update footprints
Parts:
- C52, C53, C54: manf# GRM188R71H472JA01J -> GCM188R71H153KA37D
- R35, R36, R37: manf# CR0603-FX-1000ELF -> CR0603-FX-1001ELF
Changed lines of the file:
@@
 F 2 "Resistors_SMD:R_0603" H 3350 4775 60  0001 C CNN
 F 3 "" H 3350 4775 60  0001 C CNN
-F 4 "CR0603-FX-1000ELF" H 3450 4875 50  0001 C CNN "manf#"
+F 4 "CR0603-FX-1001ELF" H 3450 4875 50  0001 C CNN "manf#"
 	1    3350 4775
 	0    1    -1   0
@@
 F 2 "Capacitors_SMD:C_0603" H 2988 5375 50  0001 C CNN
 F 3 "" H 2950 5425 50  0001 C CNN
-F 4 "GRM188R71H472JA01J" H 3050 5560 50  0001 C CNN "manf#"
+F 4 "GCM188R71H153KA37D" H 3050 5560 50  0001 C CNN "manf#"
 	1    2950 5425
 	1    0    0    -1
@@
 F 2 "Resistors_SMD:R_0603" H 6025 4775 60  0001 C CNN
 F 3 "" H 6025 4775 60  0001 C CNN
-F 4 "CR0603-FX-1000ELF" H 6125 4875 50  0001 C CNN "manf#"
+F 4 "CR0603-FX-1001ELF" H 6125 4875 50  0001 C CNN "manf#"
 	1    6025 4775
 	0    1    -1   0
@@
 F 2 "Capacitors_SMD:C_0603" H 5663 5375 50  0001 C CNN
 F 3 "" H 5625 5425 50  0001 C CNN
-F 4 "GRM188R71H472JA01J" H 5725 5560 50  0001 C CNN "manf#"
+F 4 "GCM188R71H153KA37D" H 5725 5560 50  0001 C CNN "manf#"
 	1    5625 5425
 	1    0    0    -1
@@
 F 2 "Resistors_SMD:R_0603" H 9025 4800 60  0001 C CNN
 F 3 "" H 9025 4800 60  0001 C CNN
-F 4 "CR0603-FX-1000ELF" H 9125 4900 50  0001 C CNN "manf#"
+F 4 "CR0603-FX-1001ELF" H 9125 4900 50  0001 C CNN "manf#"
 	1    9025 4800
 	0    1    -1   0
@@
 F 2 "Capacitors_SMD:C_0603" H 8663 5400 50  0001 C CNN
 F 3 "" H 8625 5450 50  0001 C CNN
-F 4 "GRM188R71H472JA01J" H 8725 5585 50  0001 C CNN "manf#"
+F 4 "GCM188R71H153KA37D" H 8725 5585 50  0001 C CNN "manf#"
 	1    8625 5450
 	1    0    0    -1
