File: design/Power.sch (KiCad schematic (older format))
At the start: 43 parts, among them P10 PH_C, P11 SUPPLY, P12 GND, P8 PH_A, P9 PH_B, Q1 IRF7749, Q2 IRF7749, Q3 IRF7749, Q4 IRF7749, Q5 IRF7749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

Commit message: TESC 1.4
Parts:
- Q1, Q2, Q3, Q4, Q5, Q6: manf# (none) -> IRF7749L1TRPBF
Changed lines of the file:
@@
 F 2 "IR-DirectFETs:DirectFET_L8" H 3700 2025 50  0001 L CIN
 F 3 "" H 3450 2100 50  0001 L CNN
+F 4 "IRF7749L1TRPBF" H 3450 2100 60  0001 C CNN "manf#"
 	1    3450 2100
 	1    0    0    -1
@@
 F 2 "IR-DirectFETs:DirectFET_L8" H 3700 3125 50  0001 L CIN
 F 3 "" H 3450 3200 50  0001 L CNN
+F 4 "IRF7749L1TRPBF" H 3450 3200 60  0001 C CNN "manf#"
 	1    3450 3200
 	1    0    0    -1
@@
 F 2 "IR-DirectFETs:DirectFET_L8" H 7050 2025 50  0001 L CIN
 F 3 "" H 6800 2100 50  0001 L CNN
+F 4 "IRF7749L1TRPBF" H 6800 2100 60  0001 C CNN "manf#"
 	1    6800 2100
 	1    0    0    -1
@@
 F 2 "IR-DirectFETs:DirectFET_L8" H 7050 3125 50  0001 L CIN
 F 3 "" H 6800 3200 50  0001 L CNN
+F 4 "IRF7749L1TRPBF" H 6800 3200 60  0001 C CNN "manf#"
 	1    6800 3200
 	1    0    0    -1
@@
 F 2 "IR-DirectFETs:DirectFET_L8" H 10375 2025 50  0001 L CIN
 F 3 "" H 10125 2100 50  0001 L CNN
+F 4 "IRF7749L1TRPBF" H 10125 2100 60  0001 C CNN "manf#"
 	1    10125 2100
 	1    0    0    -1
@@
 F 2 "IR-DirectFETs:DirectFET_L8" H 10375 3125 50  0001 L CIN
 F 3 "" H 10125 3200 50  0001 L CNN
+F 4 "IRF7749L1TRPBF" H 10125 3200 60  0001 C CNN "manf#"
 	1    10125 3200
 	1    0    0    -1

Commit message: Add manf# field
Parts:
- C29, C30, C45: manf# (none) -> GRM188R71H472JA01J
- C35, C36, C38, C42: manf# (none) -> C1608X5R1C225K080AB
- C37, C39, C40, C41, C43, C44: manf# (none) -> CGA6M3X7S2A475K200AE
- C46, C47: manf# (none) -> EKZN630ELL681MK30S
- R24, R29, R32: manf# (none) -> CSS2H-3920R-L500FE
- R25, R26, R30, R31, R33, R34: manf# (none) -> CRCW06034R70FKEA
- R27: manf# (none) -> NCP18XH103F03RB
- R28: manf# (none) -> CR0603-FX-1002ELF
- R35, R36, R37: manf# (none) -> CR0603-FX-1000ELF
- U5, U6, U7: manf# (none) -> AD8418AWBRMZ

Commit message: Support KiCad 5.1.4
Parts:
- C29, C30, C35, C36, C38, C42, C45: footprint Capacitors_SMD:C_0603 -> Capacitor_SMD:C_0603_1608Metric; symbol C -> Device:C
- C37, C39, C40, C41, C43, C44: footprint Capacitors_SMD:C_1210 -> Capacitor_SMD:C_1210_3225Metric; symbol C -> Device:C
- C46, C47: symbol CP1 -> Device:CP1
- P10, P11, P12, P8, P9: symbol Conn_01x01 -> Connector_Generic:Conn_01x01
- Q1, Q2, Q3, Q4, Q5, Q6: symbol IRF7749 -> crf_1:IRF7749
- R24, R29, R32: symbol SHUNT -> crf_1:SHUNT
- R25, R26, R27, R28, R30, R31, R33, R34, R35, R36, R37: footprint Resistors_SMD:R_0603 -> Resistor_SMD:R_0603_1608Metric; symbol R -> Device:R
- U5, U6, U7: footprint Housings_SSOP:MSOP-8_3x3mm_Pitch0.65mm -> Package_SO:MSOP-8_3x3mm_P0.65mm; symbol AD8418-CST -> crf_1:AD8418-CST

Commit message: Load KiCad 4.0.7 schematic symbols, footprints & 3D models
Parts:
- C29, C30, C35, C36, C38, C42, C45: footprint Capacitor_SMD:C_0603_1608Metric -> Capacitors_SMD:C_0603
- C37, C39, C40, C41, C43, C44: footprint Capacitor_SMD:C_1210_3225Metric -> Capacitors_SMD:C_1210
- R25, R26, R27, R28, R30, R31, R33, R34, R35, R36, R37: footprint Resistor_SMD:R_0603_1608Metric -> Resistors_SMD:R_0603
- U5, U6, U7: footprint Package_SO:MSOP-8_3x3mm_P0.65mm -> Housings_SSOP:MSOP-8_3x3mm_Pitch0.65mm
Changed lines of the file:
@@
 F 0 "R26" V 3000 3200 50  0000 C CNN
 F 1 "4.7R" V 2900 3200 50  0000 C CNN
-F 2 "Resistor_SMD:R_0603_1608Metric" H 2900 3200 60  0001 C CNN
+F 2 "Resistors_SMD:R_0603" H 2900 3200 60  0001 C CNN
 F 3 "" H 2900 3200 60  0001 C CNN
 F 4 "CRCW06034R70FKEA" H 3000 3300 50  0001 C CNN "manf#"
@@
 F 0 "R25" V 3000 2100 50  0000 C CNN
 F 1 "4.7R" V 2900 2100 50  0000 C CNN
-F 2 "Resistor_SMD:R_0603_1608Metric" H 2900 2100 60  0001 C CNN
+F 2 "Resistors_SMD:R_0603" H 2900 2100 60  0001 C CNN
 F 3 "" H 2900 2100 60  0001 C CNN
 F 4 "CRCW06034R70FKEA" H 3000 2200 50  0001 C CNN "manf#"
@@
 F 0 "R35" V 1975 5175 50  0000 C CNN
 F 1 "100R" V 1775 5175 50  0000 C CNN
-F 2 "Resistor_SMD:R_0603_1608Metric" H 1875 5175 60  0001 C CNN
+F 2 "Resistors_SMD:R_0603" H 1875 5175 60  0001 C CNN
 F 3 "" H 1875 5175 60  0001 C CNN
 F 4 "CR0603-FX-1000ELF" H 1975 5275 50  0001 C CNN "manf#"
@@
 F 0 "C35" H 1700 3875 50  0000 L CNN
 F 1 "2.2u" H 1700 3675 50  0000 L CNN
-F 2 "Capacitor_SMD:C_0603_1608Metric" H 1713 3625 50  0001 C CNN
+F 2 "Capacitors_SMD:C_0603" H 1713 3625 50  0001 C CNN
 F 3 "" H 1675 3775 50  0001 C CNN
 F 4 "C1608X5R1C225K080AB" H 1700 3975 50  0001 C CNN "manf#"
@@
 F 0 "C37" V 3800 2475 50  0000 C TNN
 F 1 "4.7u_100V" V 3800 2850 50  0000 C TNN
-F 2 "Capacitor_SMD:C_1210_3225Metric" H 3913 2450 50  0001 C CNN
+F 2 "Capacitors_SMD:C_1210" H 3913 2450 50  0001 C CNN
 F 3 "" H 3875 2600 50  0001 C CNN
 F 4 "CGA6M3X7S2A475K200AE" H 3800 2575 50  0001 C CNN "manf#"
@@
 F 0 "C39" V 4000 2475 50  0000 C TNN
 F 1 "4.7u_100V" V 4000 2850 50  0000 C TNN
-F 2 "Capacitor_SMD:C_1210_3225Metric" H 4113 2450 50  0001 C CNN
+F 2 "Capacitors_SMD:C_1210" H 4113 2450 50  0001 C CNN
 F 3 "" H 4075 2600 50  0001 C CNN
 F 4 "CGA6M3X7S2A475K200AE" H 4000 2575 50  0001 C CNN "manf#"
@@
 F 0 "R31" V 6350 3200 50  0000 C CNN
 F 1 "4.7R" V 6250 3200 50  0000 C CNN
-F 2 "Resistor_SMD:R_0603_1608Metric" H 6250 3200 60  0001 C CNN
+F 2 "Resistors_SMD:R_0603" H 6250 3200 60  0001 C CNN
 F 3 "" H 6250 3200 60  0001 C CNN
 F 4 "CRCW06034R70FKEA" H 6350 3300 50  0001 C CNN "manf#"
@@
 F 0 "R30" V 6350 2100 50  0000 C CNN
 F 1 "4.7R" V 6250 2100 50  0000 C CNN
-F 2 "Resistor_SMD:R_0603_1608Metric" H 6250 2100 60  0001 C CNN
+F 2 "Resistors_SMD:R_0603" H 6250 2100 60  0001 C CNN
 F 3 "" H 6250 2100 60  0001 C CNN
 F 4 "CRCW06034R70FKEA" H 6350 2200 50  0001 C CNN "manf#"
@@
 F 0 "C41" V 7150 2475 50  0000 C TNN
 F 1 "4.7u_100V" V 7150 2850 50  0000 C TNN
-F 2 "Capacitor_SMD:C_1210_3225Metric" H 7263 2450 50  0001 C CNN
+F 2 "Capacitors_SMD:C_1210" H 7263 2450 50  0001 C CNN
 F 3 "" H 7225 2600 50  0001 C CNN
 F 4 "CGA6M3X7S2A475K200AE" H 7150 2575 50  0001 C CNN "manf#"
@@
 F 0 "C40" V 7350 2475 50  0000 C TNN
 F 1 "4.7u_100V" V 7350 2850 50  0000 C TNN
-F 2 "Capacitor_SMD:C_1210_3225Metric" H 7463 2450 50  0001 C CNN
+F 2 "Capacitors_SMD:C_1210" H 7463 2450 50  0001 C CNN
 F 3 "" H 7425 2600 50  0001 C CNN
 F 4 "CGA6M3X7S2A475K200AE" H 7350 2575 50  0001 C CNN "manf#"
@@
 F 0 "R34" V 9675 3200 50  0000 C CNN
 F 1 "4.7R" V 9575 3200 50  0000 C CNN
-F 2 "Resistor_SMD:R_0603_1608Metric" H 9575 3200 60  0001 C CNN
+F 2 "Resistors_SMD:R_0603" H 9575 3200 60  0001 C CNN
 F 3 "" H 9575 3200 60  0001 C CNN
 F 4 "CRCW06034R70FKEA" H 9675 3300 50  0001 C CNN "manf#"
@@
 F 0 "R33" V 9675 2100 50  0000 C CNN
 F 1 "4.7R" V 9575 2100 50  0000 C CNN
-F 2 "Resistor_SMD:R_0603_1608Metric" H 9575 2100 60  0001 C CNN
+F 2 "Resistors_SMD:R_0603" H 9575 2100 60  0001 C CNN
 F 3 "" H 9575 2100 60  0001 C CNN
 F 4 "CRCW06034R70FKEA" H 9675 2200 50  0001 C CNN "manf#"
@@
 F 0 "C43" V 10475 2475 50  0000 C TNN
 F 1 "4.7u_100V" V 10475 2850 50  0000 C TNN
-F 2 "Capacitor_SMD:C_1210_3225Metric" H 10588 2450 50  0001 C CNN
+F 2 "Capacitors_SMD:C_1210" H 10588 2450 50  0001 C CNN
 F 3 "" H 10550 2600 50  0001 C CNN
 F 4 "CGA6M3X7S2A475K200AE" H 10475 2575 50  0001 C CNN "manf#"
@@
 F 0 "C44" V 10675 2475 50  0000 C TNN
 F 1 "4.7u_100V" V 10675 2850 50  0000 C TNN
-F 2 "Capacitor_SMD:C_1210_3225Metric" H 10788 2450 50  0001 C CNN
+F 2 "Capacitors_SMD:C_1210" H 10788 2450 50  0001 C CNN
 F 3 "" H 10750 2600 50  0001 C CNN
 F 4 "CGA6M3X7S2A475K200AE" H 10675 2575 50  0001 C CNN "manf#"
@@
 F 0 "C29" H 1575 5435 50  0000 L CNN
 F 1 "4.7n" H 1575 5365 50  0000 L CNN
-F 2 "Capacitor_SMD:C_0603_1608Metric" H 1513 5350 50  0001 C CNN
+F 2 "Capacitors_SMD:C_0603" H 1513 5350 50  0001 C CNN
 F 3 "" H 1475 5400 50  0001 C CNN
 F 4 "GRM188R71H472JA01J" H 1575 5535 50  0001 C CNN "manf#"
@@
 F 0 "R36" V 1975 5950 50  0000 C CNN
 F 1 "100R" V 1775 5950 50  0000 C CNN
-F 2 "Resistor_SMD:R_0603_1608Metric" H 1875 5950 60  0001 C CNN
+F 2 "Resistors_SMD:R_0603" H 1875 5950 60  0001 C CNN
 F 3 "" H 1875 5950 60  0001 C CNN
 F 4 "CR0603-FX-1000ELF" H 1975 6050 50  0001 C CNN "manf#"
@@
 F 0 "C30" H 1575 6210 50  0000 L CNN
 F 1 "4.7n" H 1575 6140 50  0000 L CNN
-F 2 "Capacitor_SMD:C_0603_1608Metric" H 1513 6125 50  0001 C CNN
+F 2 "Capacitors_SMD:C_0603" H 1513 6125 50  0001 C CNN
 F 3 "" H 1475 6175 50  0001 C CNN
 F 4 "GRM188R71H472JA01J" H 1575 6310 50  0001 C CNN "manf#"
@@
 F 0 "R37" V 1975 6725 50  0000 C CNN
 F 1 "100R" V 1775 6725 50  0000 C CNN
-F 2 "Resistor_SMD:R_0603_1608Metric" H 1875 6725 60  0001 C CNN
+F 2 "Resistors_SMD:R_0603" H 1875 6725 60  0001 C CNN
 F 3 "" H 1875 6725 60  0001 C CNN
 F 4 "CR0603-FX-1000ELF" H 1975 6825 50  0001 C CNN "manf#"
@@
 F 0 "C45" H 1575 6985 50  0000 L CNN
 F 1 "4.7n" H 1575 6915 50  0000 L CNN
-F 2 "Capacitor_SMD:C_0603_1608Metric" H 1513 6900 50  0001 C CNN
+F 2 "Capacitors_SMD:C_0603" H 1513 6900 50  0001 C CNN
 F 3 "" H 1475 6950 50  0001 C CNN
 F 4 "GRM188R71H472JA01J" H 1575 7085 50  0001 C CNN "manf#"
@@
 F 0 "R27" V 4030 5825 40  0000 C CNN
 F 1 "NTC 10k" V 3850 5826 40  0000 C CNN
-F 2 "Resistor_SMD:R_0603_1608Metric" V 3880 5825 30  0001 C CNN
+F 2 "Resistors_SMD:R_0603" V 3880 5825 30  0001 C CNN
 F 3 "" H 3950 5825 30  0000 C CNN
 F 4 "NCP18XH103F03RB" H 4030 5925 50  0001 C CNN "manf#"
@@
 F 0 "R28" V 4030 6525 40  0000 C CNN
 F 1 "10k" V 3850 6526 40  0000 C CNN
-F 2 "Resistor_SMD:R_0603_1608Metric" V 3880 6525 30  0001 C CNN
+F 2 "Resistors_SMD:R_0603" V 3880 6525 30  0001 C CNN
 F 3 "" H 3950 6525 30  0000 C CNN
 F 4 "CR0603-FX-1002ELF" H 4030 6625 50  0001 C CNN "manf#"
@@
 F 0 "C36" H 3725 6625 40  0000 L CNN
 F 1 "2.2u" H 3725 6450 40  0000 L CNN
-F 2 "Capacitor_SMD:C_0603_1608Metric" H 3738 6375 30  0001 C CNN
+F 2 "Capacitors_SMD:C_0603" H 3738 6375 30  0001 C CNN
 F 3 "" H 3700 6525 60  0000 C CNN
 F 4 "C1608X5R1C225K080AB" H 3725 6725 50  0001 C CNN "manf#"
@@
 F 0 "U5" H 1375 3700 50  0000 R CNN
 F 1 "AD8418" H 1825 2925 50  0000 R CNN
-F 2 "Package_SO:MSOP-8_3x3mm_P0.65mm" H 1725 2925 50  0001 C CNN
+F 2 "Housings_SSOP:MSOP-8_3x3mm_Pitch0.65mm" H 1725 2925 50  0001 C CNN
 F 3 "" H 2325 2575 50  0001 C CNN
 F 4 "AD8418AWBRMZ" H 1375 3800 50  0001 C CNN "manf#"
@@
 F 0 "U6" H 4725 3700 50  0000 R CNN
 F 1 "AD8418" H 5175 2925 50  0000 R CNN
-F 2 "Package_SO:MSOP-8_3x3mm_P0.65mm" H 5075 2925 50  0001 C CNN
+F 2 "Housings_SSOP:MSOP-8_3x3mm_Pitch0.65mm" H 5075 2925 50  0001 C CNN
 F 3 "" H 5675 2575 50  0001 C CNN
 F 4 "AD8418AWBRMZ" H 4725 3800 50  0001 C CNN "manf#"
@@
 F 0 "U7" H 8050 3700 50  0000 R CNN
 F 1 "AD8418" H 8500 2925 50  0000 R CNN
-F 2 "Package_SO:MSOP-8_3x3mm_P0.65mm" H 8400 2925 50  0001 C CNN
+F 2 "Housings_SSOP:MSOP-8_3x3mm_Pitch0.65mm" H 8400 2925 50  0001 C CNN
 F 3 "" H 9000 2575 50  0001 C CNN
 F 4 "AD8418AWBRMZ" H 8050 3800 50  0001 C CNN "manf#"
@@
 F 0 "C38" H 5050 3875 50  0000 L CNN
 F 1 "2.2u" H 5050 3675 50  0000 L CNN
-F 2 "Capacitor_SMD:C_0603_1608Metric" H 5063 3625 50  0001 C CNN
+F 2 "Capacitors_SMD:C_0603" H 5063 3625 50  0001 C CNN
 F 3 "" H 5025 3775 50  0001 C CNN
 F 4 "C1608X5R1C225K080AB" H 5050 3975 50  0001 C CNN "manf#"
@@
 F 0 "C42" H 8375 3875 50  0000 L CNN
 F 1 "2.2u" H 8375 3675 50  0000 L CNN
-F 2 "Capacitor_SMD:C_0603_1608Metric" H 8388 3625 50  0001 C CNN
+F 2 "Capacitors_SMD:C_0603" H 8388 3625 50  0001 C CNN
 F 3 "" H 8350 3775 50  0001 C CNN
 F 4 "C1608X5R1C225K080AB" H 8375 3975 50  0001 C CNN "manf#"
