File: design/MCU.sch (KiCad schematic (older format))
At the start: 13 parts, among them U1 STM32F40X_LQFP64, X1 8m

Commit message: initial commit
Parts:
- C10, C11, C12, C2, C3, C4, C5, C6, C7, C8, C9: footprint CRF1:SMD-0603_c -> Capacitors_SMD:C_0603

Commit message: initial commit
Parts:
- X1: footprint mojaKniznica:5x3.2KRISTALL -> Crystals:Crystal_SMD_5032_4Pads
Changed lines of the file:
@@
 LIBS:valves
 LIBS:crf_1
+LIBS:VESC_6-cache
 EELAYER 25 0
 EELAYER END
@@
 U 1 1 53F757AE
 P 6575 6075
-F 0 "C4" H 6625 6175 50 0000 L CNN
-F 1 "2.2u" H 6625 5975 50 0000 L CNN
-F 2 "Capacitors_SMD:C_0603" H 6575 6075 60 0001 C CNN
-F 3 "" H 6575 6075 60 0001 C CNN
+F 0 "C4" H 6625 6175 50  0000 L CNN
+F 1 "2.2u" H 6625 5975 50  0000 L CNN
+F 2 "Capacitors_SMD:C_0603" H 6575 6075 60  0001 C CNN
+F 3 "" H 6575 6075 60  0001 C CNN
 	1    6575 6075
 	0    1    1    0
@@
 U 1 1 53F757B5
 P 6575 5825
-F 0 "C3" H 6625 5925 50 0000 L CNN
-F 1 "2.2u" H 6625 5725 50 0000 L CNN
-F 2 "Capacitors_SMD:C_0603" H 6575 5825 60 0001 C CNN
-F 3 "" H 6575 5825 60 0001 C CNN
+F 0 "C3" H 6625 5925 50  0000 L CNN
+F 1 "2.2u" H 6625 5725 50  0000 L CNN
+F 2 "Capacitors_SMD:C_0603" H 6575 5825 60  0001 C CNN
+F 3 "" H 6575 5825 60  0001 C CNN
 	1    6575 5825
 	0    1    1    0
@@
 U 1 1 53F757C2
 P 6475 4825
-F 0 "#PWR028" H 6475 4925 30 0001 C CNN
-F 1 "VCC" H 6475 4925 30 0000 C CNN
-F 2 "" H 6475 4825 60 0001 C CNN
-F 3 "" H 6475 4825 60 0001 C CNN
+F 0 "#PWR028" H 6475 4925 30  0001 C CNN
+F 1 "VCC" H 6475 4925 30  0000 C CNN
+F 2 "" H 6475 4825 60  0001 C CNN
+F 3 "" H 6475 4825 60  0001 C CNN
 	1    6475 4825
 	1    0    0    -1
@@
 U 1 1 53F757CE
 P 6275 3925
-F 0 "#PWR029" H 6275 4025 30 0001 C CNN
-F 1 "VCC" H 6275 4025 30 0000 C CNN
-F 2 "" H 6275 3925 60 0001 C CNN
-F 3 "" H 6275 3925 60 0001 C CNN
+F 0 "#PWR029" H 6275 4025 30  0001 C CNN
+F 1 "VCC" H 6275 4025 30  0000 C CNN
+F 2 "" H 6275 3925 60  0001 C CNN
+F 3 "" H 6275 3925 60  0001 C CNN
 	1    6275 3925
 	1    0    0    -1
@@
 U 1 1 53F757DB
 P 6425 1525
-F 0 "C2" H 6475 1625 50 0000 L CNN
-F 1 "15p" H 6475 1425 50 0000 L CNN
-F 2 "Capacitors_SMD:C_0603" H 6425 1525 60 0001 C CNN
-F 3 "" H 6425 1525 60 0001 C CNN
+F 0 "C2" H 6475 1625 50  0000 L CNN
+F 1 "15p" H 6475 1425 50  0000 L CNN
+F 2 "Capacitors_SMD:C_0603" H 6425 1525 60  0001 C CNN
+F 3 "" H 6425 1525 60  0001 C CNN
 	1    6425 1525
 	-1   0    0    -1
@@
 U 1 1 53F757E2
 P 7175 1525
-F 0 "C8" H 7225 1625 50 0000 L CNN
-F 1 "15p" H 7225 1425 50 0000 L CNN
-F 2 "Capacitors_SMD:C_0603" H 7175 1525 60 0001 C CNN
-F 3 "" H 7175 1525 60 0001 C CNN
+F 0 "C8" H 7225 1625 50  0000 L CNN
+F 1 "15p" H 7225 1425 50  0000 L CNN
+F 2 "Capacitors_SMD:C_0603" H 7175 1525 60  0001 C CNN
+F 3 "" H 7175 1525 60  0001 C CNN
 	1    7175 1525
 	-1   0    0    -1
@@
 U 1 1 53F757F8
 P 6825 5175
-F 0 "C5" H 6875 5275 50 0000 L CNN
-F 1 "2.2u" H 6875 5075 50 0000 L CNN
-F 2 "Capacitors_SMD:C_0603" H 6825 5175 60 0001 C CNN
-F 3 "" H 6825 5175 60 0001 C CNN
+F 0 "C5" H 6875 5275 50  0000 L CNN
+F 1 "2.2u" H 6875 5075 50  0000 L CNN
+F 2 "Capacitors_SMD:C_0603" H 6825 5175 60  0001 C CNN
+F 3 "" H 6825 5175 60  0001 C CNN
 	1    6825 5175
 	1    0    0    -1
@@
 U 1 1 53F757FF
 P 7075 5175
-F 0 "C6" H 7125 5275 50 0000 L CNN
-F 1 "2.2u" H 7125 5075 50 0000 L CNN
-F 2 "Capacitors_SMD:C_0603" H 7075 5175 60 0001 C CNN
-F 3 "" H 7075 5175 60 0001 C CNN
+F 0 "C6" H 7125 5275 50  0000 L CNN
+F 1 "2.2u" H 7125 5075 50  0000 L CNN
+F 2 "Capacitors_SMD:C_0603" H 7075 5175 60  0001 C CNN
+F 3 "" H 7075 5175 60  0001 C CNN
 	1    7075 5175
 	1    0    0    -1
@@
 U 1 1 53F75807
 P 6275 5175
-F 0 "#PWR030" H 6275 5275 30 0001 C CNN
-F 1 "VCC" H 6275 5275 30 0000 C CNN
-F 2 "" H 6275 5175 60 0001 C CNN
-F 3 "" H 6275 5175 60 0001 C CNN
+F 0 "#PWR030" H 6275 5275 30  0001 C CNN
+F 1 "VCC" H 6275 5275 30  0000 C CNN
+F 2 "" H 6275 5175 60  0001 C CNN
+F 3 "" H 6275 5175 60  0001 C CNN
 	1    6275 5175
 	1    0    0    -1
@@
 U 1 1 53F75896
 P 7025 2750
-F 0 "C7" H 7075 2830 50 0000 L BNN
-F 1 "100n" H 7075 2650 50 0000 L CNN
-F 2 "Capacitors_SMD:C_0603" H 7025 2750 60 0001 C CNN
-F 3 "" H 7025 2750 60 0001 C CNN
+F 0 "C7" H 7075 2830 50  0000 L BNN
+F 1 "100n" H 7075 2650 50  0000 L CNN
+F 2 "Capacitors_SMD:C_0603" H 7025 2750 60  0001 C CNN
+F 3 "" H 7025 2750 60  0001 C CNN
 	1    7025 2750
 	1    0    0    -1
@@
 U 1 1 53F77426
 P 9125 1325
-F 0 "C9" H 9175 1425 50 0000 L CNN
-F 1 "2.2u" H 9175 1225 50 0000 L CNN
-F 2 "Capacitors_SMD:C_0603" H 9125 1325 60 0001 C CNN
-F 3 "" H 9125 1325 60 0001 C CNN
+F 0 "C9" H 9175 1425 50  0000 L CNN
+F 1 "2.2u" H 9175 1225 50  0000 L CNN
+F 2 "Capacitors_SMD:C_0603" H 9125 1325 60  0001 C CNN
+F 3 "" H 9125 1325 60  0001 C CNN
 	1    9125 1325
 	1    0    0    -1
@@
 U 1 1 53F7742D
 P 9375 1325
-F 0 "C10" H 9425 1425 50 0000 L CNN
-F 1 "2.2u" H 9425 1225 50 0000 L CNN
-F 2 "Capacitors_SMD:C_0603" H 9375 1325 60 0001 C CNN
-F 3 "" H 9375 1325 60 0001 C CNN
+F 0 "C10" H 9425 1425 50  0000 L CNN
+F 1 "2.2u" H 9425 1225 50  0000 L CNN
+F 2 "Capacitors_SMD:C_0603" H 9375 1325 60  0001 C CNN
+F 3 "" H 9375 1325 60  0001 C CNN
 	1    9375 1325
 	1    0    0    -1
@@
 U 1 1 53F77441
 P 8825 975
-F 0 "#PWR031" H 8825 1075 30 0001 C CNN
-F 1 "VCC" H 8825 1075 30 0000 C CNN
-F 2 "" H 8825 975 60 0001 C CNN
-F 3 "" H 8825 975 60 0001 C CNN
+F 0 "#PWR031" H 8825 1075 30  0001 C CNN
+F 1 "VCC" H 8825 1075 30  0000 C CNN
+F 2 "" H 8825 975 60  0001 C CNN
+F 3 "" H 8825 975 60  0001 C CNN
 	1    8825 975
 	1    0    0    -1
@@
 U 1 1 53F77447
 P 9625 1325
-F 0 "C11" H 9675 1425 50 0000 L CNN
-F 1 "2.2u" H 9675 1225 50 0000 L CNN
-F 2 "Capacitors_SMD:C_0603" H 9625 1325 60 0001 C CNN
-F 3 "" H 9625 1325 60 0001 C CNN
+F 0 "C11" H 9675 1425 50  0000 L CNN
+F 1 "2.2u" H 9675 1225 50  0000 L CNN
+F 2 "Capacitors_SMD:C_0603" H 9625 1325 60  0001 C CNN
+F 3 "" H 9625 1325 60  0001 C CNN
 	1    9625 1325
 	1    0    0    -1
@@
 U 1 1 53F7744E
 P 9875 1325
-F 0 "C12" H 9925 1425 50 0000 L CNN
-F 1 "2.2u" H 9925 1225 50 0000 L CNN
-F 2 "Capacitors_SMD:C_0603" H 9875 1325 60 0001 C CNN
-F 3 "" H 9875 1325 60 0001 C CNN
+F 0 "C12" H 9925 1425 50  0000 L CNN
+F 1 "2.2u" H 9925 1225 50  0000 L CNN
+F 2 "Capacitors_SMD:C_0603" H 9875 1325 60  0001 C CNN
+F 3 "" H 9875 1325 60  0001 C CNN
 	1    9875 1325
 	1    0    0    -1
@@
 U 1 1 53F757A7
 P 4825 3625
-F 0 "U1" H 4775 5925 60 0000 C CNN
-F 1 "STM32F40X_LQFP64" H 4825 1275 60 0000 C CNN
-F 2 "CRF1:lqfp64_pad_mod" H 4825 3625 60 0001 C CNN
-F 3 "" H 4825 3625 60 0001 C CNN
+F 0 "U1" H 4775 5925 60  0000 C CNN
+F 1 "STM32F40X_LQFP64" H 4825 1275 60  0000 C CNN
+F 2 "CRF1:lqfp64_pad_mod" H 4825 3625 60  0001 C CNN
+F 3 "" H 4825 3625 60  0001 C CNN
 	1    4825 3625
 	1    0    0    -1
@@
 U 1 1 5A965081
 P 7025 3025
-F 0 "#PWR032" H 7025 2775 50 0001 C CNN
-F 1 "GND" H 7025 2875 50 0000 C CNN
-F 2 "" H 7025 3025 50 0001 C CNN
-F 3 "" H 7025 3025 50 0001 C CNN
+F 0 "#PWR032" H 7025 2775 50  0001 C CNN
+F 1 "GND" H 7025 2875 50  0000 C CNN
+F 2 "" H 7025 3025 50  0001 C CNN
+F 3 "" H 7025 3025 50  0001 C CNN
 	1    7025 3025
 	1    0    0    -1
@@
 U 1 1 5A965E92
 P 6775 1975
-F 0 "#PWR033" H 6775 1725 50 0001 C CNN
-F 1 "GND" H 6775 1825 50 0000 C CNN
-F 2 "" H 6775 1975 50 0001 C CNN
-F 3 "" H 6775 1975 50 0001 C CNN
+F 0 "#PWR033" H 6775 1725 50  0001 C CNN
+F 1 "GND" H 6775 1825 50  0000 C CNN
+F 2 "" H 6775 1975 50  0001 C CNN
+F 3 "" H 6775 1975 50  0001 C CNN
 	1    6775 1975
 	1    0    0    -1
@@
 U 1 1 5A96886F
 P 7425 1350
-F 0 "#PWR034" H 7425 1100 50 0001 C CNN
-F 1 "GND" H 7425 1200 50 0000 C CNN
-F 2 "" H 7425 1350 50 0001 C CNN
-F 3 "" H 7425 1350 50 0001 C CNN
+F 0 "#PWR034" H 7425 1100 50  0001 C CNN
+F 1 "GND" H 7425 1200 50  0000 C CNN
+F 2 "" H 7425 1350 50  0001 C CNN
+F 3 "" H 7425 1350 50  0001 C CNN
 	1    7425 1350
 	1    0    0    -1
@@
 U 1 1 5A968FE6
 P 8825 1675
-F 0 "#PWR035" H 8825 1425 50 0001 C CNN
-F 1 "GND" H 8825 1525 50 0000 C CNN
-F 2 "" H 8825 1675 50 0001 C CNN
-F 3 "" H 8825 1675 50 0001 C CNN
+F 0 "#PWR035" H 8825 1425 50  0001 C CNN
+F 1 "GND" H 8825 1525 50  0000 C CNN
+F 2 "" H 8825 1675 50  0001 C CNN
+F 3 "" H 8825 1675 50  0001 C CNN
 	1    8825 1675
 	1    0    0    -1
@@
 U 1 1 5A96B952
 P 6225 2150
-F 0 "#PWR036" H 6225 1900 50 0001 C CNN
-F 1 "GND" H 6225 2000 50 0000 C CNN
-F 2 "" H 6225 2150 50 0001 C CNN
-F 3 "" H 6225 2150 50 0001 C CNN
+F 0 "#PWR036" H 6225 1900 50  0001 C CNN
+F 1 "GND" H 6225 2000 50  0000 C CNN
+F 2 "" H 6225 2150 50  0001 C CNN
+F 3 "" H 6225 2150 50  0001 C CNN
 	1    6225 2150
 	1    0    0    -1
@@
 U 1 1 5A954317
 P 7075 5775
-F 0 "#PWR037" H 7075 5525 50 0001 C CNN
-F 1 "GND" H 7075 5625 50 0000 C CNN
-F 2 "" H 7075 5775 50 0001 C CNN
-F 3 "" H 7075 5775 50 0001 C CNN
+F 0 "#PWR037" H 7075 5525 50  0001 C CNN
+F 1 "GND" H 7075 5625 50  0000 C CNN
+F 2 "" H 7075 5775 50  0001 C CNN
+F 3 "" H 7075 5775 50  0001 C CNN
 	1    7075 5775
 	1    0    0    -1
@@
 U 1 1 5A9543CD
 P 6275 4825
-F 0 "#PWR038" H 6275 4575 50 0001 C CNN
-F 1 "GND" H 6275 4675 50 0000 C CNN
-F 2 "" H 6275 4825 50 0001 C CNN
-F 3 "" H 6275 4825 50 0001 C CNN
+F 0 "#PWR038" H 6275 4575 50  0001 C CNN
+F 1 "GND" H 6275 4675 50  0000 C CNN
+F 2 "" H 6275 4825 50  0001 C CNN
+F 3 "" H 6275 4825 50  0001 C CNN
 	1    6275 4825
 	1    0    0    -1
@@
 U 1 1 5A940C20
 P 6775 1775
-F 0 "X1" H 6775 1865 50 0000 C CNN
-F 1 "8m" H 6805 1665 50 0000 L CNN
-F 2 "mojaKniznica:5x3.2KRISTALL" H 6775 1775 60 0001 C CNN
-F 3 "" H 6775 1775 60 0000 C CNN
+F 0 "X1" H 6775 1865 50  0000 C CNN
+F 1 "8m" H 6805 1665 50  0000 L CNN
+F 2 "Crystals:Crystal_SMD_5032_4Pads" H 6775 1775 60  0001 C CNN
+F 3 "" H 6775 1775 60  0000 C CNN
 	1    6775 1775
 	1    0    0    -1

Commit message: initial commit
Parts:
- U1: footprint CRF1:lqfp64_pad_mod -> CRF1:STM32F4x5RG
Changed lines of the file:
@@
 F 0 "U1" H 4775 5925 60  0000 C CNN
 F 1 "STM32F40X_LQFP64" H 4825 1275 60  0000 C CNN
-F 2 "CRF1:lqfp64_pad_mod" H 4825 3625 60  0001 C CNN
+F 2 "CRF1:STM32F4x5RG" H 4825 3625 60  0001 C CNN
 F 3 "" H 4825 3625 60  0001 C CNN
 	1    4825 3625

Commit message: TESC 1.4
Parts:
- U1: manf# (none) -> STM32F405RGT6
Changed lines of the file:
@@
 F 2 "CRF1:STM32F4x5RG" H 4825 3625 60  0001 C CNN
 F 3 "" H 4825 3625 60  0001 C CNN
+F 4 "STM32F405RGT6" H 4825 3625 60  0001 C CNN "manf#"
 	1    4825 3625
 	1    0    0    -1

Commit message: Add manf# field
Parts:
- C10, C11, C12, C3, C4, C5, C6, C9: manf# (none) -> C1608X5R1C225K080AB
- C2, C8: manf# (none) -> 06031A150JAT2A
- C7: manf# (none) -> C0603X104J5RACTU
- X1: manf# (none) -> ABM3B-8.000MHZ-10-1-U-T
