File: design/MCU.sch (KiCad schematic (older format))
At the start: 13 parts, among them U1 STM32F40X_LQFP64, X1 8m

Commit message: Support KiCad 5.1.4
Parts:
- C10, C11, C12, C2, C3, C4, C5, C6, C7, C8, C9: footprint Capacitors_SMD:C_0603 -> Capacitor_SMD:C_0603_1608Metric; symbol C -> Device:C
- U1: symbol STM32F40X_LQFP64 -> crf_1:STM32F40X_LQFP64
- X1: footprint Crystals:Crystal_SMD_5032_4Pads -> Crystal:Crystal_SMD_5032-4Pin_5.0x3.2mm; symbol CRYSTAL_SMD -> crf_1:CRYSTAL_SMD
Changed lines of the file:
@@
-EESchema Schematic File Version 2
-LIBS:power
-LIBS:device
-LIBS:transistors
-LIBS:conn
-LIBS:linear
-LIBS:regul
-LIBS:74xx
-LIBS:cmos4000
-LIBS:adc-dac
-LIBS:memory
-LIBS:xilinx
-LIBS:microcontrollers
-LIBS:dsp
-LIBS:microchip
-LIBS:analog_switches
-LIBS:motorola
-LIBS:texas
-LIBS:switches
-LIBS:intel
-LIBS:audio
-LIBS:interface
-LIBS:digital-audio
-LIBS:philips
-LIBS:display
-LIBS:cypress
-LIBS:siliconi
-LIBS:opto
-LIBS:atmel
-LIBS:contrib
-LIBS:valves
-LIBS:crf_1
+EESchema Schematic File Version 4
 LIBS:VESC_6-cache
-EELAYER 25 0
+EELAYER 30 0
 EELAYER END
 $Descr A4 11693 8268
@@
 $EndDescr
 $Comp
-L C C4
+L Device:C C4
 U 1 1 53F757AE
 P 6575 6075
 F 0 "C4" H 6625 6175 50  0000 L CNN
 F 1 "2.2u" H 6625 5975 50  0000 L CNN
-F 2 "Capacitors_SMD:C_0603" H 6575 6075 60  0001 C CNN
+F 2 "Capacitor_SMD:C_0603_1608Metric" H 6575 6075 60  0001 C CNN
 F 3 "" H 6575 6075 60  0001 C CNN
 F 4 "C1608X5R1C225K080AB" H 6625 6275 50  0001 C CNN "manf#"
@@
 $EndComp
 $Comp
-L C C3
+L Device:C C3
 U 1 1 53F757B5
 P 6575 5825
 F 0 "C3" H 6625 5925 50  0000 L CNN
 F 1 "2.2u" H 6625 5725 50  0000 L CNN
-F 2 "Capacitors_SMD:C_0603" H 6575 5825 60  0001 C CNN
+F 2 "Capacitor_SMD:C_0603_1608Metric" H 6575 5825 60  0001 C CNN
 F 3 "" H 6575 5825 60  0001 C CNN
 F 4 "C1608X5R1C225K080AB" H 6625 6025 50  0001 C CNN "manf#"
@@
 $EndComp
 $Comp
-L VCC #PWR028
+L power:VCC #PWR028
 U 1 1 53F757C2
 P 6475 4825
@@
 $EndComp
 $Comp
-L VCC #PWR029
+L power:VCC #PWR029
 U 1 1 53F757CE
 P 6275 3925
@@
 $EndComp
 $Comp
-L C C2
+L Device:C C2
 U 1 1 53F757DB
 P 6425 1525
 F 0 "C2" H 6475 1625 50  0000 L CNN
 F 1 "15p" H 6475 1425 50  0000 L CNN
-F 2 "Capacitors_SMD:C_0603" H 6425 1525 60  0001 C CNN
+F 2 "Capacitor_SMD:C_0603_1608Metric" H 6425 1525 60  0001 C CNN
 F 3 "" H 6425 1525 60  0001 C CNN
 F 4 "06031A150JAT2A" H 6475 1725 50  0001 C CNN "manf#"
@@
 $EndComp
 $Comp
-L C C8
+L Device:C C8
 U 1 1 53F757E2
 P 7175 1525
 F 0 "C8" H 7225 1625 50  0000 L CNN
 F 1 "15p" H 7225 1425 50  0000 L CNN
-F 2 "Capacitors_SMD:C_0603" H 7175 1525 60  0001 C CNN
+F 2 "Capacitor_SMD:C_0603_1608Metric" H 7175 1525 60  0001 C CNN
 F 3 "" H 7175 1525 60  0001 C CNN
 F 4 "06031A150JAT2A" H 7225 1725 50  0001 C CNN "manf#"
@@
 $EndComp
 $Comp
-L C C5
+L Device:C C5
 U 1 1 53F757F8
 P 6825 5175
 F 0 "C5" H 6875 5275 50  0000 L CNN
 F 1 "2.2u" H 6875 5075 50  0000 L CNN
-F 2 "Capacitors_SMD:C_0603" H 6825 5175 60  0001 C CNN
+F 2 "Capacitor_SMD:C_0603_1608Metric" H 6825 5175 60  0001 C CNN
 F 3 "" H 6825 5175 60  0001 C CNN
 F 4 "C1608X5R1C225K080AB" H 6875 5375 50  0001 C CNN "manf#"
@@
 $EndComp
 $Comp
-L C C6
+L Device:C C6
 U 1 1 53F757FF
 P 7075 5175
 F 0 "C6" H 7125 5275 50  0000 L CNN
 F 1 "2.2u" H 7125 5075 50  0000 L CNN
-F 2 "Capacitors_SMD:C_0603" H 7075 5175 60  0001 C CNN
+F 2 "Capacitor_SMD:C_0603_1608Metric" H 7075 5175 60  0001 C CNN
 F 3 "" H 7075 5175 60  0001 C CNN
 F 4 "C1608X5R1C225K080AB" H 7125 5375 50  0001 C CNN "manf#"
@@
 $EndComp
 $Comp
-L VCC #PWR030
+L power:VCC #PWR030
 U 1 1 53F75807
 P 6275 5175
@@
 $EndComp
 $Comp
-L C C7
+L Device:C C7
 U 1 1 53F75896
 P 7025 2750
 F 0 "C7" H 7075 2830 50  0000 L BNN
 F 1 "100n" H 7075 2650 50  0000 L CNN
-F 2 "Capacitors_SMD:C_0603" H 7025 2750 60  0001 C CNN
+F 2 "Capacitor_SMD:C_0603_1608Metric" H 7025 2750 60  0001 C CNN
 F 3 "" H 7025 2750 60  0001 C CNN
 F 4 "C0603X104J5RACTU" H 7075 2930 50  0001 C CNN "manf#"
@@
 $EndComp
 $Comp
-L C C9
+L Device:C C9
 U 1 1 53F77426
 P 9125 1325
 F 0 "C9" H 9175 1425 50  0000 L CNN
 F 1 "2.2u" H 9175 1225 50  0000 L CNN
-F 2 "Capacitors_SMD:C_0603" H 9125 1325 60  0001 C CNN
+F 2 "Capacitor_SMD:C_0603_1608Metric" H 9125 1325 60  0001 C CNN
 F 3 "" H 9125 1325 60  0001 C CNN
 F 4 "C1608X5R1C225K080AB" H 9175 1525 50  0001 C CNN "manf#"
@@
 $EndComp
 $Comp
-L C C10
+L Device:C C10
 U 1 1 53F7742D
 P 9375 1325
 F 0 "C10" H 9425 1425 50  0000 L CNN
 F 1 "2.2u" H 9425 1225 50  0000 L CNN
-F 2 "Capacitors_SMD:C_0603" H 9375 1325 60  0001 C CNN
+F 2 "Capacitor_SMD:C_0603_1608Metric" H 9375 1325 60  0001 C CNN
 F 3 "" H 9375 1325 60  0001 C CNN
 F 4 "C1608X5R1C225K080AB" H 9425 1525 50  0001 C CNN "manf#"
@@
 $EndComp
 $Comp
-L VCC #PWR031
+L power:VCC #PWR031
 U 1 1 53F77441
 P 8825 975
@@
 $EndComp
 $Comp
-L C C11
+L Device:C C11
 U 1 1 53F77447
 P 9625 1325
 F 0 "C11" H 9675 1425 50  0000 L CNN
 F 1 "2.2u" H 9675 1225 50  0000 L CNN
-F 2 "Capacitors_SMD:C_0603" H 9625 1325 60  0001 C CNN
+F 2 "Capacitor_SMD:C_0603_1608Metric" H 9625 1325 60  0001 C CNN
 F 3 "" H 9625 1325 60  0001 C CNN
 F 4 "C1608X5R1C225K080AB" H 9675 1525 50  0001 C CNN "manf#"
@@
 $EndComp
 $Comp
-L C C12
+L Device:C C12
 U 1 1 53F7744E
 P 9875 1325
 F 0 "C12" H 9925 1425 50  0000 L CNN
 F 1 "2.2u" H 9925 1225 50  0000 L CNN
-F 2 "Capacitors_SMD:C_0603" H 9875 1325 60  0001 C CNN
+F 2 "Capacitor_SMD:C_0603_1608Metric" H 9875 1325 60  0001 C CNN
 F 3 "" H 9875 1325 60  0001 C CNN
 F 4 "C1608X5R1C225K080AB" H 9925 1525 50  0001 C CNN "manf#"
@@
 $EndComp
 $Comp
-L STM32F40X_LQFP64 U1
+L crf_1:STM32F40X_LQFP64 U1
 U 1 1 53F757A7
 P 4825 3625
@@
 $EndComp
 $Comp
-L GND #PWR032
+L power:GND #PWR032
 U 1 1 5A965081
 P 7025 3025
@@
 $EndComp
 $Comp
-L GND #PWR033
+L power:GND #PWR033
 U 1 1 5A965E92
 P 6775 1975
@@
 $EndComp
 $Comp
-L GND #PWR034
+L power:GND #PWR034
 U 1 1 5A96886F
 P 7425 1350
@@
 $EndComp
 $Comp
-L GND #PWR035
+L power:GND #PWR035
 U 1 1 5A968FE6
 P 8825 1675
@@
 $EndComp
 $Comp
-L GND #PWR036
+L power:GND #PWR036
 U 1 1 5A96B952
 P 6225 2150
@@
 $EndComp
 $Comp
-L GND #PWR037
+L power:GND #PWR037
 U 1 1 5A954317
 P 7075 5775
@@
 $EndComp
 $Comp
-L GND #PWR038
+L power:GND #PWR038
 U 1 1 5A9543CD
 P 6275 4825
@@
 $EndComp
 $Comp
-L CRYSTAL_SMD X1
+L crf_1:CRYSTAL_SMD X1
 U 1 1 5A940C20
 P 6775 1775
 F 0 "X1" H 6775 1865 50  0000 C CNN
 F 1 "8m" H 6805 1665 50  0000 L CNN
-F 2 "Crystals:Crystal_SMD_5032_4Pads" H 6775 1775 60  0001 C CNN
+F 2 "Crystal:Crystal_SMD_5032-4Pin_5.0x3.2mm" H 6775 1775 60  0001 C CNN
 F 3 "" H 6775 1775 60  0000 C CNN
 F 4 "ABM3B-8.000MHZ-10-1-U-T" H 6775 1965 50  0001 C CNN "manf#"
@@
 	8825 975  8825 1025
 Wire Wire Line
-	8825 1025 9875 1025
+	8825 1025 9125 1025
 Wire Wire Line
 	9875 1025 9875 1175
@@
 	6825 5825 6725 5825
 Wire Wire Line
-	6825 5325 6825 6075
-Wire Wire Line
-	6075 5475 7075 5475
+	6825 5325 6825 5475
+Wire Wire Line
+	6075 5475 6825 5475
 Wire Wire Line
 	6075 5675 6325 5675
@@
 	6225 6075 6425 6075
 Wire Wire Line
-	7075 5325 7075 5775
-Wire Wire Line
-	6475 4825 6475 5375
+	7075 5325 7075 5475
+Wire Wire Line
+	6475 4825 6475 4875
 Wire Wire Line
 	6075 4675 6275 4675
@@
 	6075 4075 6275 4075
 Wire Wire Line
-	6075 1775 6575 1775
+	6075 1775 6425 1775
 Wire Wire Line
 	6525 1875 6075 1875
@@
 	6525 2175 6525 1875
 Wire Wire Line
-	7175 1675 7175 2175
+	7175 1675 7175 1775
 Wire Wire Line
 	6425 1675 6425 1775
@@
 	7175 1275 7175 1375
 Wire Wire Line
-	6425 1275 7425 1275
+	6425 1275 7175 1275
 Wire Wire Line
 	6075 2075 6225 2075
@@
 	6225 2075 6225 2150
 Wire Wire Line
-	6275 3925 6275 4375
+	6275 3925 6275 4075
 Wire Wire Line
 	6475 5375 6075 5375
@@
 	6825 4875 6825 5025
 Wire Wire Line
-	6475 4875 7075 4875
+	6475 4875 6825 4875
 Wire Wire Line
 	7075 4875 7075 5025
@@
 	6775 1875 6775 1975
 Wire Wire Line
-	8825 1625 9875 1625
-Wire Wire Line
-	6275 4675 6275 4825
-Connection ~ 9875 1025
+	8825 1625 9125 1625
+Wire Wire Line
+	6275 4675 6275 4775
+Wire Wire Line
+	9625 1025 9875 1025
+Wire Wire Line
+	9375 1025 9625 1025
+Wire Wire Line
+	9125 1025 9375 1025
+Wire Wire Line
+	9125 1625 9375 1625
+Wire Wire Line
+	9375 1625 9625 1625
+Wire Wire Line
+	9625 1625 9875 1625
+Wire Wire Line
+	6825 5825 6825 6075
+Wire Wire Line
+	6825 5475 6825 5825
+Wire Wire Line
+	6825 5475 7075 5475
+Wire Wire Line
+	6275 4775 6275 4825
+Wire Wire Line
+	6275 4275 6275 4375
+Wire Wire Line
+	6275 4175 6275 4275
+Wire Wire Line
+	6275 4075 6275 4175
+Wire Wire Line
+	7175 1775 7175 2175
+Wire Wire Line
+	6425 1775 6575 1775
+Wire Wire Line
+	7175 1275 7425 1275
+Wire Wire Line
+	6475 4875 6475 5375
+Wire Wire Line
+	6825 4875 7075 4875
+Wire Wire Line
+	7075 5475 7075 5775
 Connection ~ 9625 1025
 Connection ~ 9375 1025
@@
 Connection ~ 9375 1625
 Connection ~ 9625 1625
-Connection ~ 9875 1625
 Connection ~ 6825 5825
 Connection ~ 6825 5475

Commit message: Load KiCad 4.0.7 schematic symbols, footprints & 3D models
Parts:
- C10, C11, C12, C2, C3, C4, C5, C6, C7, C8, C9: footprint Capacitor_SMD:C_0603_1608Metric -> Capacitors_SMD:C_0603
- X1: footprint Crystal:Crystal_SMD_5032-4Pin_5.0x3.2mm -> Crystals:Crystal_SMD_5032_4Pads
Changed lines of the file:
@@
 F 0 "C4" H 6625 6175 50  0000 L CNN
 F 1 "2.2u" H 6625 5975 50  0000 L CNN
-F 2 "Capacitor_SMD:C_0603_1608Metric" H 6575 6075 60  0001 C CNN
+F 2 "Capacitors_SMD:C_0603" H 6575 6075 60  0001 C CNN
 F 3 "" H 6575 6075 60  0001 C CNN
 F 4 "C1608X5R1C225K080AB" H 6625 6275 50  0001 C CNN "manf#"
@@
 F 0 "C3" H 6625 5925 50  0000 L CNN
 F 1 "2.2u" H 6625 5725 50  0000 L CNN
-F 2 "Capacitor_SMD:C_0603_1608Metric" H 6575 5825 60  0001 C CNN
+F 2 "Capacitors_SMD:C_0603" H 6575 5825 60  0001 C CNN
 F 3 "" H 6575 5825 60  0001 C CNN
 F 4 "C1608X5R1C225K080AB" H 6625 6025 50  0001 C CNN "manf#"
@@
 F 0 "C2" H 6475 1625 50  0000 L CNN
 F 1 "15p" H 6475 1425 50  0000 L CNN
-F 2 "Capacitor_SMD:C_0603_1608Metric" H 6425 1525 60  0001 C CNN
+F 2 "Capacitors_SMD:C_0603" H 6425 1525 60  0001 C CNN
 F 3 "" H 6425 1525 60  0001 C CNN
 F 4 "06031A150JAT2A" H 6475 1725 50  0001 C CNN "manf#"
@@
 F 0 "C8" H 7225 1625 50  0000 L CNN
 F 1 "15p" H 7225 1425 50  0000 L CNN
-F 2 "Capacitor_SMD:C_0603_1608Metric" H 7175 1525 60  0001 C CNN
+F 2 "Capacitors_SMD:C_0603" H 7175 1525 60  0001 C CNN
 F 3 "" H 7175 1525 60  0001 C CNN
 F 4 "06031A150JAT2A" H 7225 1725 50  0001 C CNN "manf#"
@@
 F 0 "C5" H 6875 5275 50  0000 L CNN
 F 1 "2.2u" H 6875 5075 50  0000 L CNN
-F 2 "Capacitor_SMD:C_0603_1608Metric" H 6825 5175 60  0001 C CNN
+F 2 "Capacitors_SMD:C_0603" H 6825 5175 60  0001 C CNN
 F 3 "" H 6825 5175 60  0001 C CNN
 F 4 "C1608X5R1C225K080AB" H 6875 5375 50  0001 C CNN "manf#"
@@
 F 0 "C6" H 7125 5275 50  0000 L CNN
 F 1 "2.2u" H 7125 5075 50  0000 L CNN
-F 2 "Capacitor_SMD:C_0603_1608Metric" H 7075 5175 60  0001 C CNN
+F 2 "Capacitors_SMD:C_0603" H 7075 5175 60  0001 C CNN
 F 3 "" H 7075 5175 60  0001 C CNN
 F 4 "C1608X5R1C225K080AB" H 7125 5375 50  0001 C CNN "manf#"
@@
 F 0 "C7" H 7075 2830 50  0000 L BNN
 F 1 "100n" H 7075 2650 50  0000 L CNN
-F 2 "Capacitor_SMD:C_0603_1608Metric" H 7025 2750 60  0001 C CNN
+F 2 "Capacitors_SMD:C_0603" H 7025 2750 60  0001 C CNN
 F 3 "" H 7025 2750 60  0001 C CNN
 F 4 "C0603X104J5RACTU" H 7075 2930 50  0001 C CNN "manf#"
@@
 F 0 "C9" H 9175 1425 50  0000 L CNN
 F 1 "2.2u" H 9175 1225 50  0000 L CNN
-F 2 "Capacitor_SMD:C_0603_1608Metric" H 9125 1325 60  0001 C CNN
+F 2 "Capacitors_SMD:C_0603" H 9125 1325 60  0001 C CNN
 F 3 "" H 9125 1325 60  0001 C CNN
 F 4 "C1608X5R1C225K080AB" H 9175 1525 50  0001 C CNN "manf#"
@@
 F 0 "C10" H 9425 1425 50  0000 L CNN
 F 1 "2.2u" H 9425 1225 50  0000 L CNN
-F 2 "Capacitor_SMD:C_0603_1608Metric" H 9375 1325 60  0001 C CNN
+F 2 "Capacitors_SMD:C_0603" H 9375 1325 60  0001 C CNN
 F 3 "" H 9375 1325 60  0001 C CNN
 F 4 "C1608X5R1C225K080AB" H 9425 1525 50  0001 C CNN "manf#"
@@
 F 0 "C11" H 9675 1425 50  0000 L CNN
 F 1 "2.2u" H 9675 1225 50  0000 L CNN
-F 2 "Capacitor_SMD:C_0603_1608Metric" H 9625 1325 60  0001 C CNN
+F 2 "Capacitors_SMD:C_0603" H 9625 1325 60  0001 C CNN
 F 3 "" H 9625 1325 60  0001 C CNN
 F 4 "C1608X5R1C225K080AB" H 9675 1525 50  0001 C CNN "manf#"
@@
 F 0 "C12" H 9925 1425 50  0000 L CNN
 F 1 "2.2u" H 9925 1225 50  0000 L CNN
-F 2 "Capacitor_SMD:C_0603_1608Metric" H 9875 1325 60  0001 C CNN
+F 2 "Capacitors_SMD:C_0603" H 9875 1325 60  0001 C CNN
 F 3 "" H 9875 1325 60  0001 C CNN
 F 4 "C1608X5R1C225K080AB" H 9925 1525 50  0001 C CNN "manf#"
@@
 F 0 "X1" H 6775 1865 50  0000 C CNN
 F 1 "8m" H 6805 1665 50  0000 L CNN
-F 2 "Crystal:Crystal_SMD_5032-4Pin_5.0x3.2mm" H 6775 1775 60  0001 C CNN
+F 2 "Crystals:Crystal_SMD_5032_4Pads" H 6775 1775 60  0001 C CNN
 F 3 "" H 6775 1775 60  0000 C CNN
 F 4 "ABM3B-8.000MHZ-10-1-U-T" H 6775 1965 50  0001 C CNN "manf#"

Commit message: Design VESC6 plus sch done
Parts:
- Y1: renamed from X1; value 8m -> 8M; footprint Crystals:Crystal_SMD_5032_4Pads -> Crystals:Crystal_SMD_5032-4pin_5.0x3.2mm; symbol crf_1:CRYSTAL_SMD -> Device:Crystal_GND24
Connections:
- net labels added: CURR_FILTER_ON, PA15, PB2
- net labels removed: PB12, PB3, PB4, PD2
- wire segments 73 -> 78
- no-connect marks 5 -> 6
Changed lines of the file:
@@
 $Descr A4 11693 8268
 encoding utf-8
-Sheet 2 7
-Title "VESC 6.4"
-Date "2016-07-07"
+Sheet 2 6
+Title "VESC 6.5"
+Date "2018-02-27"
 Rev "A"
 Comp "Benjamin Vedder"
@@
 $EndComp
 $Comp
-L power:VCC #PWR028
+L power:VCC #PWR0121
 U 1 1 53F757C2
 P 6475 4825
-F 0 "#PWR028" H 6475 4925 30  0001 C CNN
+F 0 "#PWR0121" H 6475 4925 30  0001 C CNN
 F 1 "VCC" H 6475 4925 30  0000 C CNN
 F 2 "" H 6475 4825 60  0001 C CNN
@@
 $EndComp
 $Comp
-L power:VCC #PWR029
+L power:VCC #PWR0122
 U 1 1 53F757CE
 P 6275 3925
-F 0 "#PWR029" H 6275 4025 30  0001 C CNN
+F 0 "#PWR0122" H 6275 4025 30  0001 C CNN
 F 1 "VCC" H 6275 4025 30  0000 C CNN
 F 2 "" H 6275 3925 60  0001 C CNN
@@
 $EndComp
 $Comp
-L power:VCC #PWR030
+L power:VCC #PWR0123
 U 1 1 53F75807
 P 6275 5175
-F 0 "#PWR030" H 6275 5275 30  0001 C CNN
+F 0 "#PWR0123" H 6275 5275 30  0001 C CNN
 F 1 "VCC" H 6275 5275 30  0000 C CNN
 F 2 "" H 6275 5175 60  0001 C CNN
@@
 $EndComp
 $Comp
-L power:VCC #PWR031
+L power:VCC #PWR0124
 U 1 1 53F77441
 P 8825 975
-F 0 "#PWR031" H 8825 1075 30  0001 C CNN
+F 0 "#PWR0124" H 8825 1075 30  0001 C CNN
 F 1 "VCC" H 8825 1075 30  0000 C CNN
 F 2 "" H 8825 975 60  0001 C CNN
@@
 $EndComp
 $Comp
-L power:GND #PWR032
+L power:GND #PWR0125
 U 1 1 5A965081
 P 7025 3025
-F 0 "#PWR032" H 7025 2775 50  0001 C CNN
+F 0 "#PWR0125" H 7025 2775 50  0001 C CNN
 F 1 "GND" H 7025 2875 50  0000 C CNN
 F 2 "" H 7025 3025 50  0001 C CNN
@@
 $EndComp
 $Comp
-L power:GND #PWR033
+L power:GND #PWR0126
 U 1 1 5A965E92
-P 6775 1975
-F 0 "#PWR033" H 6775 1725 50  0001 C CNN
-F 1 "GND" H 6775 1825 50  0000 C CNN
-F 2 "" H 6775 1975 50  0001 C CNN
-F 3 "" H 6775 1975 50  0001 C CNN
-	1    6775 1975
+P 6850 2050
+F 0 "#PWR0126" H 6850 1800 50  0001 C CNN
+F 1 "GND" H 6850 1900 50  0000 C CNN
+F 2 "" H 6850 2050 50  0001 C CNN
+F 3 "" H 6850 2050 50  0001 C CNN
+	1    6850 2050
 	1    0    0    -1
 $EndComp
 $Comp
-L power:GND #PWR034
+L power:GND #PWR0127
 U 1 1 5A96886F
 P 7425 1350
-F 0 "#PWR034" H 7425 1100 50  0001 C CNN
+F 0 "#PWR0127" H 7425 1100 50  0001 C CNN
 F 1 "GND" H 7425 1200 50  0000 C CNN
 F 2 "" H 7425 1350 50  0001 C CNN
@@
 $EndComp
 $Comp
-L power:GND #PWR035
+L power:GND #PWR0128
 U 1 1 5A968FE6
 P 8825 1675
-F 0 "#PWR035" H 8825 1425 50  0001 C CNN
+F 0 "#PWR0128" H 8825 1425 50  0001 C CNN
 F 1 "GND" H 8825 1525 50  0000 C CNN
 F 2 "" H 8825 1675 50  0001 C CNN
@@
 $EndComp
 $Comp
-L power:GND #PWR036
+L power:GND #PWR0129
 U 1 1 5A96B952
-P 6225 2150
-F 0 "#PWR036" H 6225 1900 50  0001 C CNN
-F 1 "GND" H 6225 2000 50  0000 C CNN
-F 2 "" H 6225 2150 50  0001 C CNN
-F 3 "" H 6225 2150 50  0001 C CNN
-	1    6225 2150
+P 6450 2150
+F 0 "#PWR0129" H 6450 1900 50  0001 C CNN
+F 1 "GND" H 6450 2000 50  0000 C CNN
+F 2 "" H 6450 2150 50  0001 C CNN
+F 3 "" H 6450 2150 50  0001 C CNN
+	1    6450 2150
 	1    0    0    -1
 $EndComp
 $Comp
-L power:GND #PWR037
+L power:GND #PWR0130
 U 1 1 5A954317
 P 7075 5775
-F 0 "#PWR037" H 7075 5525 50  0001 C CNN
+F 0 "#PWR0130" H 7075 5525 50  0001 C CNN
 F 1 "GND" H 7075 5625 50  0000 C CNN
 F 2 "" H 7075 5775 50  0001 C CNN
@@
 $EndComp
 $Comp
-L power:GND #PWR038
+L power:GND #PWR0131
 U 1 1 5A9543CD
 P 6275 4825
-F 0 "#PWR038" H 6275 4575 50  0001 C CNN
+F 0 "#PWR0131" H 6275 4575 50  0001 C CNN
 F 1 "GND" H 6275 4675 50  0000 C CNN
 F 2 "" H 6275 4825 50  0001 C CNN
@@
 $EndComp
 $Comp
-L crf_1:CRYSTAL_SMD X1
+L Device:Crystal_GND24 Y1
 U 1 1 5A940C20
-P 6775 1775
-F 0 "X1" H 6775 1865 50  0000 C CNN
-F 1 "8m" H 6805 1665 50  0000 L CNN
-F 2 "Crystals:Crystal_SMD_5032_4Pads" H 6775 1775 60  0001 C CNN
-F 3 "" H 6775 1775 60  0000 C CNN
-F 4 "ABM3B-8.000MHZ-10-1-U-T" H 6775 1965 50  0001 C CNN "manf#"
-	1    6775 1775
+P 6850 1775
+F 0 "Y1" H 7000 1675 50  0000 C CNN
+F 1 "8M" H 6800 2075 50  0000 L CNN
+F 2 "Crystals:Crystal_SMD_5032-4pin_5.0x3.2mm" H 6850 1775 60  0001 C CNN
+F 3 "" H 6850 1775 60  0000 C CNN
+F 4 "ABM3B-8.000MHZ-10-1-U-T" H 6850 1965 50  0001 C CNN "manf#"
+	1    6850 1775
 	1    0    0    -1
 $EndComp
@@
 Text HLabel 3575 5275 0    60   Input ~ 0
 SPI3_SCK
-Text HLabel 3575 3775 0    60   Input ~ 0
-PB12
 Text Notes 9075 1725 0    40   ~ 0
 Bypass, place next to VDD pins
@@
 Text HLabel 3575 5175 0    60   Input ~ 0
 SPI3_CS
-Text HLabel 3575 5775 0    60   Input ~ 0
-PD2
-Text HLabel 6075 3025 2    60   Input ~ 0
-PB3
-Text HLabel 6075 3125 2    60   Input ~ 0
-PB4
+Text HLabel 3575 5775 0    60   Output ~ 0
+CURR_FILTER_ON
 Text HLabel 6075 2725 2    60   Input ~ 0
 SWDIO
@@
 	7425 1275 7425 1350
 Wire Wire Line
-	6975 1775 7175 1775
-Wire Wire Line
 	7025 2900 7025 3025
 Wire Wire Line
-	7175 2175 6525 2175
+	7175 2250 6575 2250
 Wire Wire Line
 	7025 2475 7025 2600
@@
 	6075 1775 6425 1775
 Wire Wire Line
-	6525 1875 6075 1875
-Wire Wire Line
-	6525 2175 6525 1875
+	6575 1875 6075 1875
+Wire Wire Line
+	6575 2250 6575 1875
 Wire Wire Line
 	7175 1675 7175 1775
@@
 	6425 1275 7175 1275
 Wire Wire Line
-	6075 2075 6225 2075
-Wire Wire Line
-	6225 2075 6225 2150
+	6450 2075 6450 2150
 Wire Wire Line
 	6275 3925 6275 4075
@@
 	6075 5175 6275 5175
 Wire Wire Line
-	6775 1875 6775 1975
-Wire Wire Line
 	8825 1625 9125 1625
 Wire Wire Line
@@
 	6275 4075 6275 4175
 Wire Wire Line
-	7175 1775 7175 2175
-Wire Wire Line
-	6425 1775 6575 1775
+	7175 1775 7175 2250
 Wire Wire Line
 	7175 1275 7425 1275
@@
 Connection ~ 6275 4075
 Connection ~ 7175 1775
-Connection ~ 6425 1775
 Connection ~ 7175 1275
 Connection ~ 6475 4875
 Connection ~ 6825 4875
 Connection ~ 7075 5475
-NoConn ~ 6075 2175
-NoConn ~ 6075 2925
 NoConn ~ 6075 1475
 NoConn ~ 6075 1575
 NoConn ~ 3575 5575
+NoConn ~ 3575 3775
+Text HLabel 6075 2925 2    60   Input ~ 0
+PA15
+NoConn ~ 6075 3025
+NoConn ~ 6075 3125
+Text HLabel 6075 2175 2    60   Input ~ 0
+PB2
+Wire Wire Line
+	6075 2075 6450 2075
+Wire Wire Line
+	6425 1775 6700 1775
+Wire Wire Line
+	7000 1775 7175 1775
+Wire Wire Line
+	6850 2050 6850 2025
+Wire Wire Line
+	6850 1575 6850 1525
+Wire Wire Line
+	6850 1525 6675 1525
+Wire Wire Line
+	6675 1525 6675 2025
+Wire Wire Line
+	6675 2025 6850 2025
+Connection ~ 6850 2025
+Wire Wire Line
+	6850 2025 6850 1975
+Connection ~ 6425 1775
 $EndSCHEMATC
