File: design/MCU.sch (KiCad schematic (older format))
At the start: 13 parts, among them U1 STM32F40X_LQFP64, X1 8m

Commit message: Update C2/C8/C51/C52 BOM(06035A150GAT2A)
Parts:
- C2, C8: manf# 06031A150JAT2A -> 06035A150GAT2A
Changed lines of the file:
@@
 EESchema Schematic File Version 4
-LIBS:VESC_6-cache
 EELAYER 30 0
 EELAYER END
@@
 F 2 "Capacitors_SMD:C_0603" H 6425 1525 60  0001 C CNN
 F 3 "" H 6425 1525 60  0001 C CNN
-F 4 "06031A150JAT2A" H 6475 1725 50  0001 C CNN "manf#"
+F 4 "06035A150GAT2A" H 6475 1725 50  0001 C CNN "manf#"
 	1    6425 1525
 	-1   0    0    -1
@@
 F 2 "Capacitors_SMD:C_0603" H 7175 1525 60  0001 C CNN
 F 3 "" H 7175 1525 60  0001 C CNN
-F 4 "06031A150JAT2A" H 7225 1725 50  0001 C CNN "manf#"
+F 4 "06035A150GAT2A" H 7225 1725 50  0001 C CNN "manf#"
 	1    7175 1525
 	-1   0    0    -1
