File: design/mpu9250.sch (KiCad schematic (older format))
At the start: 4 parts, among them U10 MPU9250

Commit message: Regenerate Gerber
Parts:
- added R40, R41: 1k, Resistors_SMD:R_0603, symbol R
Connections:
- wire segments 18 -> 27
- no-connect marks 4 -> 6
Changed lines of the file:
@@
 $EndDescr
-$Comp
-L MPU9250 U10
-U 1 1 5A8CD83F
-P 4425 3800
-F 0 "U10" H 4350 4625 50  0000 L BNN
-F 1 "MPU9250" H 4250 2900 50  0000 L BNN
-F 2 "Housings_DFN_QFN:QFN-24_3x3mm_Pitch0.4mm" H 3400 4725 50  0001 L BNN
-F 3 "" H 3400 4725 50  0001 L BNN
-	1    4425 3800
-	1    0    0    -1
-$EndComp
 $Comp
 L GND #PWR093
 U 1 1 5A8CDBDA
-P 3500 4450
-F 0 "#PWR093" H 3500 4200 50  0001 C CNN
-F 1 "GND" H 3500 4300 50  0000 C CNN
-F 2 "" H 3500 4450 50  0001 C CNN
-F 3 "" H 3500 4450 50  0001 C CNN
-	1    3500 4450
-	1    0    0    -1
-$EndComp
-$Comp
-L VCC #PWR094
-U 1 1 5A8CDC21
-P 3350 4075
-F 0 "#PWR094" H 3350 3925 50  0001 C CNN
-F 1 "VCC" H 3350 4225 50  0000 C CNN
-F 2 "" H 3350 4075 50  0001 C CNN
-F 3 "" H 3350 4075 50  0001 C CNN
-	1    3350 4075
+P 3675 3850
+F 0 "#PWR093" H 3675 3600 50  0001 C CNN
+F 1 "GND" H 3675 3700 50  0000 C CNN
+F 2 "" H 3675 3850 50  0001 C CNN
+F 3 "" H 3675 3850 50  0001 C CNN
+	1    3675 3850
 	1    0    0    -1
 $EndComp
@@
 $EndComp
 $Comp
-L VCC #PWR095
+L VCC #PWR094
 U 1 1 5A8CE66F
 P 5550 3000
-F 0 "#PWR095" H 5550 2850 50  0001 C CNN
+F 0 "#PWR094" H 5550 2850 50  0001 C CNN
 F 1 "VCC" H 5550 3150 50  0000 C CNN
 F 2 "" H 5550 3000 50  0001 C CNN
@@
 $EndComp
 $Comp
-L GND #PWR096
+L GND #PWR095
 U 1 1 5A8CE6B3
 P 5150 4600
-F 0 "#PWR096" H 5150 4350 50  0001 C CNN
+F 0 "#PWR095" H 5150 4350 50  0001 C CNN
 F 1 "GND" H 5150 4450 50  0000 C CNN
 F 2 "" H 5150 4600 50  0001 C CNN
@@
 	1    0    0    -1
 $EndComp
-Text HLabel 3875 4400 0    60   Input ~ 0
-SCL
-Text HLabel 3875 4500 0    60   Input ~ 0
-SDA
 NoConn ~ 3875 3200
 NoConn ~ 3875 3900
@@
 	-1   0    0    -1
 $EndComp
+$Comp
+L VCC #PWR096
+U 1 1 5AF1D016
+P 3125 3850
+F 0 "#PWR096" H 3125 3700 50  0001 C CNN
+F 1 "VCC" H 3125 4000 50  0000 C CNN
+F 2 "" H 3125 3850 50  0001 C CNN
+F 3 "" H 3125 3850 50  0001 C CNN
+	1    3125 3850
+	1    0    0    -1
+$EndComp
+$Comp
+L R R40
+U 1 1 5AF1D017
+P 3125 4175
+F 0 "R40" V 3025 4275 50  0000 C CNN
+F 1 "1k" V 3025 4075 50  0000 C CNN
+F 2 "Resistors_SMD:R_0603" V 3055 4175 50  0001 C CNN
+F 3 "" H 3125 4175 50  0001 C CNN
+F 4 "CR0603-FX-1001ELF" H 3025 4375 50  0001 C CNN "manf#"
+	1    3125 4175
+	1    0    0    -1
+$EndComp
+$Comp
+L R R41
+U 1 1 5AF1D018
+P 3375 4175
+F 0 "R41" V 3275 4275 50  0000 C CNN
+F 1 "1k" V 3275 4075 50  0000 C CNN
+F 2 "Resistors_SMD:R_0603" V 3305 4175 50  0001 C CNN
+F 3 "" H 3375 4175 50  0001 C CNN
+F 4 "CR0603-FX-1001ELF" H 3275 4375 50  0001 C CNN "manf#"
+	1    3375 4175
+	1    0    0    -1
+$EndComp
+$Comp
+L VCC #PWR097
+U 1 1 5AF1D01C
+P 5550 3000
+F 0 "#PWR097" H 5550 2850 50  0001 C CNN
+F 1 "VCC" H 5550 3150 50  0000 C CNN
+F 2 "" H 5550 3000 50  0001 C CNN
+F 3 "" H 5550 3000 50  0001 C CNN
+	1    5550 3000
+	1    0    0    -1
+$EndComp
+Text HLabel 2950 4400 0    60   Input ~ 0
+SCL
+Text HLabel 2950 4500 0    60   Input ~ 0
+SDA
+NoConn ~ 3875 3900
+NoConn ~ 3875 3400
+$Comp
+L MPU9250 U10
+U 1 1 5A8CD83F
+P 4425 3800
+F 0 "U10" H 4350 4625 50  0000 L BNN
+F 1 "MPU9250" H 4250 2900 50  0000 L BNN
+F 2 "Housings_DFN_QFN:QFN-24_3x3mm_Pitch0.4mm" H 3400 4725 50  0001 L BNN
+F 3 "" H 3400 4725 50  0001 L BNN
+	1    4425 3800
+	1    0    0    -1
+$EndComp
 Wire Wire Line
 	4975 3200 5350 3200
-Wire Wire Line
-	5350 3100 5350 3950
 Wire Wire Line
 	4975 4500 5550 4500
@@
 	4975 3100 5550 3100
 Wire Wire Line
-	4975 3300 5550 3300
-Wire Wire Line
 	5150 3800 4975 3800
 Wire Wire Line
-	5150 3800 5150 3950
-Wire Wire Line
-	5150 4250 5150 4600
-Wire Wire Line
-	3875 3800 3500 3800
-Wire Wire Line
-	3500 3800 3500 4450
-Wire Wire Line
-	3875 4200 3500 4200
-Connection ~ 3500 4200
-Wire Wire Line
-	3875 4300 3350 4300
-Wire Wire Line
-	3350 4300 3350 4075
+	3675 3800 3875 3800
+Wire Wire Line
+	3875 4200 3800 4200
+Wire Wire Line
+	3525 4300 3875 4300
 Wire Wire Line
 	4975 4400 5150 4400
-Wire Wire Line
-	5350 4250 5350 4500
 Connection ~ 5350 4500
 Connection ~ 5350 3300
@@
 	5550 3100 5550 3000
 Wire Wire Line
+	5550 4500 5550 4250
+Wire Wire Line
+	2950 4500 3875 4500
+Wire Wire Line
+	3375 4500 3375 4325
+Wire Wire Line
+	3125 3850 3125 4025
+Wire Wire Line
+	3125 3925 3525 3925
+Wire Wire Line
+	3375 3925 3375 4025
+Wire Wire Line
+	2950 4400 3875 4400
+Wire Wire Line
+	3125 4400 3125 4325
+Wire Wire Line
+	5150 4500 5350 4500
+Connection ~ 3125 3925
+Connection ~ 3125 4400
+Connection ~ 3375 4500
+Wire Wire Line
+	5350 3100 5350 3950
+Wire Wire Line
 	5550 3300 5550 3950
 Wire Wire Line
-	5550 4500 5550 4250
+	5150 4250 5150 4600
+Wire Wire Line
+	5150 3800 5150 3950
+Wire Wire Line
+	4975 3300 5550 3300
+Wire Wire Line
+	5350 4500 5350 4250
+Wire Wire Line
+	3525 3925 3525 4300
+Connection ~ 3375 3925
+Wire Wire Line
+	3800 4200 3800 3800
+Wire Wire Line
+	3675 3800 3675 3850
+Connection ~ 3800 3800
 $EndSCHEMATC

Commit message: MPU9250: add part number field
Parts:
- U10: manf# (none) -> MPU-9250
Changed lines of the file:
@@
 F 2 "Housings_DFN_QFN:QFN-24_3x3mm_Pitch0.4mm" H 3400 4725 50  0001 L BNN
 F 3 "" H 3400 4725 50  0001 L BNN
+F 4 "MPU-9250" H 4425 3800 60  0001 C CNN "manf#"
 	1    4425 3800
 	1    0    0    -1

Commit message: Support KiCad 5.1.4
Parts:
- C60, C61, C62: footprint Capacitors_SMD:C_0603 -> Capacitor_SMD:C_0603_1608Metric; symbol C -> Device:C
- R40, R41: footprint Resistors_SMD:R_0603 -> Resistor_SMD:R_0603_1608Metric; symbol R -> Device:R
- U10: footprint Housings_DFN_QFN:QFN-24_3x3mm_Pitch0.4mm -> Package_DFN_QFN:QFN-24-1EP_3x3mm_P0.4mm_EP1.75x1.6mm; symbol MPU9250 -> crf_1:MPU9250
Connections:
- wire segments 27 -> 39
- no-connect marks 6 -> 4
Changed lines of the file:
@@
-EESchema Schematic File Version 2
-LIBS:power
-LIBS:device
-LIBS:transistors
-LIBS:conn
-LIBS:linear
-LIBS:regul
-LIBS:74xx
-LIBS:cmos4000
-LIBS:adc-dac
-LIBS:memory
-LIBS:xilinx
-LIBS:microcontrollers
-LIBS:dsp
-LIBS:microchip
-LIBS:analog_switches
-LIBS:motorola
-LIBS:texas
-LIBS:switches
-LIBS:intel
-LIBS:audio
-LIBS:interface
-LIBS:digital-audio
-LIBS:philips
-LIBS:display
-LIBS:cypress
-LIBS:siliconi
-LIBS:opto
-LIBS:atmel
-LIBS:contrib
-LIBS:valves
-LIBS:crf_1
+EESchema Schematic File Version 4
 LIBS:VESC_6-cache
-EELAYER 25 0
+EELAYER 30 0
 EELAYER END
 $Descr A4 11693 8268
@@
 $EndDescr
 $Comp
-L GND #PWR093
+L power:GND #PWR093
 U 1 1 5A8CDBDA
 P 3675 3850
@@
 $EndComp
 $Comp
-L C C61
+L Device:C C61
 U 1 1 5A8CE4DF
 P 5350 4100
 F 0 "C61" H 5175 4000 50  0000 L CNN
 F 1 "2.2u" H 5175 4200 50  0000 L CNN
-F 2 "Capacitors_SMD:C_0603" H 5388 3950 50  0001 C CNN
+F 2 "Capacitor_SMD:C_0603_1608Metric" H 5388 3950 50  0001 C CNN
 F 3 "" H 5350 4100 50  0001 C CNN
 F 4 "C1608X5R1C225K080AB" H 5175 4100 50  0001 C CNN "manf#"
@@
 $EndComp
 $Comp
-L VCC #PWR094
+L power:VCC #PWR094
 U 1 1 5A8CE66F
 P 5550 3000
@@
 $EndComp
 $Comp
-L GND #PWR095
+L power:GND #PWR095
 U 1 1 5A8CE6B3
 P 5150 4600
@@
 	1    0    0    -1
 $EndComp
-NoConn ~ 3875 3200
-NoConn ~ 3875 3900
-NoConn ~ 3875 3400
-NoConn ~ 3875 3100
-$Comp
-L C C62
+$Comp
+L Device:C C62
 U 1 1 5A8CE506
 P 5550 4100
 F 0 "C62" H 5375 4000 50  0000 L CNN
 F 1 "2.2u" H 5375 4200 50  0000 L CNN
-F 2 "Capacitors_SMD:C_0603" H 5588 3950 50  0001 C CNN
+F 2 "Capacitor_SMD:C_0603_1608Metric" H 5588 3950 50  0001 C CNN
 F 3 "" H 5550 4100 50  0001 C CNN
 F 4 "C1608X5R1C225K080AB" H 5375 4100 50  0001 C CNN "manf#"
@@
 $EndComp
 $Comp
-L C C60
+L Device:C C60
 U 1 1 5A8CE80E
 P 5150 4100
 F 0 "C60" H 5175 4000 50  0000 L CNN
 F 1 "100n" H 5175 4200 50  0000 L CNN
-F 2 "Capacitors_SMD:C_0603" H 5188 3950 50  0001 C CNN
+F 2 "Capacitor_SMD:C_0603_1608Metric" H 5188 3950 50  0001 C CNN
 F 3 "" H 5150 4100 50  0001 C CNN
 F 4 "C0603X104J5RACTU" H 4975 4100 50  0001 C CNN "manf#"
@@
 $EndComp
 $Comp
-L VCC #PWR096
+L power:VCC #PWR096
 U 1 1 5AF1D016
 P 3125 3850
@@
 $EndComp
 $Comp
-L R R40
+L Device:R R40
 U 1 1 5AF1D017
 P 3125 4175
 F 0 "R40" V 3025 4275 50  0000 C CNN
 F 1 "1k" V 3025 4075 50  0000 C CNN
-F 2 "Resistors_SMD:R_0603" V 3055 4175 50  0001 C CNN
+F 2 "Resistor_SMD:R_0603_1608Metric" V 3055 4175 50  0001 C CNN
 F 3 "" H 3125 4175 50  0001 C CNN
 F 4 "CR0603-FX-1001ELF" H 3025 4375 50  0001 C CNN "manf#"
@@
 $EndComp
 $Comp
-L R R41
+L Device:R R41
 U 1 1 5AF1D018
 P 3375 4175
 F 0 "R41" V 3275 4275 50  0000 C CNN
 F 1 "1k" V 3275 4075 50  0000 C CNN
-F 2 "Resistors_SMD:R_0603" V 3305 4175 50  0001 C CNN
+F 2 "Resistor_SMD:R_0603_1608Metric" V 3305 4175 50  0001 C CNN
 F 3 "" H 3375 4175 50  0001 C CNN
 F 4 "CR0603-FX-1001ELF" H 3275 4375 50  0001 C CNN "manf#"
@@
 $EndComp
 $Comp
-L VCC #PWR097
+L power:VCC #PWR097
 U 1 1 5AF1D01C
 P 5550 3000
@@
 	1    0    0    -1
 $EndComp
+$Comp
+L crf_1:MPU9250 U10
+U 1 1 5A8CD83F
+P 4425 3800
+F 0 "U10" H 4350 4625 50  0000 L BNN
+F 1 "MPU9250" H 4250 2900 50  0000 L BNN
+F 2 "Package_DFN_QFN:QFN-24-1EP_3x3mm_P0.4mm_EP1.75x1.6mm" H 3400 4725 50  0001 L BNN
+F 3 "" H 3400 4725 50  0001 L BNN
+F 4 "MPU-9250" H 4425 3800 60  0001 C CNN "manf#"
+	1    4425 3800
+	1    0    0    -1
+$EndComp
 Text HLabel 2950 4400 0    60   Input ~ 0
 SCL
 Text HLabel 2950 4500 0    60   Input ~ 0
 SDA
-NoConn ~ 3875 3900
-NoConn ~ 3875 3400
-$Comp
-L MPU9250 U10
-U 1 1 5A8CD83F
-P 4425 3800
-F 0 "U10" H 4350 4625 50  0000 L BNN
-F 1 "MPU9250" H 4250 2900 50  0000 L BNN
-F 2 "Housings_DFN_QFN:QFN-24_3x3mm_Pitch0.4mm" H 3400 4725 50  0001 L BNN
-F 3 "" H 3400 4725 50  0001 L BNN
-F 4 "MPU-9250" H 4425 3800 60  0001 C CNN "manf#"
-	1    4425 3800
-	1    0    0    -1
-$EndComp
 Wire Wire Line
 	4975 3200 5350 3200
 Wire Wire Line
-	4975 4500 5550 4500
+	4975 4500 5150 4500
+Wire Wire Line
+	4975 3100 5350 3100
+Wire Wire Line
+	5150 3800 4975 3800
+Wire Wire Line
+	3675 3800 3800 3800
+Wire Wire Line
+	3875 4200 3800 4200
+Wire Wire Line
+	3525 4300 3875 4300
+Wire Wire Line
+	4975 4400 5150 4400
+Wire Wire Line
+	5550 3100 5550 3000
+Wire Wire Line
+	5550 4500 5550 4250
+Wire Wire Line
+	2950 4500 3375 4500
+Wire Wire Line
+	3375 4500 3375 4325
+Wire Wire Line
+	3125 3850 3125 3925
+Wire Wire Line
+	3125 3925 3375 3925
+Wire Wire Line
+	3375 3925 3375 4025
+Wire Wire Line
+	2950 4400 3125 4400
+Wire Wire Line
+	3125 4400 3125 4325
+Wire Wire Line
+	5150 4500 5350 4500
+Wire Wire Line
+	5350 3100 5350 3200
+Wire Wire Line
+	5550 3300 5550 3950
+Wire Wire Line
+	5150 4250 5150 4400
+Wire Wire Line
+	5150 3800 5150 3950
+Wire Wire Line
+	4975 3300 5350 3300
+Wire Wire Line
+	5350 4500 5350 4250
+Wire Wire Line
+	3525 3925 3525 4300
+Wire Wire Line
+	3800 4200 3800 3800
+Wire Wire Line
+	3675 3800 3675 3850
 Connection ~ 5150 4500
 Connection ~ 5150 4400
-Wire Wire Line
-	4975 3100 5550 3100
-Wire Wire Line
-	5150 3800 4975 3800
-Wire Wire Line
-	3675 3800 3875 3800
-Wire Wire Line
-	3875 4200 3800 4200
-Wire Wire Line
-	3525 4300 3875 4300
-Wire Wire Line
-	4975 4400 5150 4400
 Connection ~ 5350 4500
 Connection ~ 5350 3300
 Connection ~ 5350 3100
 Connection ~ 5350 3200
-Wire Wire Line
-	5550 3100 5550 3000
-Wire Wire Line
-	5550 4500 5550 4250
-Wire Wire Line
-	2950 4500 3875 4500
-Wire Wire Line
-	3375 4500 3375 4325
-Wire Wire Line
-	3125 3850 3125 4025
-Wire Wire Line
-	3125 3925 3525 3925
-Wire Wire Line
-	3375 3925 3375 4025
-Wire Wire Line
-	2950 4400 3875 4400
-Wire Wire Line
-	3125 4400 3125 4325
-Wire Wire Line
-	5150 4500 5350 4500
 Connection ~ 3125 3925
 Connection ~ 3125 4400
 Connection ~ 3375 4500
-Wire Wire Line
-	5350 3100 5350 3950
-Wire Wire Line
-	5550 3300 5550 3950
-Wire Wire Line
-	5150 4250 5150 4600
-Wire Wire Line
-	5150 3800 5150 3950
-Wire Wire Line
-	4975 3300 5550 3300
-Wire Wire Line
-	5350 4500 5350 4250
-Wire Wire Line
-	3525 3925 3525 4300
 Connection ~ 3375 3925
-Wire Wire Line
-	3800 4200 3800 3800
-Wire Wire Line
-	3675 3800 3675 3850
 Connection ~ 3800 3800
+NoConn ~ 3875 3200
+NoConn ~ 3875 3900
+NoConn ~ 3875 3400
+NoConn ~ 3875 3100
+Wire Wire Line
+	5150 4500 5150 4600
+Wire Wire Line
+	5150 4400 5150 4500
+Wire Wire Line
+	5350 4500 5550 4500
+Wire Wire Line
+	5350 3300 5350 3950
+Wire Wire Line
+	5350 3300 5550 3300
+Wire Wire Line
+	5350 3100 5550 3100
+Wire Wire Line
+	5350 3200 5350 3300
+Wire Wire Line
+	3125 3925 3125 4025
+Wire Wire Line
+	3125 4400 3875 4400
+Wire Wire Line
+	3375 4500 3875 4500
+Wire Wire Line
+	3375 3925 3525 3925
+Wire Wire Line
+	3800 3800 3875 3800
 $EndSCHEMATC

Commit message: Load KiCad 4.0.7 schematic symbols, footprints & 3D models
Parts:
- C60, C61, C62: footprint Capacitor_SMD:C_0603_1608Metric -> Capacitors_SMD:C_0603
- R40, R41: footprint Resistor_SMD:R_0603_1608Metric -> Resistors_SMD:R_0603
- U10: footprint Package_DFN_QFN:QFN-24-1EP_3x3mm_P0.4mm_EP1.75x1.6mm -> Housings_DFN_QFN:QFN-24_3x3mm_Pitch0.4mm
Changed lines of the file:
@@
 F 0 "C61" H 5175 4000 50  0000 L CNN
 F 1 "2.2u" H 5175 4200 50  0000 L CNN
-F 2 "Capacitor_SMD:C_0603_1608Metric" H 5388 3950 50  0001 C CNN
+F 2 "Capacitors_SMD:C_0603" H 5388 3950 50  0001 C CNN
 F 3 "" H 5350 4100 50  0001 C CNN
 F 4 "C1608X5R1C225K080AB" H 5175 4100 50  0001 C CNN "manf#"
@@
 F 0 "C62" H 5375 4000 50  0000 L CNN
 F 1 "2.2u" H 5375 4200 50  0000 L CNN
-F 2 "Capacitor_SMD:C_0603_1608Metric" H 5588 3950 50  0001 C CNN
+F 2 "Capacitors_SMD:C_0603" H 5588 3950 50  0001 C CNN
 F 3 "" H 5550 4100 50  0001 C CNN
 F 4 "C1608X5R1C225K080AB" H 5375 4100 50  0001 C CNN "manf#"
@@
 F 0 "C60" H 5175 4000 50  0000 L CNN
 F 1 "100n" H 5175 4200 50  0000 L CNN
-F 2 "Capacitor_SMD:C_0603_1608Metric" H 5188 3950 50  0001 C CNN
+F 2 "Capacitors_SMD:C_0603" H 5188 3950 50  0001 C CNN
 F 3 "" H 5150 4100 50  0001 C CNN
 F 4 "C0603X104J5RACTU" H 4975 4100 50  0001 C CNN "manf#"
@@
 F 0 "R40" V 3025 4275 50  0000 C CNN
 F 1 "1k" V 3025 4075 50  0000 C CNN
-F 2 "Resistor_SMD:R_0603_1608Metric" V 3055 4175 50  0001 C CNN
+F 2 "Resistors_SMD:R_0603" V 3055 4175 50  0001 C CNN
 F 3 "" H 3125 4175 50  0001 C CNN
 F 4 "CR0603-FX-1001ELF" H 3025 4375 50  0001 C CNN "manf#"
@@
 F 0 "R41" V 3275 4275 50  0000 C CNN
 F 1 "1k" V 3275 4075 50  0000 C CNN
-F 2 "Resistor_SMD:R_0603_1608Metric" V 3305 4175 50  0001 C CNN
+F 2 "Resistors_SMD:R_0603" V 3305 4175 50  0001 C CNN
 F 3 "" H 3375 4175 50  0001 C CNN
 F 4 "CR0603-FX-1001ELF" H 3275 4375 50  0001 C CNN "manf#"
@@
 F 0 "U10" H 4350 4625 50  0000 L BNN
 F 1 "MPU9250" H 4250 2900 50  0000 L BNN
-F 2 "Package_DFN_QFN:QFN-24-1EP_3x3mm_P0.4mm_EP1.75x1.6mm" H 3400 4725 50  0001 L BNN
+F 2 "Housings_DFN_QFN:QFN-24_3x3mm_Pitch0.4mm" H 3400 4725 50  0001 L BNN
 F 3 "" H 3400 4725 50  0001 L BNN
 F 4 "MPU-9250" H 4425 3800 60  0001 C CNN "manf#"
@@
 Wire Wire Line
 	3675 3800 3675 3850
+Wire Wire Line
+	5150 4500 5150 4600
+Wire Wire Line
+	5150 4400 5150 4500
+Wire Wire Line
+	5350 4500 5550 4500
+Wire Wire Line
+	5350 3300 5350 3950
+Wire Wire Line
+	5350 3300 5550 3300
+Wire Wire Line
+	5350 3100 5550 3100
+Wire Wire Line
+	5350 3200 5350 3300
+Wire Wire Line
+	3125 3925 3125 4025
+Wire Wire Line
+	3125 4400 3875 4400
+Wire Wire Line
+	3375 4500 3875 4500
+Wire Wire Line
+	3375 3925 3525 3925
+Wire Wire Line
+	3800 3800 3875 3800
 Connection ~ 5150 4500
 Connection ~ 5150 4400
@@
 NoConn ~ 3875 3400
 NoConn ~ 3875 3100
-Wire Wire Line
-	5150 4500 5150 4600
-Wire Wire Line
-	5150 4400 5150 4500
-Wire Wire Line
-	5350 4500 5550 4500
-Wire Wire Line
-	5350 3300 5350 3950
-Wire Wire Line
-	5350 3300 5550 3300
-Wire Wire Line
-	5350 3100 5550 3100
-Wire Wire Line
-	5350 3200 5350 3300
-Wire Wire Line
-	3125 3925 3125 4025
-Wire Wire Line
-	3125 4400 3875 4400
-Wire Wire Line
-	3375 4500 3875 4500
-Wire Wire Line
-	3375 3925 3525 3925
-Wire Wire Line
-	3800 3800 3875 3800
 $EndSCHEMATC

Commit message: Design VESC6 plus sch done
Parts:
- removed R40, R41: 1k, Resistors_SMD:R_0603, symbol Device:R
- renumbered C60 to C49, C61 to C50, C62 to C51, U10 to U9
Connections:
- wire segments 39 -> 27
Changed lines of the file:
@@
 $Descr A4 11693 8268
 encoding utf-8
-Sheet 7 7
-Title "VESC 6.4"
-Date "2016-07-07"
+Sheet 4 6
+Title "VESC 6.5"
+Date "2018-02-27"
 Rev "A"
 Comp "Benjamin Vedder"
@@
 $EndDescr
 $Comp
-L power:GND #PWR093
+L power:GND #PWR0108
 U 1 1 5A8CDBDA
 P 3675 3850
-F 0 "#PWR093" H 3675 3600 50  0001 C CNN
+F 0 "#PWR0108" H 3675 3600 50  0001 C CNN
 F 1 "GND" H 3675 3700 50  0000 C CNN
 F 2 "" H 3675 3850 50  0001 C CNN
@@
 $EndComp
 $Comp
-L Device:C C61
+L Device:C C50
 U 1 1 5A8CE4DF
 P 5350 4100
-F 0 "C61" H 5175 4000 50  0000 L CNN
+F 0 "C50" H 5200 4000 50  0000 L CNN
 F 1 "2.2u" H 5175 4200 50  0000 L CNN
 F 2 "Capacitors_SMD:C_0603" H 5388 3950 50  0001 C CNN
@@
 F 4 "C1608X5R1C225K080AB" H 5175 4100 50  0001 C CNN "manf#"
 	1    5350 4100
-	1    0    0    -1
+	-1   0    0    1
 $EndComp
 $Comp
-L power:VCC #PWR094
-U 1 1 5A8CE66F
-P 5550 3000
-F 0 "#PWR094" H 5550 2850 50  0001 C CNN
-F 1 "VCC" H 5550 3150 50  0000 C CNN
-F 2 "" H 5550 3000 50  0001 C CNN
-F 3 "" H 5550 3000 50  0001 C CNN
-	1    5550 3000
-	1    0    0    -1
-$EndComp
-$Comp
-L power:GND #PWR095
+L power:GND #PWR0110
 U 1 1 5A8CE6B3
 P 5150 4600
-F 0 "#PWR095" H 5150 4350 50  0001 C CNN
+F 0 "#PWR0110" H 5150 4350 50  0001 C CNN
 F 1 "GND" H 5150 4450 50  0000 C CNN
 F 2 "" H 5150 4600 50  0001 C CNN
@@
 $EndComp
 $Comp
-L Device:C C62
+L Device:C C51
 U 1 1 5A8CE506
 P 5550 4100
-F 0 "C62" H 5375 4000 50  0000 L CNN
+F 0 "C51" H 5400 4000 50  0000 L CNN
 F 1 "2.2u" H 5375 4200 50  0000 L CNN
 F 2 "Capacitors_SMD:C_0603" H 5588 3950 50  0001 C CNN
@@
 F 4 "C1608X5R1C225K080AB" H 5375 4100 50  0001 C CNN "manf#"
 	1    5550 4100
+	-1   0    0    1
+$EndComp
+$Comp
+L power:VCC #PWR0111
+U 1 1 5AF1D016
+P 3525 3925
+F 0 "#PWR0111" H 3525 3775 50  0001 C CNN
+F 1 "VCC" H 3525 4075 50  0000 C CNN
+F 2 "" H 3525 3925 50  0001 C CNN
+F 3 "" H 3525 3925 50  0001 C CNN
+	1    3525 3925
 	1    0    0    -1
 $EndComp
 $Comp
-L Device:C C60
-U 1 1 5A8CE80E
-P 5150 4100
-F 0 "C60" H 5175 4000 50  0000 L CNN
-F 1 "100n" H 5175 4200 50  0000 L CNN
-F 2 "Capacitors_SMD:C_0603" H 5188 3950 50  0001 C CNN
-F 3 "" H 5150 4100 50  0001 C CNN
-F 4 "C0603X104J5RACTU" H 4975 4100 50  0001 C CNN "manf#"
-	1    5150 4100
-	-1   0    0    -1
-$EndComp
-$Comp
-L power:VCC #PWR096
-U 1 1 5AF1D016
-P 3125 3850
-F 0 "#PWR096" H 3125 3700 50  0001 C CNN
-F 1 "VCC" H 3125 4000 50  0000 C CNN
-F 2 "" H 3125 3850 50  0001 C CNN
-F 3 "" H 3125 3850 50  0001 C CNN
-	1    3125 3850
-	1    0    0    -1
-$EndComp
-$Comp
-L Device:R R40
-U 1 1 5AF1D017
-P 3125 4175
-F 0 "R40" V 3025 4275 50  0000 C CNN
-F 1 "1k" V 3025 4075 50  0000 C CNN
-F 2 "Resistors_SMD:R_0603" V 3055 4175 50  0001 C CNN
-F 3 "" H 3125 4175 50  0001 C CNN
-F 4 "CR0603-FX-1001ELF" H 3025 4375 50  0001 C CNN "manf#"
-	1    3125 4175
-	1    0    0    -1
-$EndComp
-$Comp
-L Device:R R41
-U 1 1 5AF1D018
-P 3375 4175
-F 0 "R41" V 3275 4275 50  0000 C CNN
-F 1 "1k" V 3275 4075 50  0000 C CNN
-F 2 "Resistors_SMD:R_0603" V 3305 4175 50  0001 C CNN
-F 3 "" H 3375 4175 50  0001 C CNN
-F 4 "CR0603-FX-1001ELF" H 3275 4375 50  0001 C CNN "manf#"
-	1    3375 4175
-	1    0    0    -1
-$EndComp
-$Comp
-L power:VCC #PWR097
-U 1 1 5AF1D01C
-P 5550 3000
-F 0 "#PWR097" H 5550 2850 50  0001 C CNN
-F 1 "VCC" H 5550 3150 50  0000 C CNN
-F 2 "" H 5550 3000 50  0001 C CNN
-F 3 "" H 5550 3000 50  0001 C CNN
-	1    5550 3000
-	1    0    0    -1
-$EndComp
-$Comp
-L crf_1:MPU9250 U10
+L crf_1:MPU9250 U9
 U 1 1 5A8CD83F
 P 4425 3800
-F 0 "U10" H 4350 4625 50  0000 L BNN
+F 0 "U9" H 4350 4625 50  0000 L BNN
 F 1 "MPU9250" H 4250 2900 50  0000 L BNN
 F 2 "Housings_DFN_QFN:QFN-24_3x3mm_Pitch0.4mm" H 3400 4725 50  0001 L BNN
@@
 	1    0    0    -1
 $EndComp
-Text HLabel 2950 4400 0    60   Input ~ 0
-SCL
-Text HLabel 2950 4500 0    60   Input ~ 0
+Text HLabel 3875 4500 0    60   Input ~ 0
 SDA
 Wire Wire Line
@@
 	4975 4400 5150 4400
 Wire Wire Line
-	5550 3100 5550 3000
+	5350 3100 5350 3025
 Wire Wire Line
 	5550 4500 5550 4250
-Wire Wire Line
-	2950 4500 3375 4500
-Wire Wire Line
-	3375 4500 3375 4325
-Wire Wire Line
-	3125 3850 3125 3925
-Wire Wire Line
-	3125 3925 3375 3925
-Wire Wire Line
-	3375 3925 3375 4025
-Wire Wire Line
-	2950 4400 3125 4400
-Wire Wire Line
-	3125 4400 3125 4325
 Wire Wire Line
 	5150 4500 5350 4500
@@
 	5350 3300 5550 3300
 Wire Wire Line
-	5350 3100 5550 3100
-Wire Wire Line
 	5350 3200 5350 3300
-Wire Wire Line
-	3125 3925 3125 4025
-Wire Wire Line
-	3125 4400 3875 4400
-Wire Wire Line
-	3375 4500 3875 4500
-Wire Wire Line
-	3375 3925 3525 3925
 Wire Wire Line
 	3800 3800 3875 3800
@@
 Connection ~ 5350 3100
 Connection ~ 5350 3200
-Connection ~ 3125 3925
-Connection ~ 3125 4400
-Connection ~ 3375 4500
-Connection ~ 3375 3925
 Connection ~ 3800 3800
 NoConn ~ 3875 3200
@@
 NoConn ~ 3875 3400
 NoConn ~ 3875 3100
+$Comp
+L Device:C C49
+U 1 1 5A8CE80E
+P 5150 4100
+F 0 "C49" H 5150 4000 50  0000 L CNN
+F 1 "100n" H 5150 4200 50  0000 L CNN
+F 2 "Capacitors_SMD:C_0603" H 5188 3950 50  0001 C CNN
+F 3 "" H 5150 4100 50  0001 C CNN
+F 4 "C0603X104J5RACTU" H 4975 4100 50  0001 C CNN "manf#"
+	1    5150 4100
+	1    0    0    1
+$EndComp
+Text HLabel 3875 4400 0    60   Input ~ 0
+SCL
+$Comp
+L power:VCC #PWR0112
+U 1 1 5AF1D01C
+P 5350 3025
+F 0 "#PWR0112" H 5350 2875 50  0001 C CNN
+F 1 "VCC" H 5350 3175 50  0000 C CNN
+F 2 "" H 5350 3025 50  0001 C CNN
+F 3 "" H 5350 3025 50  0001 C CNN
+	1    5350 3025
+	1    0    0    -1
+$EndComp
 $EndSCHEMATC
