File: design/TESC.kicad_pcb (KiCad board)
At the start: 4 copper layers, 62.5 x 60 mm, 141 parts, among them P1 USB_OTG, P10 PH_C, P11 SUPPLY, P12 GND, P2 CAN, P4 HALL_ENC, P5 COM, P6 SERVO, P7 SWD, P8 PH_A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

Commit message: Add LEO MOTION logo
Parts:
- added G***: LOGO, CRF1:Reinfored logo, B.Cu at (124.0, 69.1)
Other:
- board text removed: "MADE IN CHINA"
- board text removed: "TESC"

Commit message: Generate Gerber files
Parts:
- removed the G*** at (124.0, 69.1)
- added G***: LOGO, CRF1:TESC-logo, B.Cu at (123.2, 69.1)
